File: OpenHT-RF/fpga.kicad_sch (KiCad schematic)
At the start: 1 part, among them IC1 LIFCL-40-7SG72I

Commit message: Added FPGA power rails
Parts:
- added FB1, FB2, FB3, FB4: FerriteBead_Small, symbol Device:FerriteBead_Small
Connections:
- net VCC: now reaches IC1.12 (VCC_2)
- net VCC: now also IC1.21 (VCC_3), IC1.35 (VCC_4), IC1.38 (VCC_5), IC1.40 (VCC_6), IC1.6 (VCC_1), IC1.62 (VCC_7), IC1.63 (VCCPLLDPHY0), IC1.70 (VCCDPHY0_1), IC1.72 (VCCDPHY0_2), FB1.2
- net VCCAUX: now reaches IC1.17 (VCCAUXH5)
- net VCCAUX: now also IC1.29 (VCCAUXH3), IC1.39 (VCCAUX_2), IC1.47 (VCCAUX_3), IC1.7 (VCCAUX_1), FB2.2
- net VCCIO: now reaches IC1.18 (VCCIO5)
- net VCCIO: now also IC1.26 (VCCIO3_1), IC1.32 (VCCIO3_2), IC1.49 (VCCIO1), IC1.54 (VCCIO0), FB3.2
- net VCCADPHY: now reaches IC1.71 (VCCADPHY0)
- net VCCADPHY: now also FB4.2
- net GND: now reaches IC1.73 (VSS)
- new net +1V0: FB1.1
- new net +1V8: FB2.1, FB4.1
- new net +3V3: FB3.1
Other:
- note added: "Analog"
- note added: "Idk which supply it corresponds to"

Commit message: FPGA diagram [WIP]
Parts:
- added C1, C10, C11, C12, C13, C14, C15, C16, C17, C18, C19, C2, C20, C21, C22, C3, C4, C5, C6, C7, C8, C9: 0.1uF, symbol Device:C
- added C23, C24, C25, C26: 1uF, symbol Device:C
- added JP1: Jumper_3_Bridged12, symbol Jumper:Jumper_3_Bridged12
- added R10, R2, R3, R4, R5, R7, R8, R9: 100R, symbol Device:R
- added R6: 10kR, symbol Device:R
Connections:
- net GND: now also C1.2, C10.2, C11.2, C12.2, C13.2, C14.2, C15.2, C16.2, C17.2, C18.2, C19.2, C2.2, C20.2, C21.2, C22.2, C23.2, C24.2, C25.2, C26.2, C3.2, C4.2, C5.2, C6.2, C7.2, C8.2, C9.2, JP1.1 (A)
- net VCC: now also IC1.18 (VCCIO5), IC1.26 (VCCIO3_1), IC1.32 (VCCIO3_2), C1.1, C10.1, C11.1, C18.1, C19.1, C2.1, C20.1, C23.1, C3.1, C4.1, C5.1, C6.1, C7.1, C8.1, C9.1
- net VCCADPHY: now also C17.1, C25.1
- net VCCAUX: now also C12.1, C13.1, C14.1, C15.1, C16.1, C24.1
- net VCCIO: now also R6.1; no longer FB3.2, IC1.18 (VCCIO5), IC1.26 (VCCIO3_1), IC1.32 (VCCIO3_2), IC1.49 (VCCIO1), IC1.54 (VCCIO0)
- net LVDS_RXCLK_P: now reaches IC1.22 (PB54A)
- net LVDS_RXCLK_N: now reaches IC1.23 (PB54B)
- net LVDS_RX0_P: now reaches IC1.24 (PB58A)
- net LVDS_RX0_N: now reaches IC1.25 (PB58B)
- net LVDS_RX1_P: now reaches IC1.27 (PB68A)
- net LVDS_RX1_N: now reaches IC1.28 (PB68B)
- net LVDS_TXCLK_P: now reaches IC1.30 (PB72A)
- net LVDS_TXCLK_N: now reaches IC1.31 (PB72B)
- net LVDS_TX0_P: now reaches IC1.33 (PB74A)
- net LVDS_TX0_N: now reaches IC1.34 (PB74B)
- net at IC1.41 (PR13A): now also R4.1
- net at IC1.45 (PR10B): now also R3.1
- net at IC1.46 (PR8B): now also R2.1
- net at IC1.48 (PR6B): now also R5.1
- net at IC1.50 (JTAG_EN): now also JP1.2 (C)
- net at IC1.55 (PT80B): now also R7.1
- net at IC1.56 (PT78A): now also R8.1
- net at IC1.57 (PT78B): now also R9.1
- net at IC1.58 (PT76B): now also R10.1
- net CLK_IN: now reaches IC1.59 (PT76A)
- net PROGRAMN: now reaches IC1.60 (PT74B)
- new net: JP1.3 (B), R6.2
- new net M_SPI_CLK: R10.2
- new net M_SPI_MISO: R8.2
- new net M_SPI_MOSI: R9.2
- new net M_SPI_SS: R7.2
- new net S_SPI_CLK: R4.2
- new net S_SPI_CS: R5.2
- new net S_SPI_MISO: R3.2
- new net S_SPI_MOSI: R2.2
- new net VCCIO_3V3: C21.1, C22.1, C26.1, FB3.2, IC1.49 (VCCIO1), IC1.54 (VCCIO0)
Other:
- note added: "Analog, may not be required"
- note removed: "Analog"
- note removed: "Idk which supply it corresponds to"
- moved on the sheet: FB2, FB3, FB4

Commit message: FPGA Diagram [WIP]
Connections:
- net VCC: now also IC1.5 (VCCPLL_ULC)
- net LVDS_RX0_N renamed LVDS_RX09_N
- net LVDS_RX0_P renamed LVDS_RX09_P
- net LVDS_RX1_N renamed LVDS_RX24_N
- net LVDS_RX1_P renamed LVDS_RX24_P
- net LVDS_TX0_N renamed LVDS_TX_N
- net LVDS_TX0_P renamed LVDS_TX_P
Changed lines of the file:
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@@
     (stroke (width 0) (type default))
-  )
-  (text_box "IDK which supply VCCPLL_ULC corresponds to. No ref in the datasheet."
-    (at 92.71 72.39 0) (size 17.78 13.97)
-    (stroke (width 0) (type default))
-    (fill (type none))
-    (effects (font (size 1.27 1.27)) (justify left top))
   )
   (text_box "If pulled high, the SPI pins will be reconfigured as JTAG pins"
@@
     (effects (font (size 1.27 1.27)) (justify left bottom))
   )
+  (label "VCC" (at 101.6 87.63 0) (fields_autoplaced)
+    (effects (font (size 1.27 1.27)) (justify left bottom))
+  )
   (label "TMS{slash}SCSN" (at 196.85 92.71 0) (fields_autoplaced)
     (effects (font (size 1.27 1.27)) (justify left bottom))
@@
     (effects (font (size 1.27 1.27)) (justify left))
   )
-  (hierarchical_label "LVDS_TX0_N" (shape input) (at 157.48 151.13 270) (fields_autoplaced)
+  (hierarchical_label "LVDS_TX_N" (shape input) (at 157.48 151.13 270) (fields_autoplaced)
     (effects (font (size 1.27 1.27)) (justify right))
   )
@@
     (effects (font (size 1.27 1.27)) (justify left))
   )
-  (hierarchical_label "LVDS_RX1_P" (shape input) (at 139.7 151.13 270) (fields_autoplaced)
+  (hierarchical_label "LVDS_RX24_P" (shape input) (at 139.7 151.13 270) (fields_autoplaced)
     (effects (font (size 1.27 1.27)) (justify right))
   )
@@
     (effects (font (size 1.27 1.27)) (justify left))
   )
-  (hierarchical_label "LVDS_RX0_N" (shape input) (at 134.62 151.13 270) (fields_autoplaced)
+  (hierarchical_label "LVDS_RX09_N" (shape input) (at 134.62 151.13 270) (fields_autoplaced)
     (effects (font (size 1.27 1.27)) (justify right))
   )
-  (hierarchical_label "LVDS_TX0_P" (shape input) (at 154.94 151.13 270) (fields_autoplaced)
+  (hierarchical_label "LVDS_TX_P" (shape input) (at 154.94 151.13 270) (fields_autoplaced)
     (effects (font (size 1.27 1.27)) (justify right))
   )
-  (hierarchical_label "LVDS_RX1_N" (shape input) (at 142.24 151.13 270) (fields_autoplaced)
+  (hierarchical_label "LVDS_RX24_N" (shape input) (at 142.24 151.13 270) (fields_autoplaced)
     (effects (font (size 1.27 1.27)) (justify right))
   )
@@
     (effects (font (size 1.27 1.27)) (justify right))
   )
-  (hierarchical_label "LVDS_RX0_P" (shape input) (at 132.08 151.13 270) (fields_autoplaced)
+  (hierarchical_label "LVDS_RX09_P" (shape input) (at 132.08 151.13 270) (fields_autoplaced)
     (effects (font (size 1.27 1.27)) (justify right))
   )

Commit message: Updated FPGA, RF and connectors sheets [WIP]
Parts:
- removed R10, R2, R3, R4, R5, R7, R8, R9: 100R, symbol Device:R
Connections:
- net S_SPI_CLK: now also IC1.41 (PR13A)
- net S_SPI_CS: now also IC1.48 (PR6B)
- net S_SPI_MISO: now also IC1.45 (PR10B)
- net S_SPI_MOSI: now also IC1.46 (PR8B)

Commit message: Updated FPGA, RF and connectors sheets [WIP]
Connections:
- net IO0: now reaches IC1.42 (PR11A)
- net IO1: now reaches IC1.44 (PR11B)
- net IO2: now reaches IC1.51 (PT80A)
- net IO3: now reaches IC1.52 (PT82A)
- net IO4: now reaches IC1.53 (PT82B)
- net IO5: now reaches IC1.55 (PT80B)
- net IO6: now reaches IC1.56 (PT78A)
- net IO7: now reaches IC1.57 (PT78B)
- net DONE: now reaches IC1.58 (PT76B)
- net INITN: now reaches IC1.61 (PT74A)
- no-connect marks 0 -> 10
Changed lines of the file:
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@@
   (junction (at 38.1 97.79) (diameter 0) (color 0 0 0 0)
   )
+  (no_connect (at 111.76 77.47))
+  (no_connect (at 134.62 52.07))
+  (no_connect (at 111.76 82.55))
+  (no_connect (at 111.76 85.09))
+  (no_connect (at 137.16 52.07))
+  (no_connect (at 132.08 52.07))
+  (no_connect (at 129.54 52.07))
+  (no_connect (at 139.7 52.07))
+  (no_connect (at 142.24 52.07))
+  (no_connect (at 111.76 80.01))
   (wire (pts (xy 24.13 64.77) (xy 24.13 66.04))
     (stroke (width 0) (type default))
@@
     (stroke (width 0) (type default))
   )
+  (wire (pts (xy 172.72 82.55) (xy 187.96 82.55))
+    (stroke (width 0) (type default))
+  )
   (wire (pts (xy 46.99 162.56) (xy 46.99 160.02))
     (stroke (width 0) (type default))
@@
     (stroke (width 0) (type default))
   )
+  (wire (pts (xy 157.48 52.07) (xy 157.48 44.45))
+    (stroke (width 0) (type default))
+  )
   (wire (pts (xy 38.1 118.11) (xy 38.1 120.65))
     (stroke (width 0) (type default))
@@
     (stroke (width 0) (type default))
   )
+  (wire (pts (xy 172.72 80.01) (xy 187.96 80.01))
+    (stroke (width 0) (type default))
+  )
   (wire (pts (xy 172.72 87.63) (xy 220.98 87.63))
     (stroke (width 0) (type default))
@@
     (stroke (width 0) (type default))
   )
+  (wire (pts (xy 149.86 52.07) (xy 149.86 44.45))
+    (stroke (width 0) (type default))
+  )
   (wire (pts (xy 55.88 138.43) (xy 55.88 140.97))
     (stroke (width 0) (type default))
@@
     (stroke (width 0) (type default))
   )
+  (wire (pts (xy 172.72 107.95) (xy 187.96 107.95))
+    (stroke (width 0) (type default))
+  )
   (wire (pts (xy 172.72 113.03) (xy 184.15 113.03))
     (stroke (width 0) (type default))
@@
     (stroke (width 0) (type default))
   )
+  (wire (pts (xy 162.56 44.45) (xy 162.56 52.07))
+    (stroke (width 0) (type default))
+  )
   (wire (pts (xy 152.4 140.97) (xy 152.4 149.86))
     (stroke (width 0) (type default))
@@
     (stroke (width 0) (type default))
   )
+  (wire (pts (xy 160.02 44.45) (xy 160.02 52.07))
+    (stroke (width 0) (type default))
+  )
+  (wire (pts (xy 172.72 85.09) (xy 187.96 85.09))
+    (stroke (width 0) (type default))
+  )
   (wire (pts (xy 48.26 82.55) (xy 67.31 82.55))
     (stroke (width 0) (type default))
@@
     (stroke (width 0) (type default))
   )
+  (wire (pts (xy 172.72 102.87) (xy 187.96 102.87))
+    (stroke (width 0) (type default))
+  )
   (wire (pts (xy 139.7 140.97) (xy 139.7 151.13))
     (stroke (width 0) (type default))
@@
   )
   (wire (pts (xy 73.66 120.65) (xy 73.66 118.11))
+    (stroke (width 0) (type default))
+  )
+  (wire (pts (xy 165.1 44.45) (xy 165.1 52.07))
     (stroke (width 0) (type default))
   )
@@
     (effects (font (size 1.27 1.27)) (justify left bottom))
   )
+  (hierarchical_label "IO2" (shape bidirectional) (at 187.96 85.09 0) (fields_autoplaced)
+    (effects (font (size 1.27 1.27)) (justify left))
+  )
+  (hierarchical_label "INITN" (shape bidirectional) (at 149.86 44.45 90) (fields_autoplaced)
+    (effects (font (size 1.27 1.27)) (justify left))
+  )
   (hierarchical_label "S_SPI_MOSI" (shape input) (at 187.96 97.79 0) (fields_autoplaced)
     (effects (font (size 1.27 1.27)) (justify left))
@@
     (effects (font (size 1.27 1.27)) (justify right))
   )
+  (hierarchical_label "IO0" (shape bidirectional) (at 187.96 107.95 0) (fields_autoplaced)
+    (effects (font (size 1.27 1.27)) (justify left))
+  )
+  (hierarchical_label "IO1" (shape bidirectional) (at 187.96 102.87 0) (fields_autoplaced)
+    (effects (font (size 1.27 1.27)) (justify left))
+  )
   (hierarchical_label "LVDS_RX09_N" (shape input) (at 134.62 151.13 270) (fields_autoplaced)
     (effects (font (size 1.27 1.27)) (justify right))
@@
     (effects (font (size 1.27 1.27)) (justify right))
   )
+  (hierarchical_label "IO6" (shape bidirectional) (at 162.56 44.45 90) (fields_autoplaced)
+    (effects (font (size 1.27 1.27)) (justify left))
+  )
   (hierarchical_label "S_SPI_MISO" (shape output) (at 187.96 100.33 0) (fields_autoplaced)
     (effects (font (size 1.27 1.27)) (justify left))
@@
     (effects (font (size 1.27 1.27)) (justify left))
   )
+  (hierarchical_label "IO4" (shape bidirectional) (at 187.96 80.01 0) (fields_autoplaced)
+    (effects (font (size 1.27 1.27)) (justify left))
+  )
   (hierarchical_label "LVDS_RXCLK_N" (shape input) (at 129.54 151.13 270) (fields_autoplaced)
     (effects (font (size 1.27 1.27)) (justify right))
   )
+  (hierarchical_label "IO5" (shape bidirectional) (at 165.1 44.45 90) (fields_autoplaced)
+    (effects (font (size 1.27 1.27)) (justify left))
+  )
   (hierarchical_label "LVDS_TXCLK_P" (shape output) (at 147.32 151.13 270) (fields_autoplaced)
     (effects (font (size 1.27 1.27)) (justify right))
@@
     (effects (font (size 1.27 1.27)) (justify right))
   )
+  (hierarchical_label "IO7" (shape bidirectional) (at 160.02 44.45 90) (fields_autoplaced)
+    (effects (font (size 1.27 1.27)) (justify left))
+  )
   (hierarchical_label "LVDS_RX09_P" (shape input) (at 132.08 151.13 270) (fields_autoplaced)
     (effects (font (size 1.27 1.27)) (justify right))
   )
+  (hierarchical_label "DONE" (shape bidirectional) (at 157.48 44.45 90) (fields_autoplaced)
+    (effects (font (size 1.27 1.27)) (justify left))
+  )
+  (hierarchical_label "IO3" (shape bidirectional) (at 187.96 82.55 0) (fields_autoplaced)
+    (effects (font (size 1.27 1.27)) (justify left))
+  )
   (hierarchical_label "CLK_IN" (shape input) (at 154.94 44.45 90) (fields_autoplaced)

Commit message: Updated FPGA schematic to use M17_kicad_library
Parts:
- removed IC1: LIFCL-40-7SG72I, QFN50P1000X1000X90-73N-D, symbol LIFCL-40:LIFCL-40-7SG72I
- added U1: ~, symbol M17_FPGA:LIFCL-40-7SG72I
Connections:
- net VCCIO is gone; now on net VCCIO_3V3: R6.1
- net CLK_IN: now also U1.59 (PT76A/MCLK)
- net DONE: now also U1.58 (PT76B/DONE)
- net GND: now also U1.73 (GND)
- net INITN: now also U1.61 (PT74A/INITN)
- net IO0: now also U1.42 (PR11A/SDA)
- net IO1: now also U1.44 (PR11B/SCL)
- net IO2: now also U1.51 (PT80A/MISO)
- net IO3: now also U1.52 (PT82A)
- net IO4: now also U1.53 (PT82B/MCSNO)
- net IO5: now also U1.55 (PT80B)
- net IO6: now also U1.56 (PT78A/MCSN)
- net IO7: now also U1.57 (PT78B/MOSI)
- net PROGRAMN: now also U1.60 (PT74B/PROGRAMN)
- net S_SPI_CLK: now also U1.41 (P13A/TCK/SCLK)
- net S_SPI_CS: now also U1.48 (PR6B/TMS/SCSN)
- net S_SPI_MISO: now also U1.45 (PR10B/TDO/SSO)
- net S_SPI_MOSI: now also U1.46 (PR8B/TDI/SSI)
- net VCC: now also U1.12 (VCC), U1.18 (VCCIO5), U1.21 (VCC), U1.26 (VCCIO3), U1.32 (VCCIO3), U1.35 (VCC), U1.38 (VCC), U1.40 (VCC), U1.5 (VCCPLL_ULC), U1.6 (VCC), U1.62 (VCC), U1.63 (VCCPLLDPHY0), U1.70 (VCCDPHY0), U1.72 (VCCDPHY0)
- net VCCAUX: now also U1.17 (VCCAUXH5), U1.29 (VCCAUXH3), U1.47 (VCCAUX), U1.7 (VCCAUX); no longer C16.1
- net VCCIO_3V3: now also U1.49 (VCCIO1), U1.54 (VCCIO0)
- net at JP1.2 (C): now also U1.50 (JTAG_EN)
- net VCCADPHY renamed VCCA_1V8
- net VCCA_1V8: now also C16.1, U1.39 (VCCADC18), U1.71 (VCCADPHY0)
Other:
- note removed: "Analog, may not be required"
- moved on the sheet: C1, C10, C11, C12, C13, C14, C15, C17, C18, C19, C2, C20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

Commit message: Updated M17_kicad_library
Parts:
- U1: footprint (none) -> M17_QFN:QFN-72-1EP_10x10mm_P0.5mm_EP6.2x6.2mm
Changed lines of the file:
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@@
       (effects (font (size 1.27 1.27)))
     )
-    (property "Footprint" "" (at 219.71 62.23 0)
-      (effects (font (size 1.27 1.27)) hide)
-    )
-    (property "Datasheet" "" (at 219.71 62.23 0)
+    (property "Footprint" "M17_QFN:QFN-72-1EP_10x10mm_P0.5mm_EP6.2x6.2mm" (at 219.71 62.23 0)
+      (effects (font (size 1.27 1.27)) hide)
+    )
+    (property "Datasheet" "https://www.latticesemi.com/-/media/LatticeSemi/Documents/DataSheets/CrossLink/FPGA-DS-02049-1-6-CrossLink-NX-Family.ashx?document_id=52780" (at 219.71 62.23 0)
       (effects (font (size 1.27 1.27)) hide)
     )
@@
       (effects (font (size 1.27 1.27)))
     )
-    (property "Footprint" "" (at 144.78 21.59 0)
-      (effects (font (size 1.27 1.27)) hide)
-    )
-    (property "Datasheet" "" (at 144.78 21.59 0)
+    (property "Footprint" "M17_QFN:QFN-72-1EP_10x10mm_P0.5mm_EP6.2x6.2mm" (at 144.78 21.59 0)
+      (effects (font (size 1.27 1.27)) hide)
+    )
+    (property "Datasheet" "https://www.latticesemi.com/-/media/LatticeSemi/Documents/DataSheets/CrossLink/FPGA-DS-02049-1-6-CrossLink-NX-Family.ashx?document_id=52780" (at 144.78 21.59 0)
       (effects (font (size 1.27 1.27)) hide)
     )
@@
     )
   )
-  (symbol (lib_name "LIFCL-40-7SG72I_1") (lib_id "M17_FPGA:LIFCL-40-7SG72I") (at 213.36 124.46 0) (unit 5)
+  (symbol (lib_id "M17_FPGA:LIFCL-40-7SG72I") (at 213.36 124.46 0) (unit 5)
     (in_bom yes) (on_board yes) (dnp no)
     (property "Reference" "U1" (at 199.39 107.95 0)
@@
       (effects (font (size 1.27 1.27)))
     )
-    (property "Footprint" "" (at 220.98 109.22 0)
-      (effects (font (size 1.27 1.27)) hide)
-    )
-    (property "Datasheet" "" (at 220.98 109.22 0)
+    (property "Footprint" "M17_QFN:QFN-72-1EP_10x10mm_P0.5mm_EP6.2x6.2mm" (at 220.98 109.22 0)
+      (effects (font (size 1.27 1.27)) hide)
+    )
+    (property "Datasheet" "https://www.latticesemi.com/-/media/LatticeSemi/Documents/DataSheets/CrossLink/FPGA-DS-02049-1-6-CrossLink-NX-Family.ashx?document_id=52780" (at 220.98 109.22 0)
       (effects (font (size 1.27 1.27)) hide)
     )
@@
       (effects (font (size 1.27 1.27)))
     )
-    (property "Footprint" "" (at 144.78 119.38 0)
-      (effects (font (size 1.27 1.27)) hide)
-    )
-    (property "Datasheet" "" (at 144.78 119.38 0)
+    (property "Footprint" "M17_QFN:QFN-72-1EP_10x10mm_P0.5mm_EP6.2x6.2mm" (at 144.78 119.38 0)
+      (effects (font (size 1.27 1.27)) hide)
+    )
+    (property "Datasheet" "https://www.latticesemi.com/-/media/LatticeSemi/Documents/DataSheets/CrossLink/FPGA-DS-02049-1-6-CrossLink-NX-Family.ashx?document_id=52780" (at 144.78 119.38 0)
       (effects (font (size 1.27 1.27)) hide)
     )
@@
       (effects (font (size 1.27 1.27)))
     )
-    (property "Footprint" "" (at 219.71 20.32 0)
-      (effects (font (size 1.27 1.27)) hide)
-    )
-    (property "Datasheet" "" (at 219.71 20.32 0)
+    (property "Footprint" "M17_QFN:QFN-72-1EP_10x10mm_P0.5mm_EP6.2x6.2mm" (at 219.71 20.32 0)
+      (effects (font (size 1.27 1.27)) hide)
+    )
+    (property "Datasheet" "https://www.latticesemi.com/-/media/LatticeSemi/Documents/DataSheets/CrossLink/FPGA-DS-02049-1-6-CrossLink-NX-Family.ashx?document_id=52780" (at 219.71 20.32 0)
       (effects (font (size 1.27 1.27)) hide)
     )
@@
       (effects (font (size 1.27 1.27)))
     )
-    (property "Footprint" "" (at 144.78 64.77 0)
-      (effects (font (size 1.27 1.27)) hide)
-    )
-    (property "Datasheet" "" (at 144.78 64.77 0)
-      (effects (font (size 1.27 1.27)) hide)
-    )
+    (property "Footprint" "M17_QFN:QFN-72-1EP_10x10mm_P0.5mm_EP6.2x6.2mm" (at 144.78 64.77 0)
+      (effects (font (size 1.27 1.27)) hide)
+    )
+    (property "Datasheet" "https://www.latticesemi.com/-/media/LatticeSemi/Documents/DataSheets/CrossLink/FPGA-DS-02049-1-6-CrossLink-NX-Family.ashx?document_id=52780" (at 144.78 64.77 0)
+      (effects (font (size 1.27 1.27)) hide)
+    )
