File: OpenHT-RF/fpga.kicad_sch (KiCad schematic)
At the start: 33 parts

Commit message: Updated M17_kicad_library
Parts:
- U1: value ~ -> LIFCL-40-7SG72I
Connections:
- net LVDS_RX09_N: now also U1.25 (PB58B)
- net LVDS_RX09_P: now also U1.24 (PB58A)
- net LVDS_RX24_N: now also U1.28 (PB68B)
- net LVDS_RX24_P: now also U1.27 (PB68A)
- net LVDS_RXCLK_N: now also U1.23 (PB54B)
- net LVDS_RXCLK_P: now also U1.22 (PB54A)
- net LVDS_TXCLK_N: now also U1.31 (PB72B)
- net LVDS_TXCLK_P: now also U1.30 (PB72A)
- net LVDS_TX_N: now also U1.34 (PB74B)
- net LVDS_TX_P: now also U1.33 (PB74A)
Changed lines of the file:
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@@
     )
   )
-  (symbol (lib_id "M17_FPGA:LIFCL-40-7SG72I") (at 212.09 77.47 0) (unit 4)
+  (symbol (lib_id "M17_FPGA:LIFCL-40-7SG72I") (at 199.39 62.23 0) (unit 4)
     (in_bom yes) (on_board yes) (dnp no)
     (property "Reference" "U1" (at 199.39 60.96 0)
       (effects (font (size 1.27 1.27)) (justify left))
     )
-    (property "Value" "~" (at 219.71 62.23 0)
-      (effects (font (size 1.27 1.27)))
-    )
-    (property "Footprint" "M17_QFN:QFN-72-1EP_10x10mm_P0.5mm_EP6.2x6.2mm" (at 219.71 62.23 0)
-      (effects (font (size 1.27 1.27)) hide)
-    )
-    (property "Datasheet" "https://www.latticesemi.com/-/media/LatticeSemi/Documents/DataSheets/CrossLink/FPGA-DS-02049-1-6-CrossLink-NX-Family.ashx?document_id=52780" (at 219.71 62.23 0)
+    (property "Value" "LIFCL-40-7SG72I" (at 215.9 60.96 0)
+      (effects (font (size 1.27 1.27)))
+    )
+    (property "Footprint" "M17_QFN:QFN-72-1EP_10x10mm_P0.5mm_EP6.2x6.2mm" (at 207.01 46.99 0)
+      (effects (font (size 1.27 1.27)) hide)
+    )
+    (property "Datasheet" "https://www.latticesemi.com/-/media/LatticeSemi/Documents/DataSheets/CrossLink/FPGA-DS-02049-1-6-CrossLink-NX-Family.ashx?document_id=52780" (at 207.01 46.99 0)
       (effects (font (size 1.27 1.27)) hide)
     )
@@
     )
   )
-  (symbol (lib_id "M17_FPGA:LIFCL-40-7SG72I") (at 137.16 36.83 0) (unit 1)
+  (symbol (lib_id "M17_FPGA:LIFCL-40-7SG72I") (at 124.46 21.59 0) (unit 1)
     (in_bom yes) (on_board yes) (dnp no)
     (property "Reference" "U1" (at 124.46 20.32 0)
       (effects (font (size 1.27 1.27)) (justify left))
     )
-    (property "Value" "~" (at 144.78 21.59 0)
-      (effects (font (size 1.27 1.27)))
-    )
-    (property "Footprint" "M17_QFN:QFN-72-1EP_10x10mm_P0.5mm_EP6.2x6.2mm" (at 144.78 21.59 0)
-      (effects (font (size 1.27 1.27)) hide)
-    )
-    (property "Datasheet" "https://www.latticesemi.com/-/media/LatticeSemi/Documents/DataSheets/CrossLink/FPGA-DS-02049-1-6-CrossLink-NX-Family.ashx?document_id=52780" (at 144.78 21.59 0)
+    (property "Value" "LIFCL-40-7SG72I" (at 140.97 20.32 0)
+      (effects (font (size 1.27 1.27)))
+    )
+    (property "Footprint" "M17_QFN:QFN-72-1EP_10x10mm_P0.5mm_EP6.2x6.2mm" (at 132.08 6.35 0)
+      (effects (font (size 1.27 1.27)) hide)
+    )
+    (property "Datasheet" "https://www.latticesemi.com/-/media/LatticeSemi/Documents/DataSheets/CrossLink/FPGA-DS-02049-1-6-CrossLink-NX-Family.ashx?document_id=52780" (at 132.08 6.35 0)
       (effects (font (size 1.27 1.27)) hide)
     )
@@
     )
   )
-  (symbol (lib_id "M17_FPGA:LIFCL-40-7SG72I") (at 213.36 124.46 0) (unit 5)
+  (symbol (lib_id "M17_FPGA:LIFCL-40-7SG72I") (at 199.39 109.22 0) (unit 5)
     (in_bom yes) (on_board yes) (dnp no)
     (property "Reference" "U1" (at 199.39 107.95 0)
       (effects (font (size 1.27 1.27)) (justify left))
     )
-    (property "Value" "~" (at 220.98 109.22 0)
-      (effects (font (size 1.27 1.27)))
-    )
-    (property "Footprint" "M17_QFN:QFN-72-1EP_10x10mm_P0.5mm_EP6.2x6.2mm" (at 220.98 109.22 0)
-      (effects (font (size 1.27 1.27)) hide)
-    )
-    (property "Datasheet" "https://www.latticesemi.com/-/media/LatticeSemi/Documents/DataSheets/CrossLink/FPGA-DS-02049-1-6-CrossLink-NX-Family.ashx?document_id=52780" (at 220.98 109.22 0)
+    (property "Value" "LIFCL-40-7SG72I" (at 218.44 107.95 0)
+      (effects (font (size 1.27 1.27)))
+    )
+    (property "Footprint" "M17_QFN:QFN-72-1EP_10x10mm_P0.5mm_EP6.2x6.2mm" (at 207.01 93.98 0)
+      (effects (font (size 1.27 1.27)) hide)
+    )
+    (property "Datasheet" "https://www.latticesemi.com/-/media/LatticeSemi/Documents/DataSheets/CrossLink/FPGA-DS-02049-1-6-CrossLink-NX-Family.ashx?document_id=52780" (at 207.01 93.98 0)
       (effects (font (size 1.27 1.27)) hide)
     )
@@
     )
   )
-  (symbol (lib_id "M17_FPGA:LIFCL-40-7SG72I") (at 137.16 134.62 0) (unit 6)
+  (symbol (lib_id "M17_FPGA:LIFCL-40-7SG72I") (at 125.73 109.22 0) (unit 6)
     (in_bom yes) (on_board yes) (dnp no)
     (property "Reference" "U1" (at 125.73 107.95 0)
       (effects (font (size 1.27 1.27)) (justify left))
     )
-    (property "Value" "~" (at 144.78 119.38 0)
-      (effects (font (size 1.27 1.27)))
-    )
-    (property "Footprint" "M17_QFN:QFN-72-1EP_10x10mm_P0.5mm_EP6.2x6.2mm" (at 144.78 119.38 0)
-      (effects (font (size 1.27 1.27)) hide)
-    )
-    (property "Datasheet" "https://www.latticesemi.com/-/media/LatticeSemi/Documents/DataSheets/CrossLink/FPGA-DS-02049-1-6-CrossLink-NX-Family.ashx?document_id=52780" (at 144.78 119.38 0)
+    (property "Value" "LIFCL-40-7SG72I" (at 140.97 107.95 0)
+      (effects (font (size 1.27 1.27)))
+    )
+    (property "Footprint" "M17_QFN:QFN-72-1EP_10x10mm_P0.5mm_EP6.2x6.2mm" (at 133.35 93.98 0)
+      (effects (font (size 1.27 1.27)) hide)
+    )
+    (property "Datasheet" "https://www.latticesemi.com/-/media/LatticeSemi/Documents/DataSheets/CrossLink/FPGA-DS-02049-1-6-CrossLink-NX-Family.ashx?document_id=52780" (at 133.35 93.98 0)
       (effects (font (size 1.27 1.27)) hide)
     )
@@
     )
   )
-  (symbol (lib_id "M17_FPGA:LIFCL-40-7SG72I") (at 212.09 35.56 0) (unit 2)
+  (symbol (lib_id "M17_FPGA:LIFCL-40-7SG72I") (at 199.39 22.86 0) (unit 2)
     (in_bom yes) (on_board yes) (dnp no)
     (property "Reference" "U1" (at 199.39 21.59 0)
       (effects (font (size 1.27 1.27)) (justify left))
     )
-    (property "Value" "~" (at 219.71 20.32 0)
-      (effects (font (size 1.27 1.27)))
-    )
-    (property "Footprint" "M17_QFN:QFN-72-1EP_10x10mm_P0.5mm_EP6.2x6.2mm" (at 219.71 20.32 0)
-      (effects (font (size 1.27 1.27)) hide)
-    )
-    (property "Datasheet" "https://www.latticesemi.com/-/media/LatticeSemi/Documents/DataSheets/CrossLink/FPGA-DS-02049-1-6-CrossLink-NX-Family.ashx?document_id=52780" (at 219.71 20.32 0)
+    (property "Value" "LIFCL-40-7SG72I" (at 215.9 21.59 0)
+      (effects (font (size 1.27 1.27)))
+    )
+    (property "Footprint" "M17_QFN:QFN-72-1EP_10x10mm_P0.5mm_EP6.2x6.2mm" (at 207.01 7.62 0)
+      (effects (font (size 1.27 1.27)) hide)
+    )
+    (property "Datasheet" "https://www.latticesemi.com/-/media/LatticeSemi/Documents/DataSheets/CrossLink/FPGA-DS-02049-1-6-CrossLink-NX-Family.ashx?document_id=52780" (at 207.01 7.62 0)
       (effects (font (size 1.27 1.27)) hide)
     )
@@
     )
   )
-  (symbol (lib_id "M17_FPGA:LIFCL-40-7SG72I") (at 137.16 80.01 0) (unit 3)
+  (symbol (lib_id "M17_FPGA:LIFCL-40-7SG72I") (at 124.46 62.23 0) (unit 3)
     (in_bom yes) (on_board yes) (dnp no)
     (property "Reference" "U1" (at 124.46 60.96 0)
       (effects (font (size 1.27 1.27)) (justify left))
     )
-    (property "Value" "~" (at 144.78 64.77 0)
-      (effects (font (size 1.27 1.27)))
-    )
-    (property "Footprint" "M17_QFN:QFN-72-1EP_10x10mm_P0.5mm_EP6.2x6.2mm" (at 144.78 64.77 0)
-      (effects (font (size 1.27 1.27)) hide)
-    )
-    (property "Datasheet" "https://www.latticesemi.com/-/media/LatticeSemi/Documents/DataSheets/CrossLink/FPGA-DS-02049-1-6-CrossLink-NX-Family.ashx?document_id=52780" (at 144.78 64.77 0)
-      (effects (font (size 1.27 1.27)) hide)
-    )
+    (property "Value" "LIFCL-40-7SG72I" (at 140.97 60.96 0)
+      (effects (font (size 1.27 1.27)))
+    )
+    (property "Footprint" "M17_QFN:QFN-72-1EP_10x10mm_P0.5mm_EP6.2x6.2mm" (at 132.08 46.99 0)
+      (effects (font (size 1.27 1.27)) hide)
+    )
+    (property "Datasheet" "https://www.latticesemi.com/-/media/LatticeSemi/Documents/DataSheets/CrossLink/FPGA-DS-02049-1-6-CrossLink-NX-Family.ashx?document_id=52780" (at 132.08 46.99 0)
+      (effects (font (size 1.27 1.27)) hide)
+    )

Commit message: Updated FPGA power supply
Design updated according to Lattice Hardware Checklist (https://www.latticesemi.com/view_document?document_id=52782)
Parts:
- removed C22: 0.1uF, symbol Device:C
- removed C23, C26: 1uF, symbol Device:C
- added C55, C57: 10uF, symbol Device:C
- added C56, C58, C59: 0.1uF, symbol Device:C
- C10, C11, C16, C17, C18, C9: value 0.1uF -> 10uF
- C20: value 0.1uF -> 1uF
- C24: value 1uF -> 10uF
- C25: value 1uF -> 0.1uF
- FB2, FB4: value FerriteBead_Small -> 120R
Connections:
- net GND: now also C55.2, C56.2, C57.2, C58.2, C59.2
- net VCC: now also C57.1, C58.1, C59.1; no longer C18.1, U1.63 (VCCPLLDPHY0), U1.70 (VCCDPHY0), U1.72 (VCCDPHY0)
- net VCCAUX: now also C16.1
- net VCCIO_3V3: now also C18.1, C55.1, C56.1
- net VCCA_1V8: no longer names the net of C17.1, C25.1, FB4.2, U1.39 (VCCADC18)
- net VCCA_1V8: no longer C16.1, U1.71 (VCCADPHY0)
- no-connect marks 10 -> 27
Other:
- note added: "Leave VCCADC18 open if not used."
- moved on the sheet: C1, C12, C13, C14, C15, C2, C24, C3, C4, C5, C6, C7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

Commit message: Fixed FPGA power supply
vccio_1V8 is now correctly connected to 1V8
Connections:
- net VCC: no longer C19.1, C20.1, C57.1, C58.1, C59.1, U1.18 (VCCIO5), U1.26 (VCCIO3), U1.32 (VCCIO3)
- net VCCAUX: now also C19.1, C20.1, C57.1, C58.1, C59.1, U1.18 (VCCIO5), U1.26 (VCCIO3), U1.32 (VCCIO3)
Other:
- moved on the sheet: C18, C21, JP1, R6, U1B

Commit message: Optimised IO routing, renumbered components
Parts:
- added J401: Conn_01x06, symbol Connector_Generic:Conn_01x06
- C423: renamed from C17; now not fitted
- C424: renamed from C25; now not fitted
- FB404: renamed from FB4; now not fitted
- renumbered C9 to C401, C10 to C402, C24 to C403, C11 to C404, C16 to C405, C1 to C406, C12 to C407, C2 to C408, C13 to C409, C3 to C410, C14 to C411, C4 to C412, C15 to C413, C5 to C414, C6 to C415, C57 to C416, C7 to C417, C58 to C418, C55 to C419, C8 to C420, C19 to C421, C56 to C422, C18 to C425, C20 to C426, C21 to C427, C59 to C428, FB1 to FB401, FB3 to FB402, FB2 to FB403, JP1 to JP401, R6 to R401, U1 to U401
Connections:
- net GND: now also J401.6 (Pin_6)
- net S_SPI_CLK: now also J401.1 (Pin_1)
- net S_SPI_CS: now also J401.2 (Pin_2)
- net S_SPI_MISO: now also J401.4 (Pin_4)
- net S_SPI_MOSI: now also J401.3 (Pin_3)
- new net +3.3V: J401.5 (Pin_5)

Commit message: Added MPN for ferrite beads
Parts:
- FB401, FB402: value FerriteBead_Small -> BLM15AG121SN1D
- FB403, FB404: value 120R -> BLM15AG121SN1D
Changed lines of the file:
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@@
     (stroke (width 0) (type default))
   )
-  (wire (pts (xy 165.1 115.57) (xy 165.1 116.84))
+  (wire (pts (xy 162.56 115.57) (xy 162.56 116.84))
     (stroke (width 0) (type default))
   )
@@
     (stroke (width 0) (type default))
   )
-  (wire (pts (xy 165.1 116.84) (xy 170.18 116.84))
+  (wire (pts (xy 162.56 116.84) (xy 170.18 116.84))
     (stroke (width 0) (type default))
   )
@@
       (effects (font (size 1.27 1.27)))
     )
-    (property "Value" "120R" (at 29.1719 41.91 90)
+    (property "Value" "BLM15AG121SN1D" (at 29.1719 41.91 90)
       (effects (font (size 1.27 1.27)))
     )
@@
       (effects (font (size 1.27 1.27)))
     )
-    (property "Value" "120R" (at 172.6819 114.3 90)
+    (property "Value" "BLM15AG121SN1D" (at 172.6819 114.3 90)
       (effects (font (size 1.27 1.27)))
     )
@@
       (effects (font (size 1.27 1.27)))
     )
-    (property "Value" "FerriteBead_Small" (at 29.1719 31.75 90)
+    (property "Value" "BLM15AG121SN1D" (at 29.1719 31.75 90)
       (effects (font (size 1.27 1.27)))
     )
@@
     )
   )
-  (symbol (lib_id "power:+1V8") (at 165.1 115.57 0) (unit 1)
-    (in_bom yes) (on_board yes) (dnp no) (fields_autoplaced)
-    (property "Reference" "#PWR0426" (at 165.1 119.38 0)
-      (effects (font (size 1.27 1.27)) hide)
-    )
-    (property "Value" "+1V8" (at 165.1 111.76 0)
-      (effects (font (size 1.27 1.27)))
-    )
-    (property "Footprint" "" (at 165.1 115.57 0)
-      (effects (font (size 1.27 1.27)) hide)
-    )
-    (property "Datasheet" "" (at 165.1 115.57 0)
+  (symbol (lib_id "power:+1V8") (at 162.56 115.57 0) (unit 1)
+    (in_bom yes) (on_board yes) (dnp no) (fields_autoplaced)
+    (property "Reference" "#PWR0426" (at 162.56 119.38 0)
+      (effects (font (size 1.27 1.27)) hide)
+    )
+    (property "Value" "+1V8" (at 162.56 111.76 0)
+      (effects (font (size 1.27 1.27)))
+    )
+    (property "Footprint" "" (at 162.56 115.57 0)
+      (effects (font (size 1.27 1.27)) hide)
+    )
+    (property "Datasheet" "" (at 162.56 115.57 0)
       (effects (font (size 1.27 1.27)) hide)
     )
@@
       (effects (font (size 1.27 1.27)))
     )
-    (property "Value" "FerriteBead_Small" (at 29.1719 21.59 90)
-      (effects (font (size 1.27 1.27)))
-    )
+    (property "Value" "BLM15AG121SN1D" (at 29.1719 21.59 90)
+      (effects (font (size 1.27 1.27)))
+    )

Commit message: [WIP] symbol-footprint association
Parts:
- C401, C402, C403, C404, C405, C416, C419, C423, C425: footprint (none) -> Capacitor_SMD:C_0805_2012Metric
- C406, C407, C408, C409, C410, C411, C412, C413, C414, C415, C417, C418, C420, C421, C422, C424, C426, C427, C428: footprint (none) -> Capacitor_SMD:C_0402_1005Metric
- FB401, FB402, FB403, FB404: footprint (none) -> Inductor_SMD:L_0402_1005Metric
- J401: footprint (none) -> Connector_PinSocket_2.54mm:PinSocket_1x06_P2.54mm_Horizontal
- JP401: footprint (none) -> Connector_PinHeader_2.54mm:PinHeader_1x03_P2.54mm_Vertical
- R401: footprint (none) -> Resistor_SMD:R_0402_1005Metric
Changed lines of the file:
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@@
       (effects (font (size 1.27 1.27)) (justify left))
     )
-    (property "Footprint" "" (at 101.2952 99.06 0)
+    (property "Footprint" "Capacitor_SMD:C_0402_1005Metric" (at 101.2952 99.06 0)
       (effects (font (size 1.27 1.27)) hide)
     )
@@
       (effects (font (size 1.27 1.27)) (justify left))
     )
-    (property "Footprint" "" (at 201.6252 76.2 0)
+    (property "Footprint" "Capacitor_SMD:C_0402_1005Metric" (at 201.6252 76.2 0)
       (effects (font (size 1.27 1.27)) hide)
     )
@@
       (effects (font (size 1.27 1.27)) (justify left))
     )
-    (property "Footprint" "" (at 103.8352 76.2 0)
+    (property "Footprint" "Capacitor_SMD:C_0402_1005Metric" (at 103.8352 76.2 0)
       (effects (font (size 1.27 1.27)) hide)
     )
@@
       (effects (font (size 1.27 1.27)) (justify left))
     )
-    (property "Footprint" "" (at 267.462 33.02 90)
+    (property "Footprint" "Resistor_SMD:R_0402_1005Metric" (at 267.462 33.02 90)
       (effects (font (size 1.27 1.27)) hide)
     )
@@
       (effects (font (size 1.27 1.27)))
     )
-    (property "Footprint" "" (at 29.21 46.228 90)
+    (property "Footprint" "Inductor_SMD:L_0402_1005Metric" (at 29.21 46.228 90)
       (effects (font (size 1.27 1.27)) hide)
     )
@@
       (effects (font (size 1.27 1.27)) (justify left))
     )
-    (property "Footprint" "" (at 108.9152 35.56 0)
+    (property "Footprint" "Capacitor_SMD:C_0805_2012Metric" (at 108.9152 35.56 0)
       (effects (font (size 1.27 1.27)) hide)
     )
@@
       (effects (font (size 1.27 1.27)) (justify left))
     )
-    (property "Footprint" "" (at 83.5152 99.06 0)
+    (property "Footprint" "Capacitor_SMD:C_0402_1005Metric" (at 83.5152 99.06 0)
       (effects (font (size 1.27 1.27)) hide)
     )
@@
       (effects (font (size 1.27 1.27)) (justify left))
     )
-    (property "Footprint" "" (at 110.1852 99.06 0)
+    (property "Footprint" "Capacitor_SMD:C_0402_1005Metric" (at 110.1852 99.06 0)
       (effects (font (size 1.27 1.27)) hide)
     )
@@
       (effects (font (size 1.27 1.27)) (justify left))
     )
-    (property "Footprint" "" (at 65.7352 99.06 0)
+    (property "Footprint" "Capacitor_SMD:C_0402_1005Metric" (at 65.7352 99.06 0)
       (effects (font (size 1.27 1.27)) hide)
     )
@@
       (effects (font (size 1.27 1.27)) (justify left))
     )
-    (property "Footprint" "" (at 47.9552 99.06 0)
+    (property "Footprint" "Capacitor_SMD:C_0402_1005Metric" (at 47.9552 99.06 0)
       (effects (font (size 1.27 1.27)) hide)
     )
@@
       (effects (font (size 1.27 1.27)) (justify left))
     )
-    (property "Footprint" "" (at 259.08 120.65 0)
+    (property "Footprint" "Connector_PinSocket_2.54mm:PinSocket_1x06_P2.54mm_Horizontal" (at 259.08 120.65 0)
       (effects (font (size 1.27 1.27)) hide)
     )
@@
       (effects (font (size 1.27 1.27)) (justify left))
     )
-    (property "Footprint" "" (at 92.4052 99.06 0)
+    (property "Footprint" "Capacitor_SMD:C_0402_1005Metric" (at 92.4052 99.06 0)
       (effects (font (size 1.27 1.27)) hide)
     )
@@
       (effects (font (size 1.27 1.27)))
     )
-    (property "Footprint" "" (at 172.72 118.618 90)
+    (property "Footprint" "Inductor_SMD:L_0402_1005Metric" (at 172.72 118.618 90)
       (effects (font (size 1.27 1.27)) hide)
     )
@@
       (effects (font (size 1.27 1.27)) (justify left))
     )
-    (property "Footprint" "" (at 180.0352 125.73 0)
+    (property "Footprint" "Capacitor_SMD:C_0805_2012Metric" (at 180.0352 125.73 0)
       (effects (font (size 1.27 1.27)) hide)
     )
@@
       (effects (font (size 1.27 1.27)) (justify left))
     )
-    (property "Footprint" "" (at 194.0052 35.56 0)
+    (property "Footprint" "Capacitor_SMD:C_0805_2012Metric" (at 194.0052 35.56 0)
       (effects (font (size 1.27 1.27)) hide)
     )
@@
       (effects (font (size 1.27 1.27)) (justify left))
     )
-    (property "Footprint" "" (at 53.0352 53.34 0)
+    (property "Footprint" "Capacitor_SMD:C_0402_1005Metric" (at 53.0352 53.34 0)
       (effects (font (size 1.27 1.27)) hide)
     )
@@
       (effects (font (size 1.27 1.27)) (justify left))
     )
-    (property "Footprint" "" (at 21.2852 99.06 0)
+    (property "Footprint" "Capacitor_SMD:C_0805_2012Metric" (at 21.2852 99.06 0)
       (effects (font (size 1.27 1.27)) hide)
     )
@@
       (effects (font (size 1.27 1.27)) (justify left))
     )
-    (property "Footprint" "" (at 201.6252 35.56 0)
+    (property "Footprint" "Capacitor_SMD:C_0402_1005Metric" (at 201.6252 35.56 0)
       (effects (font (size 1.27 1.27)) hide)
     )
@@
       (effects (font (size 1.27 1.27)) (justify left))
     )
-    (property "Footprint" "" (at 56.8452 99.06 0)
+    (property "Footprint" "Capacitor_SMD:C_0402_1005Metric" (at 56.8452 99.06 0)
       (effects (font (size 1.27 1.27)) hide)
     )
@@
       (effects (font (size 1.27 1.27)) (justify left))
     )
-    (property "Footprint" "" (at 74.6252 99.06 0)
+    (property "Footprint" "Capacitor_SMD:C_0402_1005Metric" (at 74.6252 99.06 0)
       (effects (font (size 1.27 1.27)) hide)
     )
@@
       (effects (font (size 1.27 1.27)) (justify left))
     )
-    (property "Footprint" "" (at 30.1752 99.06 0)
+    (property "Footprint" "Capacitor_SMD:C_0805_2012Metric" (at 30.1752 99.06 0)
       (effects (font (size 1.27 1.27)) hide)
     )
@@
       (effects (font (size 1.27 1.27)) (justify left))
     )
-    (property "Footprint" "" (at 61.9252 53.34 0)
+    (property "Footprint" "Capacitor_SMD:C_0402_1005Metric" (at 61.9252 53.34 0)
       (effects (font (size 1.27 1.27)) hide)
     )
@@
       (effects (font (size 1.27 1.27)) (justify left))
     )
-    (property "Footprint" "" (at 35.2552 53.34 0)
+    (property "Footprint" "Capacitor_SMD:C_0805_2012Metric" (at 35.2552 53.34 0)
       (effects (font (size 1.27 1.27)) hide)
     )
@@
       (effects (font (size 1.27 1.27)) (justify left))
     )
-    (property "Footprint" "" (at 187.6552 125.73 0)
+    (property "Footprint" "Capacitor_SMD:C_0402_1005Metric" (at 187.6552 125.73 0)
       (effects (font (size 1.27 1.27)) hide)
     )
@@
       (effects (font (size 1.27 1.27)))
     )
-    (property "Footprint" "" (at 29.21 36.068 90)
+    (property "Footprint" "Inductor_SMD:L_0402_1005Metric" (at 29.21 36.068 90)
       (effects (font (size 1.27 1.27)) hide)
     )
@@
       (effects (font (size 1.27 1.27)) (justify left))
     )
-    (property "Footprint" "" (at 116.5352 35.56 0)
+    (property "Footprint" "Capacitor_SMD:C_0402_1005Metric" (at 116.5352 35.56 0)
       (effects (font (size 1.27 1.27)) hide)
     )
@@
       (effects (font (size 1.27 1.27)) (justify left))
     )
-    (property "Footprint" "" (at 70.8152 53.34 0)
+    (property "Footprint" "Capacitor_SMD:C_0402_1005Metric" (at 70.8152 53.34 0)
       (effects (font (size 1.27 1.27)) hide)
     )
@@
       (effects (font (size 1.27 1.27)) (justify left))
     )
-    (property "Footprint" "" (at 44.1452 53.34 0)
+    (property "Footprint" "Capacitor_SMD:C_0805_2012Metric" (at 44.1452 53.34 0)
       (effects (font (size 1.27 1.27)) hide)
     )
@@
       (effects (font (size 1.27 1.27)) (justify left))
     )
-    (property "Footprint" "" (at 94.9452 76.2 0)
+    (property "Footprint" "Capacitor_SMD:C_0805_2012Metric" (at 94.9452 76.2 0)
       (effects (font (size 1.27 1.27)) hide)
     )
@@
       (effects (font (size 1.27 1.27)) (justify left))
     )
-    (property "Footprint" "" (at 269.24 44.45 0)
+    (property "Footprint" "Connector_PinHeader_2.54mm:PinHeader_1x03_P2.54mm_Vertical" (at 269.24 44.45 0)
       (effects (font (size 1.27 1.27)) hide)
     )
@@
       (effects (font (size 1.27 1.27)))
     )
-    (property "Footprint" "" (at 29.21 25.908 90)
+    (property "Footprint" "Inductor_SMD:L_0402_1005Metric" (at 29.21 25.908 90)
       (effects (font (size 1.27 1.27)) hide)
     )
@@
       (effects (font (size 1.27 1.27)) (justify left))
     )
-    (property "Footprint" "" (at 112.7252 76.2 0)
+    (property "Footprint" "Capacitor_SMD:C_0402_1005Metric" (at 112.7252 76.2 0)
       (effects (font (size 1.27 1.27)) hide)
     )
@@
       (effects (font (size 1.27 1.27)) (justify left))
     )
-    (property "Footprint" "" (at 79.7052 53.34 0)
+    (property "Footprint" "Capacitor_SMD:C_0402_1005Metric" (at 79.7052 53.34 0)
       (effects (font (size 1.27 1.27)) hide)
     )
@@
       (effects (font (size 1.27 1.27)) (justify left))
     )
-    (property "Footprint" "" (at 39.0652 99.06 0)
+    (property "Footprint" "Capacitor_SMD:C_0805_2012Metric" (at 39.0652 99.06 0)
       (effects (font (size 1.27 1.27)) hide)
     )
@@
       (effects (font (size 1.27 1.27)) (justify left))
     )
-    (property "Footprint" "" (at 194.0052 76.2 0)
-      (effects (font (size 1.27 1.27)) hide)
-    )
+    (property "Footprint" "Capacitor_SMD:C_0402_1005Metric" (at 194.0052 76.2 0)
+      (effects (font (size 1.27 1.27)) hide)
+    )
