File: OpenHT-RF/fpga.kicad_sch (KiCad schematic)
At the start: 36 parts, among them J401 Conn_01x06, U401 LIFCL-40-7SG72I

Commit message: Added testpoint
Parts:
- added TP401: TestPoint, symbol Connector:TestPoint
Connections:
- net at U401.43 (PR13B): now also TP401.1
- no-connect marks 27 -> 26
Other:
- moved on the sheet: J401
Changed lines of the file:
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@@
   (no_connect (at 238.76 77.47))
   (no_connect (at 156.21 114.3))
-  (no_connect (at 238.76 31.75))
   (no_connect (at 238.76 67.31))
   (no_connect (at 156.21 129.54))
@@
     (stroke (width 0) (type default))
   )
-  (wire (pts (xy 242.57 115.57) (xy 254 115.57))
+  (wire (pts (xy 248.92 124.46) (xy 260.35 124.46))
     (stroke (width 0) (type default))
   )
@@
     (stroke (width 0) (type default))
   )
+  (wire (pts (xy 238.76 31.75) (xy 248.92 31.75))
+    (stroke (width 0) (type default))
+  )
   (wire (pts (xy 31.75 34.29) (xy 52.07 34.29))
     (stroke (width 0) (type default))
@@
     (stroke (width 0) (type default))
   )
-  (wire (pts (xy 242.57 125.73) (xy 254 125.73))
+  (wire (pts (xy 248.92 134.62) (xy 260.35 134.62))
     (stroke (width 0) (type default))
   )
@@
     (stroke (width 0) (type default))
   )
-  (wire (pts (xy 242.57 118.11) (xy 254 118.11))
+  (wire (pts (xy 248.92 127) (xy 260.35 127))
     (stroke (width 0) (type default))
   )
@@
     (stroke (width 0) (type default))
   )
-  (wire (pts (xy 242.57 123.19) (xy 254 123.19))
+  (wire (pts (xy 248.92 132.08) (xy 260.35 132.08))
     (stroke (width 0) (type default))
   )
@@
     (stroke (width 0) (type default))
   )
-  (wire (pts (xy 242.57 120.65) (xy 254 120.65))
+  (wire (pts (xy 248.92 129.54) (xy 260.35 129.54))
     (stroke (width 0) (type default))
   )
@@
     (stroke (width 0) (type default))
   )
-  (wire (pts (xy 242.57 128.27) (xy 254 128.27))
+  (wire (pts (xy 248.92 137.16) (xy 260.35 137.16))
     (stroke (width 0) (type default))
   )
@@
   )
   (text_box "If pulled high, the SPI pins will be reconfigured as JTAG pins"
-    (at 377.19 -90.17 90) (size 11.43 -19.05)
+    (at 271.78 45.72 90) (size 11.43 19.05)
     (stroke (width 0) (type default))
     (fill (type none))
@@
   )
   (text_box "Configuration port: Slave SPI\n\nLIFCL-40:\nSlave MOSI (SSI)    : PR8B\nSlave MISO (SSO)    : PR10B\nSlave clock (SCLK)  : PR13A\nSlave CS (SCSN)     : PR6B\nProgramN            : PT74B\n\nLIFCL-17:\nSlave MOSI (SSI)    : PR5A\nSlave MISO (SSO)    : PR5B\nSlave clock (SCLK)  : PR9A\nSlave CS (SCSN)     : PR3B\nProgramN            : PT57B\n\nThe physical pin stays the same\n"
-    (at 246.38 67.31 0) (size 35.56 36.83)
+    (at 245.11 73.66 0) (size 35.56 36.83)
     (stroke (width 0) (type default))
     (fill (type none))
     (effects (font (size 1.27 1.27)) (justify left top))
   )
-  (text "Leave VCCADC18\nopen if not used." (at 176.53 115.57 0)
+  (text "Leave VCCADC18\nopen if not used." (at 176.53 113.03 0)
     (effects (font (size 1.27 1.27)) (justify left bottom))
   )
@@
     (effects (font (size 1.27 1.27)) (justify left bottom))
   )
-  (label "TDI{slash}SSI" (at 242.57 120.65 0) (fields_autoplaced)
+  (label "TDI{slash}SSI" (at 248.92 129.54 0) (fields_autoplaced)
     (effects (font (size 1.27 1.27)) (justify left bottom))
   )
@@
     (effects (font (size 1.27 1.27)) (justify right bottom))
   )
-  (label "TDO{slash}SSO" (at 242.57 123.19 0) (fields_autoplaced)
+  (label "TDO{slash}SSO" (at 248.92 132.08 0) (fields_autoplaced)
     (effects (font (size 1.27 1.27)) (justify left bottom))
   )
@@
     (effects (font (size 1.27 1.27)) (justify right bottom))
   )
-  (label "TCK{slash}SCLK" (at 242.57 115.57 0) (fields_autoplaced)
+  (label "TCK{slash}SCLK" (at 248.92 124.46 0) (fields_autoplaced)
     (effects (font (size 1.27 1.27)) (justify left bottom))
   )
@@
     (effects (font (size 1.27 1.27)) (justify right bottom))
   )
-  (label "TMS{slash}SCSN" (at 242.57 118.11 0) (fields_autoplaced)
+  (label "TMS{slash}SCSN" (at 248.92 127 0) (fields_autoplaced)
     (effects (font (size 1.27 1.27)) (justify left bottom))
   )
@@
     )
   )
-  (symbol (lib_id "power:+3.3V") (at 242.57 125.73 90) (unit 1)
-    (in_bom yes) (on_board yes) (dnp no) (fields_autoplaced)
-    (property "Reference" "#PWR0434" (at 246.38 125.73 0)
-      (effects (font (size 1.27 1.27)) hide)
-    )
-    (property "Value" "+3.3V" (at 238.76 126.365 90)
-      (effects (font (size 1.27 1.27)) (justify left))
-    )
-    (property "Footprint" "" (at 242.57 125.73 0)
-      (effects (font (size 1.27 1.27)) hide)
-    )
-    (property "Datasheet" "" (at 242.57 125.73 0)
+  (symbol (lib_id "power:+3.3V") (at 248.92 134.62 90) (unit 1)
+    (in_bom yes) (on_board yes) (dnp no) (fields_autoplaced)
+    (property "Reference" "#PWR0434" (at 252.73 134.62 0)
+      (effects (font (size 1.27 1.27)) hide)
+    )
+    (property "Value" "+3.3V" (at 245.11 135.255 90)
+      (effects (font (size 1.27 1.27)) (justify left))
+    )
+    (property "Footprint" "" (at 248.92 134.62 0)
+      (effects (font (size 1.27 1.27)) hide)
+    )
+    (property "Datasheet" "" (at 248.92 134.62 0)
       (effects (font (size 1.27 1.27)) hide)
     )
@@
     )
   )
-  (symbol (lib_id "Connector_Generic:Conn_01x06") (at 259.08 120.65 0) (unit 1)
-    (in_bom yes) (on_board yes) (dnp no) (fields_autoplaced)
-    (property "Reference" "J401" (at 261.62 121.285 0)
-      (effects (font (size 1.27 1.27)) (justify left))
-    )
-    (property "Value" "Conn_01x06" (at 261.62 123.825 0)
-      (effects (font (size 1.27 1.27)) (justify left))
-    )
-    (property "Footprint" "Connector_PinSocket_2.54mm:PinSocket_1x06_P2.54mm_Horizontal" (at 259.08 120.65 0)
-      (effects (font (size 1.27 1.27)) hide)
-    )
-    (property "Datasheet" "~" (at 259.08 120.65 0)
+  (symbol (lib_id "Connector_Generic:Conn_01x06") (at 265.43 129.54 0) (unit 1)
+    (in_bom yes) (on_board yes) (dnp no) (fields_autoplaced)
+    (property "Reference" "J401" (at 267.97 130.175 0)
+      (effects (font (size 1.27 1.27)) (justify left))
+    )
+    (property "Value" "Conn_01x06" (at 267.97 132.715 0)
+      (effects (font (size 1.27 1.27)) (justify left))
+    )
+    (property "Footprint" "Connector_PinSocket_2.54mm:PinSocket_1x06_P2.54mm_Horizontal" (at 265.43 129.54 0)
+      (effects (font (size 1.27 1.27)) hide)
+    )
+    (property "Datasheet" "~" (at 265.43 129.54 0)
       (effects (font (size 1.27 1.27)) hide)
     )
@@
     )
   )
+  (symbol (lib_id "Connector:TestPoint") (at 248.92 31.75 270) (unit 1)
+    (in_bom yes) (on_board yes) (dnp no)
+    (property "Reference" "TP401" (at 254 31.75 90)
+      (effects (font (size 1.27 1.27)) (justify left))
+    )
+    (property "Value" "TestPoint" (at 254 33.655 90)
+      (effects (font (size 1.27 1.27)) (justify left) hide)
+    )
+    (property "Footprint" "" (at 248.92 36.83 0)
+      (effects (font (size 1.27 1.27)) hide)
+    )
+    (property "Datasheet" "~" (at 248.92 36.83 0)
+      (effects (font (size 1.27 1.27)) hide)
+    )
+    (pin "1")
+    (instances
+      (project "OpenHT-RF"
+        (path "/3c300b59-23ec-47f8-bb91-29ca34130bcf/2f3751e7-d003-4d36-b778-c7fcad1ff611"
+          (reference "TP401") (unit 1)
+        )
+      )
+    )
+  )
   (symbol (lib_id "power:GND") (at 200.66 35.56 0) (unit 1)
     (in_bom yes) (on_board yes) (dnp no) (fields_autoplaced)
@@
     )
   )
-  (symbol (lib_id "power:GND") (at 242.57 128.27 0) (unit 1)
-    (in_bom yes) (on_board yes) (dnp no) (fields_autoplaced)
-    (property "Reference" "#PWR0435" (at 242.57 134.62 0)
-      (effects (font (size 1.27 1.27)) hide)
-    )
-    (property "Value" "GND" (at 242.57 133.35 0)
-      (effects (font (size 1.27 1.27)))
-    )
-    (property "Footprint" "" (at 242.57 128.27 0)
-      (effects (font (size 1.27 1.27)) hide)
-    )
-    (property "Datasheet" "" (at 242.57 128.27 0)
-      (effects (font (size 1.27 1.27)) hide)
-    )
+  (symbol (lib_id "power:GND") (at 248.92 137.16 0) (unit 1)
+    (in_bom yes) (on_board yes) (dnp no) (fields_autoplaced)
+    (property "Reference" "#PWR0435" (at 248.92 143.51 0)
+      (effects (font (size 1.27 1.27)) hide)
+    )
+    (property "Value" "GND" (at 248.92 142.24 0)
+      (effects (font (size 1.27 1.27)))
+    )
+    (property "Footprint" "" (at 248.92 137.16 0)
+      (effects (font (size 1.27 1.27)) hide)
+    )
+    (property "Datasheet" "" (at 248.92 137.16 0)
+      (effects (font (size 1.27 1.27)) hide)
+    )

Commit message: Selected footprint
Parts:
- TP401: footprint (none) -> TestPoint:TestPoint_Loop_D2.50mm_Drill1.0mm
Changed lines of the file:
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@@
       (effects (font (size 1.27 1.27)) (justify left) hide)
     )
-    (property "Footprint" "" (at 248.92 36.83 0)
+    (property "Footprint" "TestPoint:TestPoint_Loop_D2.50mm_Drill1.0mm" (at 248.92 36.83 0)
       (effects (font (size 1.27 1.27)) hide)
     )
