File: OpenHT-RF/fpga.kicad_sch (KiCad schematic)
At the start: 37 parts, among them J401 Conn_01x06, U401 LIFCL-40-7SG72I

Commit message: Fixed 3.3V power symbol
Use 3V3 everywhere instead of 3.3
Connections:
- net +3.3V is gone; now on net +3V3: J401.5 (Pin_5)
Changed lines of the file:
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@@
-    )
-  )
-  (symbol (lib_id "power:+3.3V") (at 248.92 134.62 90) (unit 1)
-    (in_bom yes) (on_board yes) (dnp no) (fields_autoplaced)
-    (property "Reference" "#PWR0434" (at 252.73 134.62 0)
-      (effects (font (size 1.27 1.27)) hide)
-    )
-    (property "Value" "+3.3V" (at 245.11 135.255 90)
-      (effects (font (size 1.27 1.27)) (justify left))
-    )
-    (property "Footprint" "" (at 248.92 134.62 0)
-      (effects (font (size 1.27 1.27)) hide)
-    )
-    (property "Datasheet" "" (at 248.92 134.62 0)
-      (effects (font (size 1.27 1.27)) hide)
-    )
-    (pin "1")
-    (instances
-      (project "OpenHT-RF"
-        (path "/3c300b59-23ec-47f8-bb91-29ca34130bcf/2f3751e7-d003-4d36-b778-c7fcad1ff611"
-          (reference "#PWR0434") (unit 1)
-        )
-      )
     )
   )
@@
         )
       )
+    )
+  )
+  (symbol (lib_id "power:+3V3") (at 248.92 134.62 90) (unit 1)
+    (in_bom yes) (on_board yes) (dnp no)
+    (property "Reference" "#PWR0434" (at 252.73 134.62 0)
+      (effects (font (size 1.27 1.27)) hide)
+    )
+    (property "Value" "+3V3" (at 245.11 134.62 90)
+      (effects (font (size 1.27 1.27)) (justify left))
+    )
+    (property "Footprint" "" (at 248.92 134.62 0)
+      (effects (font (size 1.27 1.27)) hide)
+    )
+    (property "Datasheet" "" (at 248.92 134.62 0)
+      (effects (font (size 1.27 1.27)) hide)
+    )
+    (pin "1")
+    (instances
+      (project "OpenHT-RF"
+        (path "/3c300b59-23ec-47f8-bb91-29ca34130bcf/2f3751e7-d003-4d36-b778-c7fcad1ff611"
+          (reference "#PWR0434") (unit 1)
+        )
+      )

Commit message: Updated QFN footprints
Parts:
- U401: footprint M17_QFN:QFN-72-1EP_10x10mm_P0.5mm_EP6.2x6.2mm -> M17_QFN:QFN-72-1EP_10x10mm_P0.5mm_EP6.2x6.2mm_ThermalVias
Changed lines of the file:
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@@
       (effects (font (size 1.27 1.27)))
     )
-    (property "Footprint" "M17_QFN:QFN-72-1EP_10x10mm_P0.5mm_EP6.2x6.2mm" (at 215.9 46.99 0)
+    (property "Footprint" "M17_QFN:QFN-72-1EP_10x10mm_P0.5mm_EP6.2x6.2mm_ThermalVias" (at 215.9 46.99 0)
       (effects (font (size 1.27 1.27)) hide)
     )
@@
       (effects (font (size 1.27 1.27)))
     )
-    (property "Footprint" "M17_QFN:QFN-72-1EP_10x10mm_P0.5mm_EP6.2x6.2mm" (at 132.08 6.35 0)
+    (property "Footprint" "M17_QFN:QFN-72-1EP_10x10mm_P0.5mm_EP6.2x6.2mm_ThermalVias" (at 132.08 6.35 0)
       (effects (font (size 1.27 1.27)) hide)
     )
@@
       (effects (font (size 1.27 1.27)))
     )
-    (property "Footprint" "M17_QFN:QFN-72-1EP_10x10mm_P0.5mm_EP6.2x6.2mm" (at 130.81 88.9 0)
+    (property "Footprint" "M17_QFN:QFN-72-1EP_10x10mm_P0.5mm_EP6.2x6.2mm_ThermalVias" (at 130.81 88.9 0)
       (effects (font (size 1.27 1.27)) hide)
     )
@@
       (effects (font (size 1.27 1.27)))
     )
-    (property "Footprint" "M17_QFN:QFN-72-1EP_10x10mm_P0.5mm_EP6.2x6.2mm" (at 217.17 86.36 0)
+    (property "Footprint" "M17_QFN:QFN-72-1EP_10x10mm_P0.5mm_EP6.2x6.2mm_ThermalVias" (at 217.17 86.36 0)
       (effects (font (size 1.27 1.27)) hide)
     )
@@
       (effects (font (size 1.27 1.27)))
     )
-    (property "Footprint" "M17_QFN:QFN-72-1EP_10x10mm_P0.5mm_EP6.2x6.2mm" (at 215.9 6.35 0)
+    (property "Footprint" "M17_QFN:QFN-72-1EP_10x10mm_P0.5mm_EP6.2x6.2mm_ThermalVias" (at 215.9 6.35 0)
       (effects (font (size 1.27 1.27)) hide)
     )
@@
       (effects (font (size 1.27 1.27)))
     )
-    (property "Footprint" "M17_QFN:QFN-72-1EP_10x10mm_P0.5mm_EP6.2x6.2mm" (at 132.08 46.99 0)
-      (effects (font (size 1.27 1.27)) hide)
-    )
+    (property "Footprint" "M17_QFN:QFN-72-1EP_10x10mm_P0.5mm_EP6.2x6.2mm_ThermalVias" (at 132.08 46.99 0)
+      (effects (font (size 1.27 1.27)) hide)
+    )

Commit message: Swapped LVDS pairs order
Connections:
- net LVDS_RX09_N: now also U401.28 (PB68B); no longer U401.25 (PB58B)
- net LVDS_RX09_P: now also U401.27 (PB68A); no longer U401.24 (PB58A)
- net LVDS_RX24_N: now also U401.23 (PB54B); no longer U401.28 (PB68B)
- net LVDS_RX24_P: now also U401.22 (PB54A); no longer U401.27 (PB68A)
- net LVDS_RXCLK_N: now also U401.25 (PB58B); no longer U401.23 (PB54B)
- net LVDS_RXCLK_P: now also U401.24 (PB58A); no longer U401.22 (PB54A)
- net LVDS_TXCLK_N: now also U401.34 (PB74B); no longer U401.31 (PB72B)
- net LVDS_TXCLK_P: now also U401.33 (PB74A); no longer U401.30 (PB72A)
- net LVDS_TX_N: now also U401.31 (PB72B); no longer U401.34 (PB74B)
- net LVDS_TX_P: now also U401.30 (PB72A); no longer U401.33 (PB74A)
Changed lines of the file:
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@@
     (effects (font (size 1.27 1.27)) (justify left))
   )
-  (hierarchical_label "LVDS_RX24_P" (shape input) (at 165.1 77.47 0) (fields_autoplaced)
+  (hierarchical_label "LVDS_RX24_N" (shape input) (at 165.1 69.85 0) (fields_autoplaced)
+    (effects (font (size 1.27 1.27)) (justify left))
+  )
+  (hierarchical_label "LVDS_RXCLK_N" (shape input) (at 165.1 74.93 0) (fields_autoplaced)
     (effects (font (size 1.27 1.27)) (justify left))
   )
@@
     (effects (font (size 1.27 1.27)) (justify left))
   )
-  (hierarchical_label "LVDS_RX24_N" (shape input) (at 165.1 80.01 0) (fields_autoplaced)
+  (hierarchical_label "LVDS_RX09_N" (shape input) (at 165.1 80.01 0) (fields_autoplaced)
     (effects (font (size 1.27 1.27)) (justify left))
   )
-  (hierarchical_label "LVDS_RXCLK_P" (shape input) (at 165.1 67.31 0) (fields_autoplaced)
-    (effects (font (size 1.27 1.27)) (justify left))
-  )
-  (hierarchical_label "LVDS_TXCLK_N" (shape output) (at 165.1 85.09 0) (fields_autoplaced)
+  (hierarchical_label "LVDS_TXCLK_N" (shape output) (at 165.1 90.17 0) (fields_autoplaced)
     (effects (font (size 1.27 1.27)) (justify left))
   )
@@
     (effects (font (size 1.27 1.27)) (justify left))
   )
+  (hierarchical_label "LVDS_RX24_P" (shape input) (at 165.1 67.31 0) (fields_autoplaced)
+    (effects (font (size 1.27 1.27)) (justify left))
+  )
   (hierarchical_label "IO3" (shape bidirectional) (at 162.56 29.21 0) (fields_autoplaced)
     (effects (font (size 1.27 1.27)) (justify left))
   )
-  (hierarchical_label "LVDS_TX_N" (shape output) (at 165.1 90.17 0) (fields_autoplaced)
+  (hierarchical_label "LVDS_TX_N" (shape output) (at 165.1 85.09 0) (fields_autoplaced)
     (effects (font (size 1.27 1.27)) (justify left))
   )
-  (hierarchical_label "LVDS_TX_P" (shape output) (at 165.1 87.63 0) (fields_autoplaced)
+  (hierarchical_label "LVDS_TX_P" (shape output) (at 165.1 82.55 0) (fields_autoplaced)
     (effects (font (size 1.27 1.27)) (justify left))
   )
@@
     (effects (font (size 1.27 1.27)) (justify left))
   )
-  (hierarchical_label "PROGRAMN" (shape input) (at 162.56 46.99 0) (fields_autoplaced)
+  (hierarchical_label "LVDS_RXCLK_P" (shape input) (at 165.1 72.39 0) (fields_autoplaced)
     (effects (font (size 1.27 1.27)) (justify left))
   )
-  (hierarchical_label "LVDS_RX09_N" (shape input) (at 165.1 74.93 0) (fields_autoplaced)
-    (effects (font (size 1.27 1.27)) (justify left))
-  )
-  (hierarchical_label "LVDS_RX09_P" (shape input) (at 165.1 72.39 0) (fields_autoplaced)
+  (hierarchical_label "PROGRAMN" (shape input) (at 162.56 46.99 0) (fields_autoplaced)
     (effects (font (size 1.27 1.27)) (justify left))
   )
@@
     (effects (font (size 1.27 1.27)) (justify left))
   )
-  (hierarchical_label "LVDS_TXCLK_P" (shape output) (at 165.1 82.55 0) (fields_autoplaced)
+  (hierarchical_label "LVDS_TXCLK_P" (shape output) (at 165.1 87.63 0) (fields_autoplaced)
     (effects (font (size 1.27 1.27)) (justify left))
   )
-  (hierarchical_label "LVDS_RXCLK_N" (shape input) (at 165.1 69.85 0) (fields_autoplaced)
+  (hierarchical_label "LVDS_RX09_P" (shape input) (at 165.1 77.47 0) (fields_autoplaced)
     (effects (font (size 1.27 1.27)) (justify left))
   )

Commit message: Connectors adjustments
Parts:
- J401: now not fitted
Changed lines of the file:
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@@
   )
   (symbol (lib_id "Connector_Generic:Conn_01x06") (at 265.43 129.54 0) (unit 1)
-    (in_bom yes) (on_board yes) (dnp no) (fields_autoplaced)
+    (in_bom yes) (on_board yes) (dnp yes) (fields_autoplaced)
     (property "Reference" "J401" (at 267.97 130.175 0)
       (effects (font (size 1.27 1.27)) (justify left))

Commit message: Rearanged IOs
Connections:
- net IO0: now also U401.55 (PT80B); no longer U401.42 (PR11A/SDA)
- net IO1: now also U401.53 (PT82B/MCSNO); no longer U401.44 (PR11B/SCL)
- net IO2: now also U401.52 (PT82A); no longer U401.51 (PT80A/MISO)
- net IO3: now also U401.51 (PT80A/MISO); no longer U401.52 (PT82A)
- net IO4: now also U401.44 (PR11B/SCL); no longer U401.53 (PT82B/MCSNO)
- net IO5: now also U401.42 (PR11A/SDA); no longer U401.55 (PT80B)
Changed lines of the file:
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@@
     (effects (font (size 1.27 1.27)) (justify left))
   )
-  (hierarchical_label "IO5" (shape bidirectional) (at 162.56 34.29 0) (fields_autoplaced)
+  (hierarchical_label "IO0" (shape bidirectional) (at 162.56 34.29 0) (fields_autoplaced)
     (effects (font (size 1.27 1.27)) (justify left))
   )
@@
     (effects (font (size 1.27 1.27)) (justify left))
   )
-  (hierarchical_label "IO3" (shape bidirectional) (at 162.56 29.21 0) (fields_autoplaced)
+  (hierarchical_label "IO3" (shape bidirectional) (at 162.56 26.67 0) (fields_autoplaced)
     (effects (font (size 1.27 1.27)) (justify left))
   )
@@
     (effects (font (size 1.27 1.27)) (justify left))
   )
-  (hierarchical_label "IO0" (shape bidirectional) (at 251.46 29.21 0) (fields_autoplaced)
+  (hierarchical_label "IO5" (shape bidirectional) (at 251.46 29.21 0) (fields_autoplaced)
     (effects (font (size 1.27 1.27)) (justify left))
   )
-  (hierarchical_label "IO2" (shape bidirectional) (at 162.56 26.67 0) (fields_autoplaced)
+  (hierarchical_label "IO2" (shape bidirectional) (at 162.56 29.21 0) (fields_autoplaced)
     (effects (font (size 1.27 1.27)) (justify left))
   )
@@
     (effects (font (size 1.27 1.27)) (justify left))
   )
-  (hierarchical_label "IO1" (shape bidirectional) (at 251.46 34.29 0) (fields_autoplaced)
+  (hierarchical_label "IO4" (shape bidirectional) (at 251.46 34.29 0) (fields_autoplaced)
     (effects (font (size 1.27 1.27)) (justify left))
   )
@@
     (effects (font (size 1.27 1.27)) (justify left))
   )
-  (hierarchical_label "IO4" (shape bidirectional) (at 162.56 31.75 0) (fields_autoplaced)
+  (hierarchical_label "IO1" (shape bidirectional) (at 162.56 31.75 0) (fields_autoplaced)
     (effects (font (size 1.27 1.27)) (justify left))
   )

Commit message: [WIP] Layout
Flipped the content upside down for the SMA connector. Reorganized GPIOs. RF routing started.
Parts:
- added R402: 100R, Resistor_SMD:R_0402_1005Metric, symbol Device:R
Connections:
- net IO0: now also U401.44 (PR11B/SCL); no longer U401.55 (PT80B)
- net IO1: now also U401.42 (PR11A/SDA); no longer U401.53 (PT82B/MCSNO)
- net IO2: now also U401.51 (PT80A/MISO); no longer U401.52 (PT82A)
- net IO3: now also U401.52 (PT82A); no longer U401.51 (PT80A/MISO)
- net IO4: now also U401.53 (PT82B/MCSNO); no longer U401.44 (PR11B/SCL)
- net IO5: now also U401.55 (PT80B); no longer U401.42 (PR11A/SDA)
- net S_SPI_MISO: now also R402.2; no longer J401.4 (Pin_4), U401.45 (PR10B/TDO/SSO)
- new net TDO/SSO: J401.4 (Pin_4), R402.1, U401.45 (PR10B/TDO/SSO)
Other:
- moved on the sheet: JP401, R401
