File: OpenHT-RF/OpenHT-RF.kicad_sch (KiCad schematic)
At the start: 4 parts, among them J5 Conn_01x08, J6 Conn_01x06, J7 Conn_01x10, J8 Conn_01x08

Commit message: Add files via upload
Parts:
- removed J5, J8: Conn_01x08, symbol Connector_Generic:Conn_01x08
- removed J6: Conn_01x06, symbol Connector_Generic:Conn_01x06
- removed J7: Conn_01x10, symbol Connector_Generic:Conn_01x10
Other:
- added sheet Connectors (conn.kicad_sch)
- added sheet FPGA (fpga.kicad_sch)
- added sheet Power supply (pwr.kicad_sch)
- added sheet RF (rf.kicad_sch)
- company: (none) -> M17 Project
- title: (none) -> OpenHT - open source SDR handheld
Changed lines of the file:
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@@
 (kicad_sch (version 20230121) (generator eeschema)
   (paper "A4")
-  (symbol (lib_id "Connector_Generic:Conn_01x08") (at 138.43 102.87 0) (mirror y) (unit 1)
-    (in_bom yes) (on_board yes) (dnp no)
-    (property "Reference" "J8" (at 138.43 92.71 0)
-      (effects (font (size 1.27 1.27)))
+  (title_block
+    (title "OpenHT - open source SDR handheld")
+    (date "2023-02-17")
+    (rev "A")
+    (company "M17 Project")
+    (comment 1 "Authors: Wojciech SP5WWP, Leo Hofer")
+  )
+  (sheet (at 25.4 25.4) (size 12.7 12.7) (fields_autoplaced)
+    (stroke (width 0.1524) (type solid))
+    (fill (color 0 0 0 0.0000))
+    (property "Sheetname" "Power supply" (at 25.4 24.6884 0)
+      (effects (font (size 1.27 1.27)) (justify left bottom))
     )
-    (property "Value" "Conn_01x08" (at 135.89 105.41 90)
-      (effects (font (size 1.27 1.27)))
+    (property "Sheetfile" "pwr.kicad_sch" (at 25.4 38.6846 0)
+      (effects (font (size 1.27 1.27)) (justify left top))
     )
-    (property "Footprint" "" (at 138.43 102.87 0)
-      (effects (font (size 1.27 1.27)) hide)
-    )
-    (property "Datasheet" "~" (at 138.43 102.87 0)
-      (effects (font (size 1.27 1.27)) hide)
-    )
-    (pin "1")
-    (pin "2")
-    (pin "3")
-    (pin "4")
-    (pin "5")
-    (pin "6")
-    (pin "7")
-    (pin "8")
     (instances
       (project "OpenHT-RF"
-        (path "/3c300b59-23ec-47f8-bb91-29ca34130bcf"
-          (reference "J8") (unit 1)
-        )
+        (path "/3c300b59-23ec-47f8-bb91-29ca34130bcf" (page "2"))
       )
     )
   )
-  (symbol (lib_id "Connector_Generic:Conn_01x10") (at 138.43 73.66 0) (mirror y) (unit 1)
-    (in_bom yes) (on_board yes) (dnp no)
-    (property "Reference" "J7" (at 139.7 60.96 0)
-      (effects (font (size 1.27 1.27)) (justify left))
+  (sheet (at 50.8 25.4) (size 12.7 12.7) (fields_autoplaced)
+    (stroke (width 0.1524) (type solid))
+    (fill (color 0 0 0 0.0000))
+    (property "Sheetname" "Connectors" (at 50.8 24.6884 0)
+      (effects (font (size 1.27 1.27)) (justify left bottom))
     )
-    (property "Value" "Conn_01x10" (at 135.89 80.01 90)
-      (effects (font (size 1.27 1.27)) (justify left))
+    (property "Sheetfile" "conn.kicad_sch" (at 50.8 38.6846 0)
+      (effects (font (size 1.27 1.27)) (justify left top))
     )
-    (property "Footprint" "" (at 138.43 73.66 0)
-      (effects (font (size 1.27 1.27)) hide)
-    )
-    (property "Datasheet" "~" (at 138.43 73.66 0)
-      (effects (font (size 1.27 1.27)) hide)
-    )
-    (pin "1")
-    (pin "10")
-    (pin "2")
-    (pin "3")
-    (pin "4")
-    (pin "5")
-    (pin "6")
-    (pin "7")
-    (pin "8")
-    (pin "9")
     (instances
       (project "OpenHT-RF"
-        (path "/3c300b59-23ec-47f8-bb91-29ca34130bcf"
-          (reference "J7") (unit 1)
-        )
+        (path "/3c300b59-23ec-47f8-bb91-29ca34130bcf" (page "3"))
       )
     )
   )
-  (symbol (lib_id "Connector_Generic:Conn_01x08") (at 109.22 81.28 0) (unit 1)
-    (in_bom yes) (on_board yes) (dnp no)
-    (property "Reference" "J5" (at 109.22 71.12 0)
-      (effects (font (size 1.27 1.27)))
+  (sheet (at 76.2 25.4) (size 12.7 12.7) (fields_autoplaced)
+    (stroke (width 0.1524) (type solid))
+    (fill (color 0 0 0 0.0000))
+    (property "Sheetname" "FPGA" (at 76.2 24.6884 0)
+      (effects (font (size 1.27 1.27)) (justify left bottom))
     )
-    (property "Value" "Conn_01x08" (at 111.76 82.55 90)
-      (effects (font (size 1.27 1.27)))
+    (property "Sheetfile" "fpga.kicad_sch" (at 76.2 38.6846 0)
+      (effects (font (size 1.27 1.27)) (justify left top))
     )
-    (property "Footprint" "" (at 109.22 81.28 0)
-      (effects (font (size 1.27 1.27)) hide)
-    )
-    (property "Datasheet" "~" (at 109.22 81.28 0)
-      (effects (font (size 1.27 1.27)) hide)
-    )
-    (pin "1")
-    (pin "2")
-    (pin "3")
-    (pin "4")
-    (pin "5")
-    (pin "6")
-    (pin "7")
-    (pin "8")
     (instances
       (project "OpenHT-RF"
-        (path "/3c300b59-23ec-47f8-bb91-29ca34130bcf"
-          (reference "J5") (unit 1)
-        )
+        (path "/3c300b59-23ec-47f8-bb91-29ca34130bcf" (page "4"))
       )
     )
   )
-  (symbol (lib_id "Connector_Generic:Conn_01x06") (at 109.22 105.41 0) (unit 1)
-    (in_bom yes) (on_board yes) (dnp no)
-    (property "Reference" "J6" (at 109.22 97.79 0)
-      (effects (font (size 1.27 1.27)))
+  (sheet (at 101.6 25.4) (size 12.7 12.7) (fields_autoplaced)
+    (stroke (width 0.1524) (type solid))
+    (fill (color 0 0 0 0.0000))
+    (property "Sheetname" "RF" (at 101.6 24.6884 0)
+      (effects (font (size 1.27 1.27)) (justify left bottom))
     )
-    (property "Value" "Conn_01x06" (at 111.76 106.68 90)
-      (effects (font (size 1.27 1.27)))
+    (property "Sheetfile" "rf.kicad_sch" (at 101.6 38.6846 0)
+      (effects (font (size 1.27 1.27)) (justify left top))
     )
-    (property "Footprint" "" (at 109.22 105.41 0)
-      (effects (font (size 1.27 1.27)) hide)
-    )
-    (property "Datasheet" "~" (at 109.22 105.41 0)
-      (effects (font (size 1.27 1.27)) hide)
-    )
-    (pin "1")
-    (pin "2")
-    (pin "3")
-    (pin "4")
-    (pin "5")
-    (pin "6")
     (instances
       (project "OpenHT-RF"
-        (path "/3c300b59-23ec-47f8-bb91-29ca34130bcf"
-          (reference "J6") (unit 1)
-        )
+        (path "/3c300b59-23ec-47f8-bb91-29ca34130bcf" (page "5"))
       )
     )

Commit message: FPGA diagram [WIP]
Other:
- sheet FPGA ports: added CLK_IN, LVDS_RX0_N, LVDS_RX0_P, LVDS_RX1_N, LVDS_RX1_P, LVDS_RXCLK_N, LVDS_RXCLK_P, LVDS_TX0_N, LVDS_TX0_P, LVDS_TXCLK_N, LVDS_TXCLK_P, M_SPI_CLK, M_SPI_MISO, M_SPI_MOSI, M_SPI_SS, PROGRAMN, S_SPI_CLK, S_SPI_CS, S_SPI_MISO, S_SPI_MOSI; removed none
Changed lines of the file:
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@@
     (rev "A")
     (company "M17 Project")
-    (comment 1 "Authors: Wojciech SP5WWP, Leo Hofer")
+    (comment 1 "Authors: Wojciech SP5WWP, Leo Hofer, Morgan ON4MOD")
   )
   (sheet (at 25.4 25.4) (size 12.7 12.7) (fields_autoplaced)
@@
     )
   )
-  (sheet (at 76.2 25.4) (size 12.7 12.7) (fields_autoplaced)
+  (sheet (at 114.3 71.12) (size 38.1 48.26) (fields_autoplaced)
     (stroke (width 0.1524) (type solid))
     (fill (color 0 0 0 0.0000))
-    (property "Sheetname" "FPGA" (at 76.2 24.6884 0)
+    (property "Sheetname" "FPGA" (at 114.3 70.4084 0)
       (effects (font (size 1.27 1.27)) (justify left bottom))
     )
-    (property "Sheetfile" "fpga.kicad_sch" (at 76.2 38.6846 0)
+    (property "Sheetfile" "fpga.kicad_sch" (at 114.3 119.9646 0)
       (effects (font (size 1.27 1.27)) (justify left top))
     )
+    (pin "LVDS_TX0_N" input (at 152.4 90.17 0)
+      (effects (font (size 1.27 1.27)) (justify right))
+    )
+    (pin "LVDS_TXCLK_N" input (at 152.4 96.52 0)
+      (effects (font (size 1.27 1.27)) (justify right))
+    )
+    (pin "LVDS_TX0_P" input (at 152.4 87.63 0)
+      (effects (font (size 1.27 1.27)) (justify right))
+    )
+    (pin "LVDS_TXCLK_P" input (at 152.4 93.98 0)
+      (effects (font (size 1.27 1.27)) (justify right))
+    )
+    (pin "LVDS_RX1_P" input (at 114.3 87.63 180)
+      (effects (font (size 1.27 1.27)) (justify left))
+    )
+    (pin "LVDS_RX0_N" input (at 114.3 83.82 180)
+      (effects (font (size 1.27 1.27)) (justify left))
+    )
+    (pin "LVDS_RX1_N" input (at 114.3 90.17 180)
+      (effects (font (size 1.27 1.27)) (justify left))
+    )
+    (pin "LVDS_RXCLK_N" input (at 114.3 96.52 180)
+      (effects (font (size 1.27 1.27)) (justify left))
+    )
+    (pin "LVDS_RXCLK_P" input (at 114.3 93.98 180)
+      (effects (font (size 1.27 1.27)) (justify left))
+    )
+    (pin "LVDS_RX0_P" input (at 114.3 81.28 180)
+      (effects (font (size 1.27 1.27)) (justify left))
+    )
+    (pin "M_SPI_SS" input (at 152.4 116.84 0)
+      (effects (font (size 1.27 1.27)) (justify right))
+    )
+    (pin "M_SPI_MISO" input (at 114.3 114.3 180)
+      (effects (font (size 1.27 1.27)) (justify left))
+    )
+    (pin "M_SPI_CLK" input (at 152.4 114.3 0)
+      (effects (font (size 1.27 1.27)) (justify right))
+    )
+    (pin "M_SPI_MOSI" input (at 152.4 111.76 0)
+      (effects (font (size 1.27 1.27)) (justify right))
+    )
+    (pin "S_SPI_MOSI" input (at 114.3 101.6 180)
+      (effects (font (size 1.27 1.27)) (justify left))
+    )
+    (pin "S_SPI_CS" input (at 114.3 106.68 180)
+      (effects (font (size 1.27 1.27)) (justify left))
+    )
+    (pin "S_SPI_MISO" input (at 152.4 104.14 0)
+      (effects (font (size 1.27 1.27)) (justify right))
+    )
+    (pin "S_SPI_CLK" input (at 114.3 104.14 180)
+      (effects (font (size 1.27 1.27)) (justify left))
+    )
+    (pin "PROGRAMN" input (at 114.3 76.2 180)
+      (effects (font (size 1.27 1.27)) (justify left))
+    )
+    (pin "CLK_IN" input (at 114.3 73.66 180)
+      (effects (font (size 1.27 1.27)) (justify left))
+    )
     (instances

Commit message: Updated FPGA, RF and connectors sheets [WIP]
Other:
- sheet Connectors ports: added SPI_MISO, SPI_MOSI, SPI_NSS1, SPI_NSS2, SPI_SCK, SPK_N, SPK_P; removed none
- sheet FPGA ports: added LVDS_RX09_N, LVDS_RX09_P, LVDS_RX24_N, LVDS_RX24_P, LVDS_TX_N, LVDS_TX_P; removed LVDS_RX0_N, LVDS_RX0_P, LVDS_RX1_N, LVDS_RX1_P, LVDS_TX0_N, LVDS_TX0_P, M_SPI_CLK, M_SPI_MISO, M_SPI_MOSI, M_SPI_SS
- sheet RF ports: added AT86RF215_IRQ, LVDS_RX09_N, LVDS_RX09_P, LVDS_RX24_N, LVDS_RX24_P, LVDS_RXCLK_N, LVDS_RXCLK_P, LVDS_TXCLK_N, LVDS_TXCLK_P, LVDS_TX_N, LVDS_TX_P, S_SPI_MISO, S_SPI_MOSI, S_SPI_SCLK, S_SPI_SELN; removed none

Commit message: Updated FPGA, RF and connectors sheets [WIP]
Other:
- sheet Connectors ports: added DONE, INITN, IO0, IO1, IO2, IO3, IO4, IO5, IO6, IO7, IRQ_AT86RF215, PROGRAMN; removed none
- sheet FPGA ports: added DONE, INITN, IO0, IO1, IO2, IO3, IO4, IO5, IO6, IO7; removed none
- sheet RF ports: added CLK_OUT; removed none

Commit message: Updated RF schematic
Other:
- sheet RF ports: added SW_CTL1, SW_CTL2, ~{RESET}; removed none
Changed lines of the file:
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@@
     (stroke (width 0) (type default))
   )
-  (wire (pts (xy 167.64 78.74) (xy 167.64 91.44))
+  (wire (pts (xy 167.64 91.44) (xy 167.64 78.74))
     (stroke (width 0) (type default))
   )
@@
     )
   )
-  (sheet (at 185.42 86.36) (size 24.13 53.34) (fields_autoplaced)
+  (sheet (at 185.42 76.2) (size 24.13 63.5) (fields_autoplaced)
     (stroke (width 0.1524) (type solid))
     (fill (color 0 0 0 0.0000))
-    (property "Sheetname" "RF" (at 185.42 85.6484 0)
+    (property "Sheetname" "RF" (at 185.42 75.4884 0)
       (effects (font (size 1.27 1.27)) (justify left bottom))
     )
@@
       (effects (font (size 1.27 1.27)) (justify left))
     )
+    (pin "SW_CTL1" input (at 185.42 87.63 180)
+      (effects (font (size 1.27 1.27)) (justify left))
+    )
+    (pin "SW_CTL2" input (at 185.42 83.82 180)
+      (effects (font (size 1.27 1.27)) (justify left))
+    )
+    (pin "~{RESET}" bidirectional (at 185.42 80.01 180)
+      (effects (font (size 1.27 1.27)) (justify left))
+    )

Commit message: Added pushbutton controller for main power
Other:
- sheet Power supply ports: added LOW_P, MAIN_KILL, PB_INT, PGOOD; removed none
Changed lines of the file:
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@@
     )
   )
-  (sheet (at 138.43 38.1) (size 12.7 12.7) (fields_autoplaced)
+  (sheet (at 134.62 53.34) (size 19.05 15.24) (fields_autoplaced)
     (stroke (width 0.1524) (type solid))
     (fill (color 0 0 0 0.0000))
-    (property "Sheetname" "Power supply" (at 138.43 37.3884 0)
+    (property "Sheetname" "Power supply" (at 134.62 52.6284 0)
       (effects (font (size 1.27 1.27)) (justify left bottom))
     )
-    (property "Sheetfile" "pwr.kicad_sch" (at 138.43 51.3846 0)
+    (property "Sheetfile" "pwr.kicad_sch" (at 134.62 69.1646 0)
       (effects (font (size 1.27 1.27)) (justify left top))
     )
+    (pin "LOW_P" output (at 134.62 57.15 180)
+      (effects (font (size 1.27 1.27)) (justify left))
+    )
+    (pin "PGOOD" input (at 134.62 59.69 180)
+      (effects (font (size 1.27 1.27)) (justify left))
+    )
+    (pin "PB_INT" input (at 134.62 62.23 180)
+      (effects (font (size 1.27 1.27)) (justify left))
+    )
+    (pin "MAIN_KILL" input (at 134.62 64.77 180)
+      (effects (font (size 1.27 1.27)) (justify left))
+    )
     (instances

Commit message: [WIP]Updating power suply diagram
Changing buck converter IC
Other:
- sheet Power supply ports: added PWR_RESET; removed LOW_P
Changed lines of the file:
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@@
       (effects (font (size 1.27 1.27)) (justify left top))
-    )
-    (pin "LOW_P" output (at 134.62 57.15 180)
-      (effects (font (size 1.27 1.27)) (justify left))
     )
     (pin "PGOOD" input (at 134.62 59.69 180)
@@
       (effects (font (size 1.27 1.27)) (justify left))
     )
-    (pin "MAIN_KILL" input (at 134.62 64.77 180)
+    (pin "MAIN_KILL" output (at 134.62 64.77 180)
       (effects (font (size 1.27 1.27)) (justify left))
     )
+    (pin "PWR_RESET" input (at 134.62 57.15 180)
+      (effects (font (size 1.27 1.27)) (justify left))
+    )
