File: OpenHT-RF/OpenHT-RF.kicad_sch (KiCad schematic)
At the start: 0 parts

Commit message: Finished power supply design
Other:
- sheet Connectors ports: added MCU_NRST; removed none
Changed lines of the file:
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@@
+    (stroke (width 0) (type default))
+  )
+  (wire (pts (xy 99.06 67.31) (xy 121.92 67.31))
     (stroke (width 0) (type default))
   )
@@
     (stroke (width 0) (type default))
   )
+  (wire (pts (xy 121.92 57.15) (xy 121.92 67.31))
+    (stroke (width 0) (type default))
+  )
   (wire (pts (xy 173.99 129.54) (xy 173.99 132.08))
     (stroke (width 0) (type default))
@@
   )
   (wire (pts (xy 179.07 134.62) (xy 185.42 134.62))
+    (stroke (width 0) (type default))
+  )
+  (wire (pts (xy 121.92 57.15) (xy 134.62 57.15))
     (stroke (width 0) (type default))
   )
@@
       (effects (font (size 1.27 1.27)) (justify right))
     )
+    (pin "MCU_NRST" input (at 99.06 67.31 0)
+      (effects (font (size 1.27 1.27)) (justify right))
+    )

Commit message: Optimised IO routing, renumbered components
Parts:
- added C69: 100nF, symbol Device:C
- added LS101: Speaker, symbol Device:Speaker
- added R11: 10kR, symbol Device:R
- added SW2: SW_Push, symbol Switch:SW_Push
Connections:
- net Connectors/SPK_N: now also LS101.2
- net Connectors/SPK_P: now also LS101.1
- new net: R11.1, SW2.2
- new net Connectors/PTT: C69.1, R11.2
- new net GND: C69.2, SW2.1
Other:
- sheet Connectors ports: added MAIN_KILL, PB_INT, PGOOD, PTT, RF_RST, SW_CTL1, SW_CTL2; removed none

Commit message: Updated PTT debounce circuit
Parts:
- C69: value 100nF -> 1uF
- R11: value 10kR -> 1kR
Changed lines of the file:
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@@
       (effects (font (size 1.27 1.27)))
     )
-    (property "Value" "10kR" (at 58.42 90.17 90)
+    (property "Value" "1kR" (at 58.42 90.17 90)
       (effects (font (size 1.27 1.27)))
     )
@@
       (effects (font (size 1.27 1.27)) (justify right))
     )
-    (property "Value" "100nF" (at 67.31 99.695 0)
+    (property "Value" "1uF" (at 67.31 99.695 0)
       (effects (font (size 1.27 1.27)) (justify right))
     )

Commit message: Added M17 logo
Parts:
- added LOGO101: M17_logo_20mmx15mm, M17_logos:M17_logo_20mmx15mm, symbol M17_logos:M17_logo_20mmx15mm
Changed lines of the file:
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@@
+    )
+  )
+  (symbol (lib_id "M17_logos:M17_logo_20mmx15mm") (at 144.78 35.56 0) (unit 1)
+    (in_bom no) (on_board yes) (dnp no) (fields_autoplaced)
+    (property "Reference" "LOGO101" (at 144.78 30.734 0)
+      (effects (font (size 1.27 1.27)) hide)
+    )
+    (property "Value" "M17_logo_20mmx15mm" (at 144.78 30.607 0)
+      (effects (font (size 1.27 1.27)) hide)
+    )
+    (property "Footprint" "M17_logos:M17_logo_20mmx15mm" (at 141.605 33.274 0)
+      (effects (font (size 1.27 1.27)) hide)
+    )
+    (property "Datasheet" "" (at 141.605 33.274 0)
+      (effects (font (size 1.27 1.27)) hide)
+    )
+    (instances
+      (project "OpenHT-RF"
+        (path "/3c300b59-23ec-47f8-bb91-29ca34130bcf"
+          (reference "LOGO101") (unit 1)
+        )
+      )
     )
   )

Commit message: [WIP] symbol-footprint association
Parts:
- C69: footprint (none) -> Capacitor_SMD:C_0402_1005Metric
- R11: footprint (none) -> Resistor_SMD:R_0402_1005Metric
Changed lines of the file:
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@@
       (effects (font (size 1.27 1.27)))
     )
-    (property "Footprint" "" (at 58.42 94.488 90)
+    (property "Footprint" "Resistor_SMD:R_0402_1005Metric" (at 58.42 94.488 90)
       (effects (font (size 1.27 1.27)) hide)
     )
@@
       (effects (font (size 1.27 1.27)) (justify right))
     )
-    (property "Footprint" "" (at 62.5348 101.6 0)
+    (property "Footprint" "Capacitor_SMD:C_0402_1005Metric" (at 62.5348 101.6 0)
       (effects (font (size 1.27 1.27)) hide)
     )

Commit message: Selected footprint
Parts:
- LS101: footprint (none) -> Connector_PinHeader_2.54mm:PinHeader_1x02_P2.54mm_Vertical
Changed lines of the file:
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@@
       (effects (font (size 1.27 1.27)) (justify left))
     )
-    (property "Footprint" "" (at 60.96 76.2 0)
+    (property "Footprint" "Connector_PinHeader_2.54mm:PinHeader_1x02_P2.54mm_Vertical" (at 60.96 76.2 0)
       (effects (font (size 1.27 1.27)) hide)
     )

Commit message: Updated switches
Parts:
- SW2: value SW_Push -> 436351045816; footprint (none) -> M17_misc_passive:SW_SPST_436351045816
Changed lines of the file:
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@@
       (effects (font (size 1.27 1.27)) (justify left))
     )
-    (property "Value" "SW_Push" (at 49.53 101.6 90)
+    (property "Value" "436351045816" (at 49.53 101.6 90)
       (effects (font (size 1.27 1.27)) (justify left))
     )
-    (property "Footprint" "" (at 48.26 99.06 0)
+    (property "Footprint" "M17_misc_passive:SW_SPST_436351045816" (at 48.26 99.06 0)
       (effects (font (size 1.27 1.27)) hide)
     )

Commit message: Speaker MPN
Parts:
- LS101: value Speaker -> SP-1605
Changed lines of the file:
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@@
       (effects (font (size 1.27 1.27)) (justify left))
     )
-    (property "Value" "Speaker" (at 55.88 74.295 0)
+    (property "Value" "SP-1605" (at 55.88 74.295 0)
       (effects (font (size 1.27 1.27)) (justify left))
     )
