File: OpenHT-RF/OpenHT-RF.kicad_sch (KiCad schematic)
At the start: 5 parts, among them SW2 436351045816

Commit message: Updated speaker footprint
Using SMD footprint
Parts:
- LS101: footprint Connector_PinHeader_2.54mm:PinHeader_1x02_P2.54mm_Vertical -> M17_connectors:Pin_1x02_P2.54mm_horizontal_SMD
Changed lines of the file:
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@@
       (effects (font (size 1.27 1.27)) (justify left))
     )
-    (property "Footprint" "Connector_PinHeader_2.54mm:PinHeader_1x02_P2.54mm_Vertical" (at 60.96 76.2 0)
+    (property "Footprint" "M17_connectors:Pin_1x02_P2.54mm_horizontal_SMD" (at 60.96 76.2 0)
       (effects (font (size 1.27 1.27)) hide)
     )

Commit message: Various schematic updates
Edited IO names, updated load switch symbol, swapped RF switch inputs
Other:
- sheet Connectors ports: added FPGA_RST; removed IO7
- sheet FPGA ports: added FPGA_RST; removed IO7
Changed lines of the file:
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@@
+    (stroke (width 0) (type default))
+  )
+  (wire (pts (xy 99.06 95.25) (xy 127 95.25))
     (stroke (width 0) (type default))
   )
@@
     (stroke (width 0) (type default))
   )
+  (wire (pts (xy 99.06 106.68) (xy 127 106.68))
+    (stroke (width 0) (type default))
+  )
+  (wire (pts (xy 102.87 125.73) (xy 102.87 137.16))
+    (stroke (width 0) (type default))
+  )
+  (wire (pts (xy 99.06 52.07) (xy 134.62 52.07))
+    (stroke (width 0) (type default))
+  )
   (wire (pts (xy 99.06 97.79) (xy 127 97.79))
     (stroke (width 0) (type default))
   )
-  (wire (pts (xy 99.06 95.25) (xy 127 95.25))
-    (stroke (width 0) (type default))
-  )
-  (wire (pts (xy 99.06 106.68) (xy 127 106.68))
-    (stroke (width 0) (type default))
-  )
-  (wire (pts (xy 102.87 125.73) (xy 102.87 137.16))
-    (stroke (width 0) (type default))
-  )
-  (wire (pts (xy 99.06 52.07) (xy 134.62 52.07))
-    (stroke (width 0) (type default))
-  )
   (wire (pts (xy 176.53 132.08) (xy 185.42 132.08))
     (stroke (width 0) (type default))
@@
     (stroke (width 0) (type default))
   )
+  (wire (pts (xy 181.61 71.12) (xy 181.61 81.28))
+    (stroke (width 0) (type default))
+  )
+  (wire (pts (xy 173.99 129.54) (xy 185.42 129.54))
+    (stroke (width 0) (type default))
+  )
+  (wire (pts (xy 165.1 106.68) (xy 185.42 106.68))
+    (stroke (width 0) (type default))
+  )
+  (wire (pts (xy 105.41 134.62) (xy 176.53 134.62))
+    (stroke (width 0) (type default))
+  )
+  (wire (pts (xy 63.5 93.98) (xy 63.5 92.71))
+    (stroke (width 0) (type default))
+  )
+  (wire (pts (xy 99.06 102.87) (xy 127 102.87))
+    (stroke (width 0) (type default))
+  )
+  (wire (pts (xy 176.53 76.2) (xy 176.53 87.63))
+    (stroke (width 0) (type default))
+  )
+  (wire (pts (xy 107.95 118.11) (xy 127 118.11))
+    (stroke (width 0) (type default))
+  )
+  (wire (pts (xy 173.99 91.44) (xy 173.99 78.74))
+    (stroke (width 0) (type default))
+  )
+  (wire (pts (xy 110.49 129.54) (xy 171.45 129.54))
+    (stroke (width 0) (type default))
+  )
+  (wire (pts (xy 99.06 76.2) (xy 176.53 76.2))
+    (stroke (width 0) (type default))
+  )
+  (wire (pts (xy 53.34 92.71) (xy 53.34 93.98))
+    (stroke (width 0) (type default))
+  )
+  (wire (pts (xy 99.06 111.76) (xy 127 111.76))
+    (stroke (width 0) (type default))
+  )
+  (wire (pts (xy 107.95 132.08) (xy 173.99 132.08))
+    (stroke (width 0) (type default))
+  )
+  (wire (pts (xy 171.45 127) (xy 171.45 129.54))
+    (stroke (width 0) (type default))
+  )
+  (wire (pts (xy 99.06 63.5) (xy 134.62 63.5))
+    (stroke (width 0) (type default))
+  )
+  (wire (pts (xy 62.23 92.71) (xy 63.5 92.71))
+    (stroke (width 0) (type default))
+  )
   (wire (pts (xy 99.06 100.33) (xy 127 100.33))
-    (stroke (width 0) (type default))
-  )
-  (wire (pts (xy 181.61 71.12) (xy 181.61 81.28))
-    (stroke (width 0) (type default))
-  )
-  (wire (pts (xy 173.99 129.54) (xy 185.42 129.54))
-    (stroke (width 0) (type default))
-  )
-  (wire (pts (xy 165.1 106.68) (xy 185.42 106.68))
-    (stroke (width 0) (type default))
-  )
-  (wire (pts (xy 105.41 134.62) (xy 176.53 134.62))
-    (stroke (width 0) (type default))
-  )
-  (wire (pts (xy 63.5 93.98) (xy 63.5 92.71))
-    (stroke (width 0) (type default))
-  )
-  (wire (pts (xy 176.53 76.2) (xy 176.53 87.63))
-    (stroke (width 0) (type default))
-  )
-  (wire (pts (xy 107.95 118.11) (xy 127 118.11))
-    (stroke (width 0) (type default))
-  )
-  (wire (pts (xy 173.99 91.44) (xy 173.99 78.74))
-    (stroke (width 0) (type default))
-  )
-  (wire (pts (xy 110.49 129.54) (xy 171.45 129.54))
-    (stroke (width 0) (type default))
-  )
-  (wire (pts (xy 99.06 76.2) (xy 176.53 76.2))
-    (stroke (width 0) (type default))
-  )
-  (wire (pts (xy 99.06 102.87) (xy 127 102.87))
-    (stroke (width 0) (type default))
-  )
-  (wire (pts (xy 53.34 92.71) (xy 53.34 93.98))
-    (stroke (width 0) (type default))
-  )
-  (wire (pts (xy 99.06 111.76) (xy 127 111.76))
-    (stroke (width 0) (type default))
-  )
-  (wire (pts (xy 107.95 132.08) (xy 173.99 132.08))
-    (stroke (width 0) (type default))
-  )
-  (wire (pts (xy 171.45 127) (xy 171.45 129.54))
-    (stroke (width 0) (type default))
-  )
-  (wire (pts (xy 99.06 63.5) (xy 134.62 63.5))
-    (stroke (width 0) (type default))
-  )
-  (wire (pts (xy 62.23 92.71) (xy 63.5 92.71))
     (stroke (width 0) (type default))
   )
@@
       (effects (font (size 1.27 1.27)) (justify right))
     )
-    (pin "IO7" bidirectional (at 99.06 102.87 0)
-      (effects (font (size 1.27 1.27)) (justify right))
-    )
     (pin "IO6" bidirectional (at 99.06 100.33 0)
       (effects (font (size 1.27 1.27)) (justify right))
     )
+    (pin "IO5" bidirectional (at 99.06 97.79 0)
+      (effects (font (size 1.27 1.27)) (justify right))
+    )
     (pin "DONE" bidirectional (at 99.06 109.22 0)
       (effects (font (size 1.27 1.27)) (justify right))
@@
       (effects (font (size 1.27 1.27)) (justify right))
     )
-    (pin "IO5" bidirectional (at 99.06 97.79 0)
+    (pin "IO4" bidirectional (at 99.06 95.25 0)
       (effects (font (size 1.27 1.27)) (justify right))
     )
@@
       (effects (font (size 1.27 1.27)) (justify right))
     )
-    (pin "IO4" bidirectional (at 99.06 95.25 0)
+    (pin "FPGA_RST" bidirectional (at 99.06 102.87 0)
       (effects (font (size 1.27 1.27)) (justify right))
     )
@@
       (effects (font (size 1.27 1.27)) (justify left))
     )
+    (pin "FPGA_RST" bidirectional (at 127 102.87 180)
+      (effects (font (size 1.27 1.27)) (justify left))
+    )
+    (pin "IO1" bidirectional (at 127 87.63 180)
+      (effects (font (size 1.27 1.27)) (justify left))
+    )
+    (pin "IO0" bidirectional (at 127 85.09 180)
+      (effects (font (size 1.27 1.27)) (justify left))
+    )
+    (pin "INITN" bidirectional (at 127 106.68 180)
+      (effects (font (size 1.27 1.27)) (justify left))
+    )
+    (pin "IO5" bidirectional (at 127 97.79 180)
+      (effects (font (size 1.27 1.27)) (justify left))
+    )
+    (pin "IO6" bidirectional (at 127 100.33 180)
+      (effects (font (size 1.27 1.27)) (justify left))
+    )
     (pin "IO4" bidirectional (at 127 95.25 180)
       (effects (font (size 1.27 1.27)) (justify left))
     )
-    (pin "IO1" bidirectional (at 127 87.63 180)
-      (effects (font (size 1.27 1.27)) (justify left))
-    )
-    (pin "IO0" bidirectional (at 127 85.09 180)
-      (effects (font (size 1.27 1.27)) (justify left))
-    )
-    (pin "INITN" bidirectional (at 127 106.68 180)
-      (effects (font (size 1.27 1.27)) (justify left))
-    )
-    (pin "IO6" bidirectional (at 127 100.33 180)
-      (effects (font (size 1.27 1.27)) (justify left))
-    )
-    (pin "IO7" bidirectional (at 127 102.87 180)
-      (effects (font (size 1.27 1.27)) (justify left))
-    )
-    (pin "IO5" bidirectional (at 127 97.79 180)
-      (effects (font (size 1.27 1.27)) (justify left))
-    )

Commit message: Layout improvements and current measurement jumpers
Parts:
- C69: footprint Capacitor_SMD:C_0402_1005Metric -> Connector_PinHeader_2.54mm:PinHeader_1x02_P2.54mm_Vertical_SMD_Pin1Right
Changed lines of the file:
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@@
       (effects (font (size 1.27 1.27)) (justify right))
     )
-    (property "Footprint" "Capacitor_SMD:C_0402_1005Metric" (at 62.5348 101.6 0)
+    (property "Footprint" "Connector_PinHeader_2.54mm:PinHeader_1x02_P2.54mm_Vertical_SMD_Pin1Right" (at 62.5348 101.6 0)
       (effects (font (size 1.27 1.27)) hide)
     )

Commit message: BOM updates
Parts:
- LS101: Manual_Placement (none) -> 1
- SW2: MPN (none) -> 436351045816
Changed lines of the file:
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@@
+      (effects (font (size 1.27 1.27)) hide)
+    )
+    (property "MPN" "436351045816" (at 53.34 99.06 0)
       (effects (font (size 1.27 1.27)) hide)
     )
@@
       (effects (font (size 1.27 1.27)) hide)
     )
+    (property "Manual_Placement" "1" (at 60.96 71.12 0)
+      (effects (font (size 1.27 1.27)) hide)
+    )

Commit message: Updated incorrect capacitor footprint
Parts:
- C69: footprint Connector_PinHeader_2.54mm:PinHeader_1x02_P2.54mm_Vertical_SMD_Pin1Right -> Capacitor_SMD:C_0402_1005Metric
Changed lines of the file:
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@@
       (effects (font (size 1.27 1.27)) (justify right))
     )
-    (property "Footprint" "Connector_PinHeader_2.54mm:PinHeader_1x02_P2.54mm_Vertical_SMD_Pin1Right" (at 62.5348 101.6 0)
+    (property "Footprint" "Capacitor_SMD:C_0402_1005Metric" (at 62.5348 101.6 0)
       (effects (font (size 1.27 1.27)) hide)
     )

Commit message: Added OSHW logo, gnd TP and via stitching
Also added comments, revision number, and an easter egg
Parts:
- added FID101, FID102, FID103: Fiducial, Fiducial:Fiducial_1mm_Mask2mm, symbol Mechanical:Fiducial
- added SYM101: Logo_Open_Hardware_Small, Symbol:OSHW-Logo_7.5x8mm_SilkScreen, symbol Graphic:Logo_Open_Hardware_Small
Changed lines of the file:
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@@
     (rev "A")
     (company "M17 Project")
-    (comment 1 "Authors: Wojciech SP5WWP, Leo Hofer, Morgan ON4MOD")
+    (comment 1 "Authors: Morgan ON4MOD, Wojciech SP5WWP, Leo Hofer")
   )
   (junction (at 110.49 115.57) (diameter 0) (color 0 0 0 0)
@@
     (property "Netclass" "LVDS" (at 170.8785 105.41 0)
       (effects (font (size 1.27 1.27) italic) (justify left))
+    )
+  )
+  (symbol (lib_id "Mechanical:Fiducial") (at 115.57 189.23 0) (unit 1)
+    (in_bom yes) (on_board yes) (dnp no) (fields_autoplaced)
+    (property "Reference" "FID102" (at 118.11 188.595 0)
+      (effects (font (size 1.27 1.27)) (justify left))
+    )
+    (property "Value" "Fiducial" (at 118.11 191.135 0)
+      (effects (font (size 1.27 1.27)) (justify left))
+    )
+    (property "Footprint" "Fiducial:Fiducial_1mm_Mask2mm" (at 115.57 189.23 0)
+      (effects (font (size 1.27 1.27)) hide)
+    )
+    (property "Datasheet" "~" (at 115.57 189.23 0)
+      (effects (font (size 1.27 1.27)) hide)
+    )
+    (instances
+      (project "OpenHT-RF"
+        (path "/3c300b59-23ec-47f8-bb91-29ca34130bcf"
+          (reference "FID102") (unit 1)
+        )
+      )
+    )
+  )
+  (symbol (lib_id "Mechanical:Fiducial") (at 101.6 189.23 0) (unit 1)
+    (in_bom yes) (on_board yes) (dnp no) (fields_autoplaced)
+    (property "Reference" "FID101" (at 104.14 188.595 0)
+      (effects (font (size 1.27 1.27)) (justify left))
+    )
+    (property "Value" "Fiducial" (at 104.14 191.135 0)
+      (effects (font (size 1.27 1.27)) (justify left))
+    )
+    (property "Footprint" "Fiducial:Fiducial_1mm_Mask2mm" (at 101.6 189.23 0)
+      (effects (font (size 1.27 1.27)) hide)
+    )
+    (property "Datasheet" "~" (at 101.6 189.23 0)
+      (effects (font (size 1.27 1.27)) hide)
+    )
+    (instances
+      (project "OpenHT-RF"
+        (path "/3c300b59-23ec-47f8-bb91-29ca34130bcf"
+          (reference "FID101") (unit 1)
+        )
+      )
     )
   )
@@
     )
   )
+  (symbol (lib_id "Mechanical:Fiducial") (at 129.54 189.23 0) (unit 1)
+    (in_bom yes) (on_board yes) (dnp no) (fields_autoplaced)
+    (property "Reference" "FID103" (at 132.08 188.595 0)
+      (effects (font (size 1.27 1.27)) (justify left))
+    )
+    (property "Value" "Fiducial" (at 132.08 191.135 0)
+      (effects (font (size 1.27 1.27)) (justify left))
+    )
+    (property "Footprint" "Fiducial:Fiducial_1mm_Mask2mm" (at 129.54 189.23 0)
+      (effects (font (size 1.27 1.27)) hide)
+    )
+    (property "Datasheet" "~" (at 129.54 189.23 0)
+      (effects (font (size 1.27 1.27)) hide)
+    )
+    (instances
+      (project "OpenHT-RF"
+        (path "/3c300b59-23ec-47f8-bb91-29ca34130bcf"
+          (reference "FID103") (unit 1)
+        )
+      )
+    )
+  )
   (symbol (lib_id "Device:Speaker") (at 60.96 71.12 0) (mirror y) (unit 1)
     (in_bom yes) (on_board yes) (dnp no)
@@
         )
       )
+    )
+  )
+  (symbol (lib_id "Graphic:Logo_Open_Hardware_Small") (at 162.56 35.56 0) (unit 1)
+    (in_bom no) (on_board yes) (dnp no) (fields_autoplaced)
+    (property "Reference" "SYM101" (at 162.56 28.575 0)
+      (effects (font (size 1.27 1.27)) hide)
+    )
+    (property "Value" "Logo_Open_Hardware_Small" (at 162.56 41.275 0)
+      (effects (font (size 1.27 1.27)) hide)
+    )
+    (property "Footprint" "Symbol:OSHW-Logo_7.5x8mm_SilkScreen" (at 162.56 35.56 0)
+      (effects (font (size 1.27 1.27)) hide)
+    )
+    (property "Datasheet" "~" (at 162.56 35.56 0)
+      (effects (font (size 1.27 1.27)) hide)
+    )
+    (property "Sim.Enable" "0" (at 162.56 35.56 0)
+      (effects (font (size 1.27 1.27)) hide)
+    )
+    (instances
+      (project "OpenHT-RF"
+        (path "/3c300b59-23ec-47f8-bb91-29ca34130bcf"
+          (reference "SYM101") (unit 1)
+        )
+      )
