File: OpenHT-RF/conn.kicad_sch (KiCad schematic)
At the start: 5 parts, among them J5 Conn_01x08, J5 Conn_02x08_Odd_Even, J6 Conn_01x06, J7 Conn_01x10, J8 Conn_01x08

Commit message: Update conn.kicad_sch
Connections:
- net VIN_BAT: now reaches J5.8 (Pin_8)
Other:
- note added: "CN5"
- note added: "CN6"
- note added: "CN7"
- note added: "CN8"
Changed lines of the file:
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@@
+    (stroke (width 0) (type default))
+  )
+  (wire (pts (xy 53.34 100.33) (xy 67.31 100.33))
     (stroke (width 0) (type default))
   )
@@
     (stroke (width 0) (type default))
   )
+  (text "CN7" (at 96.52 116.84 90)
+    (effects (font (size 1.27 1.27)) (justify left bottom))
+  )
   (text "2x8 CN12 connector" (at 144.78 127 0)
+    (effects (font (size 1.27 1.27)) (justify left bottom))
+  )
+  (text "CN8\n" (at 78.74 116.84 90)
+    (effects (font (size 1.27 1.27)) (justify left bottom))
+  )
+  (text "CN5" (at 96.52 85.09 90)
+    (effects (font (size 1.27 1.27)) (justify left bottom))
+  )
+  (text "CN6" (at 78.74 92.71 90)
     (effects (font (size 1.27 1.27)) (justify left bottom))
   )
@@
     (effects (font (size 1.27 1.27)) (justify left bottom))
   )
+  (label "VIN_BAT" (at 53.34 100.33 0) (fields_autoplaced)
+    (effects (font (size 1.27 1.27)) (justify left bottom))
+  )

Commit message: Added description of Arduino connectors
Connections:
- net +3V3: now also J5.4 (Pin_4)
- net GND: now also J5.6 (Pin_6), J5.7 (Pin_7), J7.4 (Pin_4)
- net SPI_NSS: now reaches J5.11 (Pin_11)
- net SPI_MISO: now reaches J5.5 (Pin_5)
- net SPI_SCK: now reaches J5.7 (Pin_7)
- net SPI_MOSI: now reaches J5.9 (Pin_9)
- net +5V: now reaches J5.5 (Pin_5)
- no-connect marks 0 -> 4
Other:
- note added: "(PG10)"
- note added: "(PG11)"
- note added: "(PG12)"
- note added: "(PG13)"
- note added: "+3V3"
- note added: "+5V"
- note added: "A0 (PB1)"
- note added: "A1 (PC2)"
- note added: "A2 (PC3)"
- note added: "A3 (PC4)"
- note added: "A4 (PC5)"
- note added: "A5 (PA4)"
- note added: "ANTITAMP1 (PC13)"
- note added: "AVdd"
- note added: "Arduino uno connector"
- note added: "GND"
- note added: "I2C1_SCL(PB8)"
- note added: "I2C1_SDA (PB9)"
- note added: "I2C2_WS, CAN2_RX, TIM1_BKIN (PB12)"
- note added: "I2S2_CK, CAN2_TX, USART3_CTS, TIM1_CH1N (PB13)"
- note added: "I2S2_SD, ADC1/ADC2/ADC3_IN11 (PC1)"
- note added: "IOREF"
- note added: "MCO1, TIM1_CH1 (MCO1)"
- note added: "NRST"
- note added: "SPI1_MISO, TIM3_CH1 (PB4)"
- note added: "SPI1_MOSI, TIM3_CH2, I2C1_SMBA, CAN2_RX (PB5)"
- note added: "SPI1_NSS, TIM2_CH1/2_ETR (PA15)"
- note added: "SPI1_SCK, TIM2/TIM8_CH1, ADC1/ADC2_IN5 (PA5)"
- note added: "SPI2_MISO (PB14)"
- note added: "SPI2_SCK (PD3)"
- note added: "TIM12_CH1 (PH6)"
- note added: "TIM12_CH2, SPI2_MOSI (PB15)"
- note added: "TIM14_CH1 (PA7)"
- note added: "TIM3_CH1 (PA6)"
- note added: "TIM5_CH2 (PA1)"
- note added: "TIM5_CH3 (PA2)"
- note added: "USART6_RX (PG9)"
- note added: "USART6_RX, TIM3/TIM8_CH2 (PC7)"
- note added: "USART6_TX (PG14)"
- note added: "USART6_TX, I2S2_MCK, TIM3/TIM8_CH1 (PC6)"
- note added: "Vin"
- note removed: "Arduino connector"
- note removed: "CN5"
- note removed: "CN6"
- note removed: "CN7"
- note removed: "CN8"
- moved on the sheet: J5, J7, J8

Commit message: Updated FPGA, RF and connectors sheets [WIP]
Parts:
- added R2, R3, R4, R5, R7: 100R, symbol Device:R
Connections:
- net SPI_MISO: now also R2.1; no longer J5.5 (Pin_5)
- net SPI_MOSI: now also R4.1; no longer J5.9 (Pin_9)
- net SPI_SCK: now also R3.1; no longer J5.7 (Pin_7)
- net at J7.10 (Pin_10): now also R7.1
- net SPI_NSS: no longer names the net of J5.11 (Pin_11)
- net SPI_NSS: now also R5.2
- new net: J5.7 (Pin_7), R3.2
- new net: J5.5 (Pin_5), R2.2
- new net: J5.9 (Pin_9), R4.2
- new net SPI_NSS1: R5.1
- new net SPI_NSS2: R7.2
Changed lines of the file:
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@@
+    (stroke (width 0) (type default))
+  )
+  (wire (pts (xy 25.4 146.05) (xy 29.21 146.05))
     (stroke (width 0) (type default))
   )
@@
     (stroke (width 0) (type default))
   )
+  (wire (pts (xy 25.4 151.13) (xy 29.21 151.13))
+    (stroke (width 0) (type default))
+  )
   (wire (pts (xy 67.31 88.9) (xy 68.58 88.9))
     (stroke (width 0) (type default))
   )
+  (wire (pts (xy 129.54 97.79) (xy 133.35 97.79))
+    (stroke (width 0) (type default))
+  )
   (wire (pts (xy 36.83 146.05) (xy 86.36 146.05))
     (stroke (width 0) (type default))
@@
     (stroke (width 0) (type default))
   )
+  (wire (pts (xy 25.4 148.59) (xy 29.21 148.59))
+    (stroke (width 0) (type default))
+  )
   (wire (pts (xy 36.83 156.21) (xy 86.36 156.21))
     (stroke (width 0) (type default))
   )
+  (wire (pts (xy 25.4 143.51) (xy 29.21 143.51))
+    (stroke (width 0) (type default))
+  )
   (wire (pts (xy 55.88 82.55) (xy 55.88 83.82))
     (stroke (width 0) (type default))
@@
     (stroke (width 0) (type default))
   )
+  (wire (pts (xy 121.92 97.79) (xy 118.11 97.79))
+    (stroke (width 0) (type default))
+  )
   (wire (pts (xy 36.83 151.13) (xy 86.36 151.13))
     (stroke (width 0) (type default))
@@
     (effects (font (size 1.27 1.27)) (justify left bottom))
   )
-  (hierarchical_label "SPI_SCK" (shape input) (at 36.83 146.05 180) (fields_autoplaced)
+  (hierarchical_label "SPI_SCK" (shape output) (at 25.4 146.05 180) (fields_autoplaced)
     (effects (font (size 1.27 1.27)) (justify right))
   )
-  (hierarchical_label "SPI_NSS" (shape input) (at 36.83 151.13 180) (fields_autoplaced)
+  (hierarchical_label "SPI_NSS1" (shape output) (at 25.4 151.13 180) (fields_autoplaced)
     (effects (font (size 1.27 1.27)) (justify right))
   )
-  (hierarchical_label "SPI_MISO" (shape input) (at 36.83 143.51 180) (fields_autoplaced)
+  (hierarchical_label "SPI_NSS2" (shape output) (at 132.08 97.79 0) (fields_autoplaced)
+    (effects (font (size 1.27 1.27)) (justify left))
+  )
+  (hierarchical_label "SPI_MISO" (shape input) (at 25.4 143.51 180) (fields_autoplaced)
     (effects (font (size 1.27 1.27)) (justify right))
   )
@@
     (effects (font (size 1.27 1.27)) (justify left))
   )
-  (hierarchical_label "SPI_MOSI" (shape input) (at 36.83 148.59 180) (fields_autoplaced)
+  (hierarchical_label "SPI_MOSI" (shape output) (at 25.4 148.59 180) (fields_autoplaced)
     (effects (font (size 1.27 1.27)) (justify right))
   )
@@
         (path "/3c300b59-23ec-47f8-bb91-29ca34130bcf/1ac744a1-066f-4d1a-b0df-41e1d7c4818a"
           (reference "J4") (unit 1)
+        )
+      )
+    )
+  )
+  (symbol (lib_id "Device:R") (at 33.02 146.05 90) (unit 1)
+    (in_bom yes) (on_board yes) (dnp no)
+    (property "Reference" "R3" (at 29.21 144.78 90)
+      (effects (font (size 1.27 1.27)))
+    )
+    (property "Value" "100R" (at 33.02 146.05 90)
+      (effects (font (size 1.27 1.27)))
+    )
+    (property "Footprint" "" (at 33.02 147.828 90)
+      (effects (font (size 1.27 1.27)) hide)
+    )
+    (property "Datasheet" "~" (at 33.02 146.05 0)
+      (effects (font (size 1.27 1.27)) hide)
+    )
+    (pin "1")
+    (pin "2")
+    (instances
+      (project "OpenHT-RF"
+        (path "/3c300b59-23ec-47f8-bb91-29ca34130bcf/1ac744a1-066f-4d1a-b0df-41e1d7c4818a"
+          (reference "R3") (unit 1)
         )
       )
@@
     )
   )
+  (symbol (lib_id "Device:R") (at 33.02 151.13 90) (unit 1)
+    (in_bom yes) (on_board yes) (dnp no)
+    (property "Reference" "R5" (at 29.21 149.86 90)
+      (effects (font (size 1.27 1.27)))
+    )
+    (property "Value" "100R" (at 33.02 151.13 90)
+      (effects (font (size 1.27 1.27)))
+    )
+    (property "Footprint" "" (at 33.02 152.908 90)
+      (effects (font (size 1.27 1.27)) hide)
+    )
+    (property "Datasheet" "~" (at 33.02 151.13 0)
+      (effects (font (size 1.27 1.27)) hide)
+    )
+    (pin "1")
+    (pin "2")
+    (instances
+      (project "OpenHT-RF"
+        (path "/3c300b59-23ec-47f8-bb91-29ca34130bcf/1ac744a1-066f-4d1a-b0df-41e1d7c4818a"
+          (reference "R5") (unit 1)
+        )
+      )
+    )
+  )
   (symbol (lib_id "power:+3V3") (at 74.93 137.16 0) (unit 1)
     (in_bom yes) (on_board yes) (dnp no) (fields_autoplaced)
@@
     )
   )
+  (symbol (lib_id "Device:R") (at 33.02 148.59 90) (unit 1)
+    (in_bom yes) (on_board yes) (dnp no)
+    (property "Reference" "R4" (at 29.21 147.32 90)
+      (effects (font (size 1.27 1.27)))
+    )
+    (property "Value" "100R" (at 33.02 148.59 90)
+      (effects (font (size 1.27 1.27)))
+    )
+    (property "Footprint" "" (at 33.02 150.368 90)
+      (effects (font (size 1.27 1.27)) hide)
+    )
+    (property "Datasheet" "~" (at 33.02 148.59 0)
+      (effects (font (size 1.27 1.27)) hide)
+    )
+    (pin "1")
+    (pin "2")
+    (instances
+      (project "OpenHT-RF"
+        (path "/3c300b59-23ec-47f8-bb91-29ca34130bcf/1ac744a1-066f-4d1a-b0df-41e1d7c4818a"
+          (reference "R4") (unit 1)
+        )
+      )
+    )
+  )
+  (symbol (lib_id "Device:R") (at 125.73 97.79 90) (unit 1)
+    (in_bom yes) (on_board yes) (dnp no)
+    (property "Reference" "R7" (at 121.92 96.52 90)
+      (effects (font (size 1.27 1.27)))
+    )
+    (property "Value" "100R" (at 125.73 97.79 90)
+      (effects (font (size 1.27 1.27)))
+    )
+    (property "Footprint" "" (at 125.73 99.568 90)
+      (effects (font (size 1.27 1.27)) hide)
+    )
+    (property "Datasheet" "~" (at 125.73 97.79 0)
+      (effects (font (size 1.27 1.27)) hide)
+    )
+    (pin "1")
+    (pin "2")
+    (instances
+      (project "OpenHT-RF"
+        (path "/3c300b59-23ec-47f8-bb91-29ca34130bcf/1ac744a1-066f-4d1a-b0df-41e1d7c4818a"
+          (reference "R7") (unit 1)
+        )
+      )
+    )
+  )
   (symbol (lib_id "power:GND") (at 106.68 138.43 90) (unit 1)
     (in_bom yes) (on_board yes) (dnp no) (fields_autoplaced)
@@
         )
       )
+    )
+  )
+  (symbol (lib_id "Device:R") (at 33.02 143.51 90) (unit 1)
+    (in_bom yes) (on_board yes) (dnp no)
+    (property "Reference" "R2" (at 29.21 142.24 90)
+      (effects (font (size 1.27 1.27)))
+    )
+    (property "Value" "100R" (at 33.02 143.51 90)
+      (effects (font (size 1.27 1.27)))
+    )
+    (property "Footprint" "" (at 33.02 145.288 90)
+      (effects (font (size 1.27 1.27)) hide)
+    )
+    (property "Datasheet" "~" (at 33.02 143.51 0)
+      (effects (font (size 1.27 1.27)) hide)
+    )
+    (pin "1")
+    (pin "2")
+    (instances
+      (project "OpenHT-RF"
+        (path "/3c300b59-23ec-47f8-bb91-29ca34130bcf/1ac744a1-066f-4d1a-b0df-41e1d7c4818a"
+          (reference "R2") (unit 1)
+        )
+      )

Commit message: Updated FPGA, RF and connectors sheets [WIP]
Parts:
- added R10, R11, R12, R8, R9: 100R, symbol Device:R
Connections:
- net at J8.1 (Pin_1): now also R8.1
- net DONE: now reaches J8.2 (Pin_2)
- net at J8.3 (Pin_3): now also R9.1
- net at J8.4 (Pin_4): now also R10.1
- net IO3: now reaches J8.5 (Pin_5)
- net IO2: now reaches J8.6 (Pin_6)
- net IO1: now reaches J8.7 (Pin_7)
- net IO0: now reaches J8.8 (Pin_8)
- net IRQ_AT86RF215: now reaches J7.8 (Pin_8)
- net INITN: now reaches J7.9 (Pin_9)
- net at J6.1 (Pin_1): now also R11.2
- net at J6.2 (Pin_2): now also R12.2
- new net IO4: R10.2
- new net IO5: R9.2
- new net IO6: R11.1
- new net IO7: R12.1
- new net PROGRAMN: R8.2
Other:
- moved on the sheet: J5, J6, J7, J8, R2, R3, R4, R5, R7

Commit message: Finished power supply design
Connections:
- net MCU_NRST: now reaches J5.3 (Pin_3)
Changed lines of the file:
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@@
     (comment 1 "Authors: Wojciech SP5WWP, Leo Hofer, Morgan ON4MOD")
   )
-  (junction (at 115.57 67.31) (diameter 0) (color 0 0 0 0)
-  )
-  (junction (at 101.6 69.85) (diameter 0) (color 0 0 0 0)
-  )
   (junction (at 127 72.39) (diameter 0) (color 0 0 0 0)
+  )
+  (junction (at 113.03 67.31) (diameter 0) (color 0 0 0 0)
+  )
+  (junction (at 99.06 69.85) (diameter 0) (color 0 0 0 0)
   )
   (no_connect (at 128.27 59.69))
@@
     (stroke (width 0) (type default))
   )
-  (wire (pts (xy 106.68 66.04) (xy 106.68 67.31))
-    (stroke (width 0) (type default))
-  )
   (wire (pts (xy 127 72.39) (xy 111.76 72.39))
     (stroke (width 0) (type default))
@@
     (stroke (width 0) (type default))
   )
-  (wire (pts (xy 128.27 67.31) (xy 115.57 67.31))
-    (stroke (width 0) (type default))
-  )
   (wire (pts (xy 186.69 66.04) (xy 186.69 67.31))
     (stroke (width 0) (type default))
   )
-  (wire (pts (xy 93.98 69.85) (xy 101.6 69.85))
+  (wire (pts (xy 93.98 69.85) (xy 99.06 69.85))
     (stroke (width 0) (type default))
   )
@@
     (stroke (width 0) (type default))
   )
+  (wire (pts (xy 113.03 67.31) (xy 128.27 67.31))
+    (stroke (width 0) (type default))
+  )
   (wire (pts (xy 96.52 132.08) (xy 146.05 132.08))
     (stroke (width 0) (type default))
@@
     (stroke (width 0) (type default))
   )
-  (wire (pts (xy 93.98 68.58) (xy 93.98 69.85))
-    (stroke (width 0) (type default))
-  )
   (wire (pts (xy 118.11 77.47) (xy 128.27 77.47))
     (stroke (width 0) (type default))
@@
     (stroke (width 0) (type default))
   )
+  (wire (pts (xy 99.06 69.85) (xy 128.27 69.85))
+    (stroke (width 0) (type default))
+  )
   (wire (pts (xy 96.52 127) (xy 146.05 127))
     (stroke (width 0) (type default))
   )
-  (wire (pts (xy 101.6 69.85) (xy 128.27 69.85))
-    (stroke (width 0) (type default))
-  )
-  (wire (pts (xy 101.6 68.58) (xy 101.6 69.85))
+  (wire (pts (xy 99.06 68.58) (xy 99.06 69.85))
     (stroke (width 0) (type default))
   )
@@
     (stroke (width 0) (type default))
   )
-  (wire (pts (xy 106.68 67.31) (xy 115.57 67.31))
+  (wire (pts (xy 107.95 67.31) (xy 113.03 67.31))
+    (stroke (width 0) (type default))
+  )
+  (wire (pts (xy 127 64.77) (xy 128.27 64.77))
     (stroke (width 0) (type default))
   )
@@
     (stroke (width 0) (type default))
   )
-  (wire (pts (xy 115.57 66.04) (xy 115.57 67.31))
+  (wire (pts (xy 113.03 66.04) (xy 113.03 67.31))
     (stroke (width 0) (type default))
   )
@@
     (effects (font (size 1.27 1.27)) (justify right))
   )
+  (hierarchical_label "MCU_NRST" (shape input) (at 127 64.77 180) (fields_autoplaced)
+    (effects (font (size 1.27 1.27)) (justify right))
+  )
   (hierarchical_label "SPI_MOSI" (shape output) (at 85.09 132.08 180) (fields_autoplaced)
     (effects (font (size 1.27 1.27)) (justify right))
@@
     (effects (font (size 1.27 1.27)) (justify left))
   )
-  (symbol (lib_id "power:PWR_FLAG") (at 93.98 68.58 0) (unit 1)
+  (symbol (lib_id "power:PWR_FLAG") (at 93.98 69.85 90) (unit 1)
     (in_bom yes) (on_board yes) (dnp no) (fields_autoplaced)
-    (property "Reference" "#FLG02" (at 93.98 66.675 0)
-      (effects (font (size 1.27 1.27)) hide)
-    )
-    (property "Value" "PWR_FLAG" (at 93.98 64.77 0)
-      (effects (font (size 1.27 1.27)))
-    )
-    (property "Footprint" "" (at 93.98 68.58 0)
-      (effects (font (size 1.27 1.27)) hide)
-    )
-    (property "Datasheet" "~" (at 93.98 68.58 0)
+    (property "Reference" "#FLG02" (at 92.075 69.85 0)
+      (effects (font (size 1.27 1.27)) hide)
+    )
+    (property "Value" "PWR_FLAG" (at 92.71 67.31 90)
+      (effects (font (size 1.27 1.27)))
+    )
+    (property "Footprint" "" (at 93.98 69.85 0)
+      (effects (font (size 1.27 1.27)) hide)
+    )
+    (property "Datasheet" "~" (at 93.98 69.85 0)
       (effects (font (size 1.27 1.27)) hide)
     )
@@
     )
   )
-  (symbol (lib_id "power:+5V") (at 101.6 68.58 0) (unit 1)
+  (symbol (lib_id "power:+5V") (at 99.06 68.58 0) (unit 1)
     (in_bom yes) (on_board yes) (dnp no) (fields_autoplaced)
-    (property "Reference" "#PWR06" (at 101.6 72.39 0)
-      (effects (font (size 1.27 1.27)) hide)
-    )
-    (property "Value" "+5V" (at 101.6 64.77 0)
-      (effects (font (size 1.27 1.27)))
-    )
-    (property "Footprint" "" (at 101.6 68.58 0)
-      (effects (font (size 1.27 1.27)) hide)
-    )
-    (property "Datasheet" "" (at 101.6 68.58 0)
+    (property "Reference" "#PWR06" (at 99.06 72.39 0)
+      (effects (font (size 1.27 1.27)) hide)
+    )
+    (property "Value" "+5V" (at 99.06 64.77 0)
+      (effects (font (size 1.27 1.27)))
+    )
+    (property "Footprint" "" (at 99.06 68.58 0)
+      (effects (font (size 1.27 1.27)) hide)
+    )
+    (property "Datasheet" "" (at 99.06 68.58 0)
       (effects (font (size 1.27 1.27)) hide)
     )
@@
     )
   )
-  (symbol (lib_id "power:PWR_FLAG") (at 106.68 66.04 0) (unit 1)
+  (symbol (lib_id "power:PWR_FLAG") (at 107.95 67.31 90) (unit 1)
     (in_bom yes) (on_board yes) (dnp no) (fields_autoplaced)
-    (property "Reference" "#FLG01" (at 106.68 64.135 0)
-      (effects (font (size 1.27 1.27)) hide)
-    )
-    (property "Value" "PWR_FLAG" (at 106.68 62.23 0)
-      (effects (font (size 1.27 1.27)))
-    )
-    (property "Footprint" "" (at 106.68 66.04 0)
-      (effects (font (size 1.27 1.27)) hide)
-    )
-    (property "Datasheet" "~" (at 106.68 66.04 0)
+    (property "Reference" "#FLG01" (at 106.045 67.31 0)
+      (effects (font (size 1.27 1.27)) hide)
+    )
+    (property "Value" "PWR_FLAG" (at 106.68 64.77 90)
+      (effects (font (size 1.27 1.27)))
+    )
+    (property "Footprint" "" (at 107.95 67.31 0)
+      (effects (font (size 1.27 1.27)) hide)
+    )
+    (property "Datasheet" "~" (at 107.95 67.31 0)
       (effects (font (size 1.27 1.27)) hide)
     )
@@
     )
   )
-  (symbol (lib_id "power:+3V3") (at 115.57 66.04 0) (unit 1)
+  (symbol (lib_id "power:+3V3") (at 113.03 66.04 0) (unit 1)
     (in_bom yes) (on_board yes) (dnp no) (fields_autoplaced)
-    (property "Reference" "#PWR07" (at 115.57 69.85 0)
-      (effects (font (size 1.27 1.27)) hide)
-    )
-    (property "Value" "+3V3" (at 115.57 62.23 0)
-      (effects (font (size 1.27 1.27)))
-    )
-    (property "Footprint" "" (at 115.57 66.04 0)
-      (effects (font (size 1.27 1.27)) hide)
-    )
-    (property "Datasheet" "" (at 115.57 66.04 0)
-      (effects (font (size 1.27 1.27)) hide)
-    )
+    (property "Reference" "#PWR07" (at 113.03 69.85 0)
+      (effects (font (size 1.27 1.27)) hide)
+    )
+    (property "Value" "+3V3" (at 113.03 62.23 0)
+      (effects (font (size 1.27 1.27)))
+    )
+    (property "Footprint" "" (at 113.03 66.04 0)
+      (effects (font (size 1.27 1.27)) hide)
+    )
+    (property "Datasheet" "" (at 113.03 66.04 0)
+      (effects (font (size 1.27 1.27)) hide)
+    )

Commit message: Optimised IO routing, renumbered components
Parts:
- removed R11, R12: 100R, symbol Device:R
- added JP301: SolderJumper_2_Bridged, symbol Jumper:SolderJumper_2_Bridged
- added R305, R308, R309, R312, R313, R314, R315, R316: 100R, symbol Device:R
- renumbered J5 to J303, R2 to R301, R3 to R302, R4 to R303, R5 to R304, R9 to R306, R10 to R307, R7 to R310, R8 to R311
Connections:
- net +3V3: no longer J5.4 (Pin_4)
- net DONE: now also R312.2; no longer J8.2 (Pin_2)
- net INITN: now also R309.2; no longer J7.9 (Pin_9)
- net IO3: now also R308.2; no longer J8.5 (Pin_5)
- net IO6: now also J6.1 (Pin_1)
- net IO7: now also J6.2 (Pin_2)
- net IRQ_AT86RF215: now also R315.2; no longer J7.8 (Pin_8)
- net MCU_NRST: now also JP301.1 (A); no longer J5.3 (Pin_3)
- net at J8.3 (Pin_3): now also R313.1; no longer R306.1
- net at J8.4 (Pin_4): now also R314.1; no longer R307.1
- net at J7.5 (Pin_5): now also R305.1
- net at J7.6 (Pin_6): now also R306.1
- net at J7.7 (Pin_7): now also R307.1
- net SW_CTL2: now reaches J303.10 (Pin_10)
- net at J303.12 (Pin_12): now also R316.1
- net SW_CTL1: now reaches J303.8 (Pin_8)
- net PTT: now reaches J6.3 (Pin_3)
- net VIN_BAT renamed +BATT
- new net: J8.2 (Pin_2), R312.1
- new net: J8.5 (Pin_5), R315.1
- new net: J7.9 (Pin_9), R309.1
- new net: J7.8 (Pin_8), R308.1
- new net: J5.3 (Pin_3), JP301.2 (B)
- new net MAIN_KILL: R314.2
- new net PB_INT: R313.2
- new net PGOOD: R305.2
- new net RF_RST: R316.2
- no-connect marks 4 -> 14
Other:
- note added: "ADC1/ADC2/ADC3_IN11 (PC1)"
- note added: "I2C2_WS, TIM1_BKIN (PB12)"
- note added: "SPI1_MISO (PB4)"
- note added: "SPI1_MOSI (PB5)"
- note added: "SPI1_NSS (PA15)"
- note added: "SPI1_SCK (PA5)"
- note added: "USART3_CTS, TIM1_CH1N (PB13)"
- note added: "USART6_TX, TIM3/TIM8_CH1 (PC6)"
- note removed: "I2C2_WS, CAN2_RX, TIM1_BKIN (PB12)"
- note removed: "I2S2_CK, CAN2_TX, USART3_CTS, TIM1_CH1N (PB13)"
- note removed: "I2S2_SD, ADC1/ADC2/ADC3_IN11 (PC1)"
- note removed: "SPI1_MISO, TIM3_CH1 (PB4)"
- note removed: "SPI1_MOSI, TIM3_CH2, I2C1_SMBA, CAN2_RX (PB5)"
- note removed: "SPI1_NSS, TIM2_CH1/2_ETR (PA15)"
- note removed: "SPI1_SCK, TIM2/TIM8_CH1, ADC1/ADC2_IN5 (PA5)"
- note removed: "USART6_TX, I2S2_MCK, TIM3/TIM8_CH1 (PC6)"
- moved on the sheet: R301, R302, R303, R304, R306, R307
