File: OpenHT-RF/conn.kicad_sch (KiCad schematic)
At the start: 22 parts, among them J303 Conn_02x08_Odd_Even, J5 Conn_01x08, J6 Conn_01x06, J7 Conn_01x10, J8 Conn_01x08

Commit message: Updated power routing, added test points
Parts:
- added D301: BAT60A, symbol Device:D_Schottky
- added TP301, TP302, TP303, TP304, TP305, TP306, TP307, TP308: TestPoint, symbol Connector:TestPoint
Connections:
- net +BATT: now also D301.1 (K)
- net IO0: now also TP301.1
- net IO1: now also TP302.1
- net IO2: now also TP303.1
- net IO3: now also TP304.1
- net IO4: now also TP305.1
- net IO5: now also TP306.1
- net IO6: now also TP307.1
- net IO7: now also TP308.1
- net +5V: no longer names the net of J5.5 (Pin_5)
- net +5V: now also D301.2 (A)

Commit message: [WIP] symbol-footprint association
Parts:
- D301: footprint (none) -> Diode_SMD:D_SOD-323
- J303: footprint (none) -> Connector_PinSocket_2.54mm:PinSocket_2x08_P2.54mm_Vertical
- J5: footprint (none) -> Connector_PinHeader_2.54mm:PinHeader_1x08_P2.54mm_Vertical
- J6: footprint (none) -> Connector_PinHeader_2.54mm:PinHeader_1x06_P2.54mm_Vertical
- J7: footprint (none) -> Connector_PinSocket_2.54mm:PinSocket_1x10_P2.54mm_Vertical
- J8: footprint (none) -> Connector_PinSocket_2.54mm:PinSocket_1x08_P2.54mm_Vertical
- JP301: footprint (none) -> Jumper:SolderJumper-2_P1.3mm_Open_TrianglePad1.0x1.5mm
- R301, R302, R303, R304, R305, R306, R307, R308, R309, R310, R311, R312, R313, R314, R315, R316: footprint (none) -> Resistor_SMD:R_0402_1005Metric
- TP301, TP302, TP303, TP304, TP305, TP306, TP307, TP308: footprint (none) -> TestPoint:TestPoint_Loop_D2.50mm_Drill1.0mm
Changed lines of the file:
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@@
       (effects (font (size 1.27 1.27)) hide)
     )
-    (property "Footprint" "" (at 102.87 96.52 0)
+    (property "Footprint" "TestPoint:TestPoint_Loop_D2.50mm_Drill1.0mm" (at 102.87 96.52 0)
       (effects (font (size 1.27 1.27)) hide)
     )
@@
       (effects (font (size 1.27 1.27)))
     )
-    (property "Footprint" "" (at 173.99 102.87 0)
+    (property "Footprint" "Connector_PinSocket_2.54mm:PinSocket_1x08_P2.54mm_Vertical" (at 173.99 102.87 0)
       (effects (font (size 1.27 1.27)) hide)
     )
@@
       (effects (font (size 1.27 1.27)) hide)
     )
-    (property "Footprint" "" (at 102.87 99.06 0)
+    (property "Footprint" "TestPoint:TestPoint_Loop_D2.50mm_Drill1.0mm" (at 102.87 99.06 0)
       (effects (font (size 1.27 1.27)) hide)
     )
@@
       (effects (font (size 1.27 1.27)))
     )
-    (property "Footprint" "" (at 185.42 75.438 90)
+    (property "Footprint" "Resistor_SMD:R_0402_1005Metric" (at 185.42 75.438 90)
       (effects (font (size 1.27 1.27)) hide)
     )
@@
       (effects (font (size 1.27 1.27)))
     )
-    (property "Footprint" "" (at 107.95 69.85 0)
+    (property "Footprint" "Diode_SMD:D_SOD-323" (at 107.95 69.85 0)
       (effects (font (size 1.27 1.27)) hide)
     )
@@
       (effects (font (size 1.27 1.27)))
     )
-    (property "Footprint" "" (at 120.65 131.318 90)
+    (property "Footprint" "Resistor_SMD:R_0402_1005Metric" (at 120.65 131.318 90)
       (effects (font (size 1.27 1.27)) hide)
     )
@@
       (effects (font (size 1.27 1.27)) hide)
     )
-    (property "Footprint" "" (at 102.87 93.98 0)
+    (property "Footprint" "TestPoint:TestPoint_Loop_D2.50mm_Drill1.0mm" (at 102.87 93.98 0)
       (effects (font (size 1.27 1.27)) hide)
     )
@@
       (effects (font (size 1.27 1.27)))
     )
-    (property "Footprint" "" (at 198.12 136.398 90)
+    (property "Footprint" "Resistor_SMD:R_0402_1005Metric" (at 198.12 136.398 90)
       (effects (font (size 1.27 1.27)) hide)
     )
@@
       (effects (font (size 1.27 1.27)))
     )
-    (property "Footprint" "" (at 185.42 102.108 90)
+    (property "Footprint" "Resistor_SMD:R_0402_1005Metric" (at 185.42 102.108 90)
       (effects (font (size 1.27 1.27)) hide)
     )
@@
       (effects (font (size 1.27 1.27)))
     )
-    (property "Footprint" "" (at 185.42 80.518 90)
+    (property "Footprint" "Resistor_SMD:R_0402_1005Metric" (at 185.42 80.518 90)
       (effects (font (size 1.27 1.27)) hide)
     )
@@
       (effects (font (size 1.27 1.27)) hide)
     )
-    (property "Footprint" "" (at 102.87 101.6 0)
+    (property "Footprint" "TestPoint:TestPoint_Loop_D2.50mm_Drill1.0mm" (at 102.87 101.6 0)
       (effects (font (size 1.27 1.27)) hide)
     )
@@
       (effects (font (size 1.27 1.27)) hide)
     )
-    (property "Footprint" "" (at 102.87 88.9 0)
+    (property "Footprint" "TestPoint:TestPoint_Loop_D2.50mm_Drill1.0mm" (at 102.87 88.9 0)
       (effects (font (size 1.27 1.27)) hide)
     )
@@
       (effects (font (size 1.27 1.27)))
     )
-    (property "Footprint" "" (at 185.42 97.028 90)
+    (property "Footprint" "Resistor_SMD:R_0402_1005Metric" (at 185.42 97.028 90)
       (effects (font (size 1.27 1.27)) hide)
     )
@@
       (effects (font (size 1.27 1.27)))
     )
-    (property "Footprint" "" (at 172.72 68.58 0)
+    (property "Footprint" "Connector_PinSocket_2.54mm:PinSocket_1x10_P2.54mm_Vertical" (at 172.72 68.58 0)
       (effects (font (size 1.27 1.27)) hide)
     )
@@
       (effects (font (size 1.27 1.27)))
     )
-    (property "Footprint" "" (at 185.42 107.188 90)
+    (property "Footprint" "Resistor_SMD:R_0402_1005Metric" (at 185.42 107.188 90)
       (effects (font (size 1.27 1.27)) hide)
     )
@@
       (effects (font (size 1.27 1.27)))
     )
-    (property "Footprint" "" (at 120.65 136.398 90)
+    (property "Footprint" "Resistor_SMD:R_0402_1005Metric" (at 120.65 136.398 90)
       (effects (font (size 1.27 1.27)) hide)
     )
@@
       (effects (font (size 1.27 1.27)))
     )
-    (property "Footprint" "" (at 185.42 77.978 90)
+    (property "Footprint" "Resistor_SMD:R_0402_1005Metric" (at 185.42 77.978 90)
       (effects (font (size 1.27 1.27)) hide)
     )
@@
       (effects (font (size 1.27 1.27)))
     )
-    (property "Footprint" "" (at 185.42 72.898 90)
+    (property "Footprint" "Resistor_SMD:R_0402_1005Metric" (at 185.42 72.898 90)
       (effects (font (size 1.27 1.27)) hide)
     )
@@
       (effects (font (size 1.27 1.27)))
     )
-    (property "Footprint" "" (at 185.42 70.358 90)
+    (property "Footprint" "Resistor_SMD:R_0402_1005Metric" (at 185.42 70.358 90)
       (effects (font (size 1.27 1.27)) hide)
     )
@@
       (effects (font (size 1.27 1.27)))
     )
-    (property "Footprint" "" (at 151.13 129.54 0)
+    (property "Footprint" "Connector_PinSocket_2.54mm:PinSocket_2x08_P2.54mm_Vertical" (at 151.13 129.54 0)
       (effects (font (size 1.27 1.27)) hide)
     )
@@
       (effects (font (size 1.27 1.27)))
     )
-    (property "Footprint" "" (at 133.35 67.31 0)
+    (property "Footprint" "Connector_PinHeader_2.54mm:PinHeader_1x08_P2.54mm_Vertical" (at 133.35 67.31 0)
       (effects (font (size 1.27 1.27)) hide)
     )
@@
       (effects (font (size 1.27 1.27)))
     )
-    (property "Footprint" "" (at 132.08 97.79 0)
+    (property "Footprint" "Connector_PinHeader_2.54mm:PinHeader_1x06_P2.54mm_Vertical" (at 132.08 97.79 0)
       (effects (font (size 1.27 1.27)) hide)
     )
@@
       (effects (font (size 1.27 1.27)) hide)
     )
-    (property "Footprint" "" (at 102.87 91.44 0)
+    (property "Footprint" "TestPoint:TestPoint_Loop_D2.50mm_Drill1.0mm" (at 102.87 91.44 0)
       (effects (font (size 1.27 1.27)) hide)
     )
@@
       (effects (font (size 1.27 1.27)))
     )
-    (property "Footprint" "" (at 120.65 133.858 90)
+    (property "Footprint" "Resistor_SMD:R_0402_1005Metric" (at 120.65 133.858 90)
       (effects (font (size 1.27 1.27)) hide)
     )
@@
       (effects (font (size 1.27 1.27)))
     )
-    (property "Footprint" "" (at 185.42 104.648 90)
+    (property "Footprint" "Resistor_SMD:R_0402_1005Metric" (at 185.42 104.648 90)
       (effects (font (size 1.27 1.27)) hide)
     )
@@
       (effects (font (size 1.27 1.27)))
     )
-    (property "Footprint" "" (at 185.42 83.058 90)
+    (property "Footprint" "Resistor_SMD:R_0402_1005Metric" (at 185.42 83.058 90)
       (effects (font (size 1.27 1.27)) hide)
     )
@@
       (effects (font (size 1.27 1.27)) hide)
     )
-    (property "Footprint" "" (at 102.87 86.36 0)
+    (property "Footprint" "TestPoint:TestPoint_Loop_D2.50mm_Drill1.0mm" (at 102.87 86.36 0)
       (effects (font (size 1.27 1.27)) hide)
     )
@@
       (effects (font (size 1.27 1.27)))
     )
-    (property "Footprint" "" (at 185.42 99.568 90)
+    (property "Footprint" "Resistor_SMD:R_0402_1005Metric" (at 185.42 99.568 90)
       (effects (font (size 1.27 1.27)) hide)
     )
@@
       (effects (font (size 1.27 1.27)) hide)
     )
-    (property "Footprint" "" (at 102.87 83.82 0)
+    (property "Footprint" "TestPoint:TestPoint_Loop_D2.50mm_Drill1.0mm" (at 102.87 83.82 0)
       (effects (font (size 1.27 1.27)) hide)
     )
@@
       (effects (font (size 1.27 1.27)) hide)
     )
-    (property "Footprint" "" (at 116.84 64.77 0)
+    (property "Footprint" "Jumper:SolderJumper-2_P1.3mm_Open_TrianglePad1.0x1.5mm" (at 116.84 64.77 0)
       (effects (font (size 1.27 1.27)) hide)
     )
@@
       (effects (font (size 1.27 1.27)))
     )
-    (property "Footprint" "" (at 120.65 128.778 90)
-      (effects (font (size 1.27 1.27)) hide)
-    )
+    (property "Footprint" "Resistor_SMD:R_0402_1005Metric" (at 120.65 128.778 90)
+      (effects (font (size 1.27 1.27)) hide)
+    )

Commit message: Added mechanical holes
Parts:
- added H301, H302, H303, H304: M2.5, MountingHole:MountingHole_2.7mm_M2.5, symbol Mechanical:MountingHole
Changed lines of the file:
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@@
+    )
+  )
+  (symbol (lib_id "Mechanical:MountingHole") (at 57.15 166.37 0) (unit 1)
+    (in_bom yes) (on_board yes) (dnp no) (fields_autoplaced)
+    (property "Reference" "H302" (at 59.69 165.735 0)
+      (effects (font (size 1.27 1.27)) (justify left))
+    )
+    (property "Value" "M2.5" (at 59.69 168.275 0)
+      (effects (font (size 1.27 1.27)) (justify left))
+    )
+    (property "Footprint" "MountingHole:MountingHole_2.7mm_M2.5" (at 57.15 166.37 0)
+      (effects (font (size 1.27 1.27)) hide)
+    )
+    (property "Datasheet" "~" (at 57.15 166.37 0)
+      (effects (font (size 1.27 1.27)) hide)
+    )
+    (instances
+      (project "OpenHT-RF"
+        (path "/3c300b59-23ec-47f8-bb91-29ca34130bcf/1ac744a1-066f-4d1a-b0df-41e1d7c4818a"
+          (reference "H302") (unit 1)
+        )
+      )
     )
   )
@@
         (path "/3c300b59-23ec-47f8-bb91-29ca34130bcf/1ac744a1-066f-4d1a-b0df-41e1d7c4818a"
           (reference "R316") (unit 1)
+        )
+      )
+    )
+  )
+  (symbol (lib_id "Mechanical:MountingHole") (at 57.15 179.07 0) (unit 1)
+    (in_bom yes) (on_board yes) (dnp no) (fields_autoplaced)
+    (property "Reference" "H304" (at 59.69 178.435 0)
+      (effects (font (size 1.27 1.27)) (justify left))
+    )
+    (property "Value" "M2.5" (at 59.69 180.975 0)
+      (effects (font (size 1.27 1.27)) (justify left))
+    )
+    (property "Footprint" "MountingHole:MountingHole_2.7mm_M2.5" (at 57.15 179.07 0)
+      (effects (font (size 1.27 1.27)) hide)
+    )
+    (property "Datasheet" "~" (at 57.15 179.07 0)
+      (effects (font (size 1.27 1.27)) hide)
+    )
+    (instances
+      (project "OpenHT-RF"
+        (path "/3c300b59-23ec-47f8-bb91-29ca34130bcf/1ac744a1-066f-4d1a-b0df-41e1d7c4818a"
+          (reference "H304") (unit 1)
         )
       )
@@
     )
   )
+  (symbol (lib_id "Mechanical:MountingHole") (at 57.15 172.72 0) (unit 1)
+    (in_bom yes) (on_board yes) (dnp no) (fields_autoplaced)
+    (property "Reference" "H303" (at 59.69 172.085 0)
+      (effects (font (size 1.27 1.27)) (justify left))
+    )
+    (property "Value" "M2.5" (at 59.69 174.625 0)
+      (effects (font (size 1.27 1.27)) (justify left))
+    )
+    (property "Footprint" "MountingHole:MountingHole_2.7mm_M2.5" (at 57.15 172.72 0)
+      (effects (font (size 1.27 1.27)) hide)
+    )
+    (property "Datasheet" "~" (at 57.15 172.72 0)
+      (effects (font (size 1.27 1.27)) hide)
+    )
+    (instances
+      (project "OpenHT-RF"
+        (path "/3c300b59-23ec-47f8-bb91-29ca34130bcf/1ac744a1-066f-4d1a-b0df-41e1d7c4818a"
+          (reference "H303") (unit 1)
+        )
+      )
+    )
+  )
   (symbol (lib_id "Device:R") (at 185.42 76.2 90) (unit 1)
     (in_bom yes) (on_board yes) (dnp no)
@@
         )
       )
+    )
+  )
+  (symbol (lib_id "Mechanical:MountingHole") (at 57.15 160.02 0) (unit 1)
+    (in_bom yes) (on_board yes) (dnp no) (fields_autoplaced)
+    (property "Reference" "H301" (at 59.69 159.385 0)
+      (effects (font (size 1.27 1.27)) (justify left))
+    )
+    (property "Value" "M2.5" (at 59.69 161.925 0)
+      (effects (font (size 1.27 1.27)) (justify left))
+    )
+    (property "Footprint" "MountingHole:MountingHole_2.7mm_M2.5" (at 57.15 160.02 0)
+      (effects (font (size 1.27 1.27)) hide)
+    )
+    (property "Datasheet" "~" (at 57.15 160.02 0)
+      (effects (font (size 1.27 1.27)) hide)
+    )
+    (instances
+      (project "OpenHT-RF"
+        (path "/3c300b59-23ec-47f8-bb91-29ca34130bcf/1ac744a1-066f-4d1a-b0df-41e1d7c4818a"
+          (reference "H301") (unit 1)
+        )
+      )

Commit message: Fixed 3.3V power symbol
Use 3V3 everywhere instead of 3.3
Connections:
- net +3V3: no longer names the net of J303.1 (Pin_1)
Changed lines of the file:
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@@
-    (stroke (width 0) (type default))
-  )
-  (wire (pts (xy 144.78 121.92) (xy 146.05 121.92))
-    (stroke (width 0) (type default))
-  )
-  (wire (pts (xy 144.78 121.92) (xy 144.78 120.65))
     (stroke (width 0) (type default))
   )
@@
         )
       )
-    )
-  )
-  (symbol (lib_id "power:+3V3") (at 144.78 120.65 0) (unit 1)
-    (in_bom yes) (on_board yes) (dnp no) (fields_autoplaced)
-    (property "Reference" "#PWR0304" (at 144.78 124.46 0)
-      (effects (font (size 1.27 1.27)) hide)
-    )
-    (property "Value" "+3V3" (at 144.78 117.1481 0)
-      (effects (font (size 1.27 1.27)))
-    )
-    (property "Footprint" "" (at 144.78 120.65 0)
-      (effects (font (size 1.27 1.27)) hide)
-    )
-    (property "Datasheet" "" (at 144.78 120.65 0)
-      (effects (font (size 1.27 1.27)) hide)
-    )
-    (pin "1")
-    (instances
-      (project "OpenHT-RF"
-        (path "/3c300b59-23ec-47f8-bb91-29ca34130bcf/1ac744a1-066f-4d1a-b0df-41e1d7c4818a"
-          (reference "#PWR0304") (unit 1)
-        )
-      )

Commit message: Connectors adjustments
Parts:
- J7: footprint Connector_PinSocket_2.54mm:PinSocket_1x10_P2.54mm_Vertical -> Connector_PinHeader_2.54mm:PinHeader_1x10_P2.54mm_Vertical
- J8: footprint Connector_PinSocket_2.54mm:PinSocket_1x08_P2.54mm_Vertical -> Connector_PinHeader_2.54mm:PinHeader_1x08_P2.54mm_Vertical
Changed lines of the file:
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@@
       (effects (font (size 1.27 1.27)))
     )
-    (property "Footprint" "Connector_PinSocket_2.54mm:PinSocket_1x08_P2.54mm_Vertical" (at 173.99 102.87 0)
+    (property "Footprint" "Connector_PinHeader_2.54mm:PinHeader_1x08_P2.54mm_Vertical" (at 173.99 102.87 0)
       (effects (font (size 1.27 1.27)) hide)
     )
@@
       (effects (font (size 1.27 1.27)))
     )
-    (property "Footprint" "Connector_PinSocket_2.54mm:PinSocket_1x10_P2.54mm_Vertical" (at 172.72 68.58 0)
-      (effects (font (size 1.27 1.27)) hide)
-    )
+    (property "Footprint" "Connector_PinHeader_2.54mm:PinHeader_1x10_P2.54mm_Vertical" (at 172.72 68.58 0)
+      (effects (font (size 1.27 1.27)) hide)
+    )

Commit message: Rearanged IOs
Connections:
- net INITN: now also R310.2; no longer R309.2
- net SPI_NSS2: now also R309.2; no longer R310.2
Changed lines of the file:
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@@
     (effects (font (size 1.27 1.27)) (justify left))
   )
-  (hierarchical_label "SPI_NSS2" (shape output) (at 193.04 81.28 0) (fields_autoplaced)
+  (hierarchical_label "SPI_NSS2" (shape output) (at 193.04 78.74 0) (fields_autoplaced)
     (effects (font (size 1.27 1.27)) (justify left))
   )
@@
     (effects (font (size 1.27 1.27)) (justify left))
   )
-  (hierarchical_label "INITN" (shape bidirectional) (at 193.04 78.74 0) (fields_autoplaced)
-    (effects (font (size 1.27 1.27)) (justify left))
-  )
   (hierarchical_label "DONE" (shape bidirectional) (at 191.77 97.79 0) (fields_autoplaced)
     (effects (font (size 1.27 1.27)) (justify left))
@@
     (effects (font (size 1.27 1.27)) (justify left))
   )
+  (hierarchical_label "INITN" (shape bidirectional) (at 193.04 81.28 0) (fields_autoplaced)
+    (effects (font (size 1.27 1.27)) (justify left))
+  )

Commit message: [WIP] Layout
Flipped the content upside down for the SMA connector. Reorganized GPIOs. RF routing started.
Parts:
- removed R312: 100R, Resistor_SMD:R_0402_1005Metric, symbol Device:R
Connections:
- net DONE: now also R305.2
- net INITN: now also R311.2; no longer R310.2
- net IO2: now also J8.1 (Pin_1); no longer J8.6 (Pin_6)
- net IO3: now also J7.10 (Pin_10); no longer R308.2
- net IO4: now also J7.8 (Pin_8); no longer R307.2
- net IO5: now also R307.2; no longer R306.2
- net IO6: now also R306.2; no longer J6.1 (Pin_1)
- net IO7: now also R308.2; no longer J6.2 (Pin_2)
- net PGOOD: now also R301.2; no longer R305.2
- net PROGRAMN: now also R310.2; no longer R311.2
- net PTT: now also J6.5 (Pin_5); no longer J6.3 (Pin_3)
- net SPI_MISO: now also J303.5 (Pin_5); no longer R301.1
- net SPI_NSS1: now also R309.2; no longer R304.1
- net SPI_NSS2: now also R304.1; no longer R309.2
- net at R311.1: now also J6.4 (Pin_4); no longer J8.1 (Pin_1)
- net at R310.1: now also J6.3 (Pin_3); no longer J7.10 (Pin_10)
- net at J7.5 (Pin_5): now also R308.1; no longer R305.1
- new net: J6.1 (Pin_1), R301.1
- new net: J6.2 (Pin_2), R305.1
- no-connect marks 14 -> 15
Other:
- moved on the sheet: R308, R310, R311, TP301, TP302, TP303, TP304, TP305, TP306, TP307, TP308

Commit message: Added battery measurement pin
Parts:
- added C301: 100nF, Capacitor_SMD:C_0402_1005Metric, symbol Device:C
- added R312: 200kR, Resistor_SMD:R_0402_1005Metric, symbol Device:R
- added R317: 100kR, Resistor_SMD:R_0402_1005Metric, symbol Device:R
Connections:
- net +BATT: no longer J5.8 (Pin_8)
- net GND: now also C301.2, R317.2
- net at J6.6 (Pin_6): now also C301.1, R312.2, R317.1
- new net VDD: J5.8 (Pin_8), R312.1
- no-connect marks 15 -> 14
Other:
- moved on the sheet: TP301, TP302, TP303, TP304, TP305, TP306, TP307, TP308
