File: OpenHT-RF/conn.kicad_sch (KiCad schematic)
At the start: 37 parts, among them J303 Conn_02x08_Odd_Even, J5 Conn_01x08, J6 Conn_01x06, J7 Conn_01x10, J8 Conn_01x08

Commit message: Various schematic updates
Edited IO names, updated load switch symbol, swapped RF switch inputs
Connections:
- net IO4: now also R307.2; no longer J7.8 (Pin_8)
- net IO5: now also R306.2; no longer R307.2
- net IO6: now also R308.2; no longer R306.2
- net IO7: no longer R308.2
- new net FPGA_RST: J7.8 (Pin_8)
Changed lines of the file:
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@@
     (effects (font (size 1.27 1.27)) (justify right))
   )
-  (hierarchical_label "IO5" (shape bidirectional) (at 193.04 73.66 0) (fields_autoplaced)
+  (hierarchical_label "IO4" (shape bidirectional) (at 193.04 73.66 0) (fields_autoplaced)
     (effects (font (size 1.27 1.27)) (justify left))
   )
@@
     (effects (font (size 1.27 1.27)) (justify left))
   )
-  (hierarchical_label "IO7" (shape bidirectional) (at 193.04 68.58 0) (fields_autoplaced)
+  (hierarchical_label "IO6" (shape bidirectional) (at 193.04 68.58 0) (fields_autoplaced)
     (effects (font (size 1.27 1.27)) (justify left))
   )
@@
     (effects (font (size 1.27 1.27)) (justify left))
   )
-  (hierarchical_label "IO4" (shape bidirectional) (at 193.04 76.2 0) (fields_autoplaced)
+  (hierarchical_label "FPGA_RST" (shape bidirectional) (at 193.04 76.2 0) (fields_autoplaced)
     (effects (font (size 1.27 1.27)) (justify left))
   )
@@
     (effects (font (size 1.27 1.27)) (justify left))
   )
-  (hierarchical_label "IO6" (shape bidirectional) (at 193.04 71.12 0) (fields_autoplaced)
+  (hierarchical_label "IO5" (shape bidirectional) (at 193.04 71.12 0) (fields_autoplaced)
     (effects (font (size 1.27 1.27)) (justify left))
   )

Commit message: Various updates
Updated some nets to ease up routing
Updated testpoints to smaller size
Added DNP capacitor next to RF switch
Parts:
- TP301, TP302, TP303, TP304, TP305, TP306, TP307, TP308: footprint TestPoint:TestPoint_Loop_D2.50mm_Drill1.0mm -> Connector_Pin:Pin_D0.7mm_L6.5mm_W1.8mm_FlatFork
Connections:
- net IO7 is gone; now on net FPGA_RST: TP308.1
Changed lines of the file:
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@@
     (effects (font (size 1.27 1.27)) (justify right))
+  )
+  (hierarchical_label "FPGA_RST" (shape bidirectional) (at 63.5 105.41 0) (fields_autoplaced)
+    (effects (font (size 1.27 1.27)) (justify left))
   )
   (hierarchical_label "PTT" (shape output) (at 123.19 102.87 180) (fields_autoplaced)
@@
     (effects (font (size 1.27 1.27)) (justify right))
   )
-  (hierarchical_label "IO7" (shape bidirectional) (at 63.5 105.41 0) (fields_autoplaced)
-    (effects (font (size 1.27 1.27)) (justify left))
-  )
   (hierarchical_label "RF_RST" (shape input) (at 203.2 134.62 0) (fields_autoplaced)
     (effects (font (size 1.27 1.27)) (justify left))
@@
       (effects (font (size 1.27 1.27)) hide)
     )
-    (property "Footprint" "TestPoint:TestPoint_Loop_D2.50mm_Drill1.0mm" (at 59.69 95.25 0)
+    (property "Footprint" "Connector_Pin:Pin_D0.7mm_L6.5mm_W1.8mm_FlatFork" (at 59.69 95.25 0)
       (effects (font (size 1.27 1.27)) hide)
     )
@@
       (effects (font (size 1.27 1.27)) hide)
     )
-    (property "Footprint" "TestPoint:TestPoint_Loop_D2.50mm_Drill1.0mm" (at 59.69 97.79 0)
+    (property "Footprint" "Connector_Pin:Pin_D0.7mm_L6.5mm_W1.8mm_FlatFork" (at 59.69 97.79 0)
       (effects (font (size 1.27 1.27)) hide)
     )
@@
       (effects (font (size 1.27 1.27)) hide)
     )
-    (property "Footprint" "TestPoint:TestPoint_Loop_D2.50mm_Drill1.0mm" (at 59.69 92.71 0)
+    (property "Footprint" "Connector_Pin:Pin_D0.7mm_L6.5mm_W1.8mm_FlatFork" (at 59.69 92.71 0)
       (effects (font (size 1.27 1.27)) hide)
     )
@@
       (effects (font (size 1.27 1.27)) hide)
     )
-    (property "Footprint" "TestPoint:TestPoint_Loop_D2.50mm_Drill1.0mm" (at 59.69 100.33 0)
+    (property "Footprint" "Connector_Pin:Pin_D0.7mm_L6.5mm_W1.8mm_FlatFork" (at 59.69 100.33 0)
       (effects (font (size 1.27 1.27)) hide)
     )
@@
       (effects (font (size 1.27 1.27)) hide)
     )
-    (property "Footprint" "TestPoint:TestPoint_Loop_D2.50mm_Drill1.0mm" (at 59.69 87.63 0)
+    (property "Footprint" "Connector_Pin:Pin_D0.7mm_L6.5mm_W1.8mm_FlatFork" (at 59.69 87.63 0)
       (effects (font (size 1.27 1.27)) hide)
     )
@@
       (effects (font (size 1.27 1.27)) hide)
     )
-    (property "Footprint" "TestPoint:TestPoint_Loop_D2.50mm_Drill1.0mm" (at 59.69 90.17 0)
+    (property "Footprint" "Connector_Pin:Pin_D0.7mm_L6.5mm_W1.8mm_FlatFork" (at 59.69 90.17 0)
       (effects (font (size 1.27 1.27)) hide)
     )
@@
       (effects (font (size 1.27 1.27)) hide)
     )
-    (property "Footprint" "TestPoint:TestPoint_Loop_D2.50mm_Drill1.0mm" (at 59.69 85.09 0)
+    (property "Footprint" "Connector_Pin:Pin_D0.7mm_L6.5mm_W1.8mm_FlatFork" (at 59.69 85.09 0)
       (effects (font (size 1.27 1.27)) hide)
     )
@@
       (effects (font (size 1.27 1.27)) hide)
     )
-    (property "Footprint" "TestPoint:TestPoint_Loop_D2.50mm_Drill1.0mm" (at 59.69 82.55 0)
-      (effects (font (size 1.27 1.27)) hide)
-    )
+    (property "Footprint" "Connector_Pin:Pin_D0.7mm_L6.5mm_W1.8mm_FlatFork" (at 59.69 82.55 0)
+      (effects (font (size 1.27 1.27)) hide)
+    )

Commit message: BOM updates
Parts:
- D301: MPN (none) -> BAT60AE6327HTSA1
- H301, H302, H303, H304, JP301, TP301, TP302, TP303, TP304, TP305, TP306, TP307, TP308: now left out of the parts list
- J303, J5, J6, J7, J8: Manual_Placement (none) -> 1
Changed lines of the file:
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@@
   )
   (symbol (lib_id "Connector:TestPoint") (at 59.69 100.33 90) (unit 1)
-    (in_bom yes) (on_board yes) (dnp no)
+    (in_bom no) (on_board yes) (dnp no)
     (property "Reference" "TP306" (at 52.07 100.33 90)
       (effects (font (size 1.27 1.27)))
@@
     )
     (property "Datasheet" "~" (at 173.99 102.87 0)
+      (effects (font (size 1.27 1.27)) hide)
+    )
+    (property "Manual_Placement" "1" (at 173.99 102.87 0)
       (effects (font (size 1.27 1.27)) hide)
     )
@@
   )
   (symbol (lib_id "Connector:TestPoint") (at 59.69 102.87 90) (unit 1)
-    (in_bom yes) (on_board yes) (dnp no)
+    (in_bom no) (on_board yes) (dnp no)
     (property "Reference" "TP307" (at 52.07 102.87 90)
       (effects (font (size 1.27 1.27)))
@@
   )
   (symbol (lib_id "Mechanical:MountingHole") (at 57.15 166.37 0) (unit 1)
-    (in_bom yes) (on_board yes) (dnp no) (fields_autoplaced)
+    (in_bom no) (on_board yes) (dnp no) (fields_autoplaced)
     (property "Reference" "H302" (at 59.69 165.735 0)
       (effects (font (size 1.27 1.27)) (justify left))
@@
       (effects (font (size 1.27 1.27)) hide)
     )
+    (property "MPN" "BAT60AE6327HTSA1" (at 107.95 69.85 0)
+      (effects (font (size 1.27 1.27)) hide)
+    )
     (pin "1")
     (pin "2")
@@
   )
   (symbol (lib_id "Connector:TestPoint") (at 59.69 97.79 90) (unit 1)
-    (in_bom yes) (on_board yes) (dnp no)
+    (in_bom no) (on_board yes) (dnp no)
     (property "Reference" "TP305" (at 52.07 97.79 90)
       (effects (font (size 1.27 1.27)))
@@
   )
   (symbol (lib_id "Mechanical:MountingHole") (at 57.15 179.07 0) (unit 1)
-    (in_bom yes) (on_board yes) (dnp no) (fields_autoplaced)
+    (in_bom no) (on_board yes) (dnp no) (fields_autoplaced)
     (property "Reference" "H304" (at 59.69 178.435 0)
       (effects (font (size 1.27 1.27)) (justify left))
@@
   )
   (symbol (lib_id "Connector:TestPoint") (at 59.69 105.41 90) (unit 1)
-    (in_bom yes) (on_board yes) (dnp no)
+    (in_bom no) (on_board yes) (dnp no)
     (property "Reference" "TP308" (at 52.07 105.41 90)
       (effects (font (size 1.27 1.27)))
@@
   )
   (symbol (lib_id "Connector:TestPoint") (at 59.69 92.71 90) (unit 1)
-    (in_bom yes) (on_board yes) (dnp no)
+    (in_bom no) (on_board yes) (dnp no)
     (property "Reference" "TP303" (at 52.07 92.71 90)
       (effects (font (size 1.27 1.27)))
@@
     )
     (property "Datasheet" "~" (at 172.72 68.58 0)
+      (effects (font (size 1.27 1.27)) hide)
+    )
+    (property "Manual_Placement" "1" (at 172.72 68.58 0)
       (effects (font (size 1.27 1.27)) hide)
     )
@@
   )
   (symbol (lib_id "Mechanical:MountingHole") (at 57.15 172.72 0) (unit 1)
-    (in_bom yes) (on_board yes) (dnp no) (fields_autoplaced)
+    (in_bom no) (on_board yes) (dnp no) (fields_autoplaced)
     (property "Reference" "H303" (at 59.69 172.085 0)
       (effects (font (size 1.27 1.27)) (justify left))
@@
     )
     (property "Datasheet" "~" (at 151.13 129.54 0)
+      (effects (font (size 1.27 1.27)) hide)
+    )
+    (property "Manual_Placement" "1" (at 151.13 129.54 0)
       (effects (font (size 1.27 1.27)) hide)
     )
@@
       (effects (font (size 1.27 1.27)) hide)
     )
+    (property "Manual_Placement" "1" (at 133.35 67.31 0)
+      (effects (font (size 1.27 1.27)) hide)
+    )
     (pin "1")
     (pin "2")
@@
       (effects (font (size 1.27 1.27)) hide)
     )
+    (property "Manual_Placement" "1" (at 132.08 97.79 0)
+      (effects (font (size 1.27 1.27)) hide)
+    )
     (pin "1")
     (pin "2")
@@
   )
   (symbol (lib_id "Mechanical:MountingHole") (at 57.15 160.02 0) (unit 1)
-    (in_bom yes) (on_board yes) (dnp no) (fields_autoplaced)
+    (in_bom no) (on_board yes) (dnp no) (fields_autoplaced)
     (property "Reference" "H301" (at 59.69 159.385 0)
       (effects (font (size 1.27 1.27)) (justify left))
@@
   )
   (symbol (lib_id "Connector:TestPoint") (at 59.69 95.25 90) (unit 1)
-    (in_bom yes) (on_board yes) (dnp no)
+    (in_bom no) (on_board yes) (dnp no)
     (property "Reference" "TP304" (at 52.07 95.25 90)
       (effects (font (size 1.27 1.27)))
@@
   )
   (symbol (lib_id "Connector:TestPoint") (at 59.69 90.17 90) (unit 1)
-    (in_bom yes) (on_board yes) (dnp no)
+    (in_bom no) (on_board yes) (dnp no)
     (property "Reference" "TP302" (at 52.07 90.17 90)
       (effects (font (size 1.27 1.27)))
@@
   )
   (symbol (lib_id "Connector:TestPoint") (at 59.69 87.63 90) (unit 1)
-    (in_bom yes) (on_board yes) (dnp no)
+    (in_bom no) (on_board yes) (dnp no)
     (property "Reference" "TP301" (at 52.07 87.63 90)
       (effects (font (size 1.27 1.27)))
@@
   )
   (symbol (lib_id "Jumper:SolderJumper_2_Bridged") (at 116.84 64.77 0) (unit 1)
-    (in_bom yes) (on_board yes) (dnp no)
+    (in_bom no) (on_board yes) (dnp no)
     (property "Reference" "JP301" (at 116.84 62.23 0)
       (effects (font (size 1.27 1.27)))
