File: OpenHT-RF/rf.kicad_sch (KiCad schematic)
At the start: 2 parts, among them IC2 AT86RF215-ZU, J6 Conn_Coaxial

Commit message: lfcn-490 filter added
Parts:
- added FL1: LFCN-490, Filter:Filter_Mini-Circuits_FV1206, symbol RF_Filter:LFCN-490
Connections:
- net at J6.1 (In): now also FL1.3 (OUT)
- net GND: now reaches J6.2 (Ext)
- net GND: now also FL1.2 (GND), FL1.4 (GND)
Changed lines of the file:
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@@
     (comment 1 "Authors: Wojciech SP5WWP, Leo Hofer")
+  )
+  (wire (pts (xy 219.71 80.01) (xy 227.33 80.01))
+    (stroke (width 0) (type default))
+  )
+  (wire (pts (xy 209.55 90.17) (xy 209.55 91.44))
+    (stroke (width 0) (type default))
+  )
+  (wire (pts (xy 232.41 85.09) (xy 232.41 86.36))
+    (stroke (width 0) (type default))
+  )
+  (symbol (lib_id "RF_Filter:LFCN-490") (at 209.55 80.01 0) (unit 1)
+    (in_bom yes) (on_board yes) (dnp no) (fields_autoplaced)
+    (property "Reference" "FL1" (at 209.55 68.58 0)
+      (effects (font (size 1.27 1.27)))
+    )
+    (property "Value" "LFCN-490" (at 209.55 71.12 0)
+      (effects (font (size 1.27 1.27)))
+    )
+    (property "Footprint" "Filter:Filter_Mini-Circuits_FV1206" (at 209.55 67.31 0)
+      (effects (font (size 1.27 1.27)) hide)
+    )
+    (property "Datasheet" "https://www.minicircuits.com/pdfs/LFCN-490+.pdf" (at 209.55 80.01 0)
+      (effects (font (size 1.27 1.27)) hide)
+    )
+    (pin "1")
+    (pin "2")
+    (pin "3")
+    (pin "4")
+    (instances
+      (project "OpenHT-RF"
+        (path "/3c300b59-23ec-47f8-bb91-29ca34130bcf/e3bba2b3-d2df-4b56-8e13-359b6c4f2426"
+          (reference "FL1") (unit 1)
+        )
+      )
+    )
   )
   (symbol (lib_id "Connector:Conn_Coaxial") (at 232.41 80.01 0) (unit 1)
@@
         (path "/3c300b59-23ec-47f8-bb91-29ca34130bcf/e3bba2b3-d2df-4b56-8e13-359b6c4f2426"
           (reference "J6") (unit 1)
+        )
+      )
+    )
+  )
+  (symbol (lib_id "power:GND") (at 232.41 86.36 0) (unit 1)
+    (in_bom yes) (on_board yes) (dnp no) (fields_autoplaced)
+    (property "Reference" "#PWR03" (at 232.41 92.71 0)
+      (effects (font (size 1.27 1.27)) hide)
+    )
+    (property "Value" "GND" (at 232.41 91.44 0)
+      (effects (font (size 1.27 1.27)))
+    )
+    (property "Footprint" "" (at 232.41 86.36 0)
+      (effects (font (size 1.27 1.27)) hide)
+    )
+    (property "Datasheet" "" (at 232.41 86.36 0)
+      (effects (font (size 1.27 1.27)) hide)
+    )
+    (pin "1")
+    (instances
+      (project "OpenHT-RF"
+        (path "/3c300b59-23ec-47f8-bb91-29ca34130bcf/e3bba2b3-d2df-4b56-8e13-359b6c4f2426"
+          (reference "#PWR03") (unit 1)
         )
       )
@@
         )
       )
+    )
+  )
+  (symbol (lib_id "power:GND") (at 209.55 91.44 0) (unit 1)
+    (in_bom yes) (on_board yes) (dnp no) (fields_autoplaced)
+    (property "Reference" "#PWR04" (at 209.55 97.79 0)
+      (effects (font (size 1.27 1.27)) hide)
+    )
+    (property "Value" "GND" (at 209.55 96.52 0)
+      (effects (font (size 1.27 1.27)))
+    )
+    (property "Footprint" "" (at 209.55 91.44 0)
+      (effects (font (size 1.27 1.27)) hide)
+    )
+    (property "Datasheet" "" (at 209.55 91.44 0)
+      (effects (font (size 1.27 1.27)) hide)
+    )
+    (pin "1")
+    (instances
+      (project "OpenHT-RF"
+        (path "/3c300b59-23ec-47f8-bb91-29ca34130bcf/e3bba2b3-d2df-4b56-8e13-359b6c4f2426"
+          (reference "#PWR04") (unit 1)
+        )
+      )

Commit message: Updated FPGA, RF and connectors sheets [WIP]
Parts:
- added C27, C28, C29: 100p, symbol Device:C
- added C30: 220p, symbol Device:C
- added C31: 81p, symbol Device:C
- added FL2: LFCN-2500+, Filter:Filter_Mini-Circuits_FV1206, symbol RF_Filter:LFCN-490
- added IC3: RFSW8008TR7, RFSW8008TR7, symbol RFSW8008TR7:RFSW8008TR7
- added R3: 100k, symbol Device:R
- added X1: 26 MHz, symbol Oscillator:DFA-S2
- FL1: value LFCN-490 -> LFCN-490+
Connections:
- net GND: now also IC2.10 (AVSS_4), IC2.16 (AVSS_5), IC2.19 (AVSS_6), IC2.20 (DVSS_1), IC2.23 (DVSS_2), IC2.24 (DVSS_3), IC2.3 (AVSS_1), IC2.32 (DVSS_4), IC2.38 (DVSS_5), IC2.45 (AVSS_7), IC2.48 (AVSS_8), IC2.49 (EP), IC2.6 (AVSS_2), IC2.7 (AVSS_3), C30.1, C31.1, FL2.2 (GND), FL2.4 (GND), IC3.5 (GND), R3.1, X1.2 (GND)
- net at FL1.3 (OUT): now also C27.1; no longer J6.1 (In)
- net at IC2.17 (TCXO): now also X1.3 (OUT)
- net at IC2.18 (XTAL2): now also R3.2
- net LVDS_TXCLK_N: now reaches IC2.25 (TXCLKN)
- net LVDS_TXCLK_P: now reaches IC2.26 (TXCLKP)
- net LVDS_TX_N: now reaches IC2.27 (TXDN)
- net LVDS_TX_P: now reaches IC2.28 (TXDP)
- net LVDS_RX09_N: now reaches IC2.30 (RXDN09)
- net LVDS_RX09_P: now reaches IC2.31 (RXDP09)
- net LVDS_RXCLK_N: now reaches IC2.33 (RXCLKN)
- net LVDS_RXCLK_P: now reaches IC2.34 (RXCLKP)
- net LVDS_RX24_N: now reaches IC2.35 (RXDN24)
- net LVDS_RX24_P: now reaches IC2.36 (RXDP24)
- net AT86RF215_IRQ: now reaches IC2.40 (IRQ)
- net S_SPI_SCLK: now reaches IC2.41 (SCLK)
- net S_SPI_SELN: now reaches IC2.42 (SELN)
- net S_SPI_MOSI: now reaches IC2.43 (MOSI)
- net S_SPI_MISO: now reaches IC2.44 (MISO)
- new net: C28.1, FL2.3 (OUT)
- new net: C29.1, IC3.2 (ANT)
- new net: C28.2, IC3.4 (RF1)
- new net: C27.2, IC3.6 (RF2)
- new net: C29.2, J6.1 (In)
- new net +3V3: IC3.3 (VDD), X1.4 (V+)
- new net VCTRL1: C30.2, IC3.7 (VCTRL1)
- new net VCTRL2: C31.2, IC3.1 (VCTRL2)
- no-connect marks 0 -> 6

Commit message: Updated FPGA, RF and connectors sheets [WIP]
Parts:
- added C32, C33, C34: 100nF, symbol Device:C
- added FB5: FerriteBead_Small, symbol Device:FerriteBead_Small
Connections:
- net GND: now also C32.2, C33.2, C34.2
- net ~{RESET}: now reaches IC2.13 (RSTN)
- net at IC2.14 (AVDD0): now also C34.1
- net DEVDD: now reaches IC2.15 (EVDD_1)
- net DEVDD: now also IC2.21 (DEVDD_1), IC2.29 (DEVDD_2), IC2.39 (DEVDD_3), IC2.46 (EVDD_2), FB5.2
- net CLK_OUT: now reaches IC2.22 (CLKO)
- net at IC2.37 (DVDD): now also C32.1
- net at IC2.47 (AVDD1): now also C33.1
- new net +3.3V: FB5.1
Other:
- moved on the sheet: R3, X1

Commit message: Updated RF schematic
Parts:
- removed C27, C28, C29: 100p, symbol Device:C
- removed C30: 220p, symbol Device:C
- removed C31: 81p, symbol Device:C
- removed IC2: AT86RF215-ZU, QFN50P700X700X90-49N-D, symbol AT86RF215-ZU:AT86RF215-ZU
- removed IC3: RFSW8008TR7, RFSW8008TR7, symbol RFSW8008TR7:RFSW8008TR7
- removed X1: 26 MHz, symbol Oscillator:DFA-S2
- added C35, C36, C37: 100nF, symbol Device:C
- added C38: 82pF, symbol Device:C
- added C39: 220pF, symbol Device:C
- added C40, C41, C42: 100pF, symbol Device:C
- added J7, J8: Conn_01x02, symbol Connector_Generic:Conn_01x02
- added R13: 10kR, symbol Device:R
- added SW1: ~, M17_misc_active:RFSW8008, symbol M17_RF:RFSW8008
- added U2: ~, M17_QFN:VQFN-48-1EP_7x7mm_P0.5mm_EP5.6x5.6mm, symbol M17_RF:AT86RF215
- added X1: ~, M17_misc_active:ECS-TXO-20CSMV, symbol M17_misc_active:ECS-TXO-20CSMV
- C33: value 100nF -> 1nF
- C34: value 100nF -> 10pF
Connections:
- net +3V3: now also C32.1, SW1.3 (VDD), X1.4 (VCC)
- net AT86RF215_IRQ: now also U2.40 (IRQ)
- net CLK_OUT: now also U2.22 (CLKO)
- net DEVDD: now also U2.15 (EVDD), U2.21 (DEVDD), U2.29 (DEVDD), U2.39 (DEVDD), U2.46 (EVDD)
- net GND: now also C35.2, C36.2, C37.2, C38.2, C39.2, R13.2, SW1.5 (GND), U2.10 (AVSS), U2.16 (AVSS), U2.19 (AVSS), U2.20 (DVSS), U2.23 (DVSS), U2.24 (DVSS), U2.3 (AVSS), U2.32 (DVSS), U2.38 (DVSS), U2.45 (AVSS), U2.48 (AVSS), U2.49 (AVSS), U2.6 (AVSS), U2.7 (AVSS), X1.1 (GND), X1.2 (GND); no longer C33.2
- net LVDS_RX09_N: now also U2.30 (RXDN09)
- net LVDS_RX09_P: now also U2.31 (RXDP09)
- net LVDS_RX24_N: now also U2.35 (RXDN24)
- net LVDS_RX24_P: now also U2.36 (RXDP24)
- net LVDS_RXCLK_N: now also U2.33 (RXCLKN)
- net LVDS_RXCLK_P: now also U2.34 (RXCLKP)
- net LVDS_TXCLK_N: now also U2.25 (TXCLKN)
- net LVDS_TXCLK_P: now also U2.26 (TXCLKP)
- net LVDS_TX_N: now also U2.27 (TXDN)
- net LVDS_TX_P: now also U2.28 (TXDP)
- net S_SPI_MISO: now also U2.44 (MISO)
- net S_SPI_MOSI: now also U2.43 (MOSI)
- net S_SPI_SCLK: now also U2.41 (SCLK)
- net S_SPI_SELN: now also U2.42 (~{SELN})
- net ~{RESET}: now also U2.13 (~{RSTN})
- net at C34.1: now also C33.2, R13.1, U2.17 (TCXO)
- net at FL1.3 (OUT): now also C41.1
- net at R3.2: now also U2.18 (XTAL2)
- net at FL2.3 (OUT): now also C42.1
- net at J6.1 (In): now also C40.2
- net at C33.1: now also X1.3 (OUT)
- new net: J7.1 (Pin_1), U2.1 (FEA24)
- new net: J8.1 (Pin_1), U2.11 (FEA09)
- new net: J8.2 (Pin_2), U2.12 (FEB09)
- new net: C36.1, U2.14 (AVDD0)
- new net: J7.2 (Pin_2), U2.2 (FEB24)
- new net: C35.1, U2.37 (DVDD)
- new net: C37.1, U2.47 (AVDD1)
- new net: C42.2, SW1.4 (RF1)
- new net: C41.2, SW1.6 (RF2)
- new net: C40.1, SW1.2 (ANT)
- new net RFN09: U2.9 (RFN09)
- new net RFN24: U2.5 (RFN24)
- new net RFP09: U2.8 (RFP09)
- new net RFP24: U2.4 (RFP24)
- new net SW_CTL1: C39.1, SW1.7 (CTL1)
- new net SW_CTL2: C38.1, SW1.1 (CTL2)
- no-connect marks 6 -> 0
Other:
- moved on the sheet: FL1, FL2

Commit message: Updated M17_kicad_library
Parts:
- SW?: renamed from SW1; value ~ -> RFSW8008
- U?: renamed from U2; value ~ -> AT86RF215
- X1: value ~ -> ECS-TXO-20CSMV
Changed lines of the file:
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@@
     )
   )
-  (symbol (lib_id "M17_RF:AT86RF215") (at 160.02 68.58 0) (unit 1)
-    (in_bom yes) (on_board yes) (dnp no)
-    (property "Reference" "U2" (at 132.08 40.64 0)
-      (effects (font (size 1.27 1.27)))
-    )
-    (property "Value" "~" (at 120.784 73.3058 0)
-      (effects (font (size 1.27 1.27)))
-    )
-    (property "Footprint" "M17_QFN:VQFN-48-1EP_7x7mm_P0.5mm_EP5.6x5.6mm" (at 120.784 73.3058 0)
-      (effects (font (size 1.27 1.27)) hide)
-    )
-    (property "Datasheet" "https://ww1.microchip.com/downloads/aemDocuments/documents/OTH/ProductDocuments/DataSheets/Atmel-42415-WIRELESS-AT86RF215_Datasheet.pdf#%5B%7B%22num%22%3A91%2C%22gen%22%3A0%7D%2C%7B%22name%22%3A%22XYZ%22%7D%2C33%2C245%2C0%5D" (at 120.784 73.3058 0)
+  (symbol (lib_id "M17_RF:AT86RF215") (at 130.81 41.91 0) (unit 1)
+    (in_bom yes) (on_board yes) (dnp no)
+    (property "Reference" "U?" (at 130.81 40.64 0)
+      (effects (font (size 1.27 1.27)))
+    )
+    (property "Value" "AT86RF215" (at 160.02 68.58 0)
+      (effects (font (size 1.27 1.27)))
+    )
+    (property "Footprint" "M17_QFN:VQFN-48-1EP_7x7mm_P0.5mm_EP5.6x5.6mm" (at 130.81 41.91 0)
+      (effects (font (size 1.27 1.27)) hide)
+    )
+    (property "Datasheet" "https://ww1.microchip.com/downloads/aemDocuments/documents/OTH/ProductDocuments/DataSheets/Atmel-42415-WIRELESS-AT86RF215_Datasheet.pdf#%5B%7B%22num%22%3A91%2C%22gen%22%3A0%7D%2C%7B%22name%22%3A%22XYZ%22%7D%2C33%2C245%2C0%5D" (at 130.81 41.91 0)
       (effects (font (size 1.27 1.27)) hide)
     )
@@
       (project "OpenHT-RF"
         (path "/3c300b59-23ec-47f8-bb91-29ca34130bcf/e3bba2b3-d2df-4b56-8e13-359b6c4f2426"
-          (reference "U2") (unit 1)
+          (reference "U?") (unit 1)
         )
       )
@@
     )
   )
-  (symbol (lib_id "M17_misc_active:ECS-TXO-20CSMV") (at 66.04 68.58 0) (unit 1)
-    (in_bom yes) (on_board yes) (dnp no) (fields_autoplaced)
-    (property "Reference" "X1" (at 66.04 60.96 0)
-      (effects (font (size 1.27 1.27)))
-    )
-    (property "Value" "~" (at 66.04 71.12 0)
-      (effects (font (size 1.27 1.27)))
-    )
-    (property "Footprint" "M17_misc_active:ECS-TXO-20CSMV" (at 66.04 71.12 0)
-      (effects (font (size 1.27 1.27)) hide)
-    )
-    (property "Datasheet" "https://ecsxtal.com/store/pdf/ECS-TXO-20CSMV.pdf" (at 66.04 71.12 0)
+  (symbol (lib_id "M17_misc_active:ECS-TXO-20CSMV") (at 58.42 62.23 0) (unit 1)
+    (in_bom yes) (on_board yes) (dnp no)
+    (property "Reference" "X1" (at 59.69 60.96 0)
+      (effects (font (size 1.27 1.27)))
+    )
+    (property "Value" "ECS-TXO-20CSMV" (at 66.04 76.2 0)
+      (effects (font (size 1.27 1.27)))
+    )
+    (property "Footprint" "M17_misc_active:ECS-TXO-20CSMV" (at 58.42 62.23 0)
+      (effects (font (size 1.27 1.27)) hide)
+    )
+    (property "Datasheet" "https://ecsxtal.com/store/pdf/ECS-TXO-20CSMV.pdf" (at 58.42 62.23 0)
       (effects (font (size 1.27 1.27)) hide)
     )
@@
     )
   )
-  (symbol (lib_id "M17_RF:RFSW8008") (at 144.78 151.13 0) (mirror y) (unit 1)
-    (in_bom yes) (on_board yes) (dnp no)
-    (property "Reference" "SW1" (at 144.78 158.75 0)
-      (effects (font (size 1.27 1.27)))
-    )
-    (property "Value" "~" (at 148.59 146.05 0)
-      (effects (font (size 1.27 1.27)))
-    )
-    (property "Footprint" "M17_misc_active:RFSW8008" (at 148.59 146.05 0)
-      (effects (font (size 1.27 1.27)) hide)
-    )
-    (property "Datasheet" "https://www.qorvo.com/products/d/da006546" (at 148.59 146.05 0)
+  (symbol (lib_id "M17_RF:RFSW8008") (at 152.4 143.51 0) (mirror y) (unit 1)
+    (in_bom yes) (on_board yes) (dnp no)
+    (property "Reference" "SW?" (at 137.16 142.24 0)
+      (effects (font (size 1.27 1.27)) (justify right))
+    )
+    (property "Value" "RFSW8008" (at 144.78 157.48 0)
+      (effects (font (size 1.27 1.27)))
+    )
+    (property "Footprint" "M17_misc_active:RFSW8008" (at 152.4 143.51 0)
+      (effects (font (size 1.27 1.27)) hide)
+    )
+    (property "Datasheet" "https://www.qorvo.com/products/d/da006546" (at 152.4 143.51 0)
       (effects (font (size 1.27 1.27)) hide)
     )
@@
       (project "OpenHT-RF"
         (path "/3c300b59-23ec-47f8-bb91-29ca34130bcf/e3bba2b3-d2df-4b56-8e13-359b6c4f2426"
-          (reference "SW1") (unit 1)
-        )
-      )
+          (reference "SW?") (unit 1)
+        )
+      )

Commit message: Added RF baluns
Parts:
- added C49: 1nF, symbol Device:C
- added C50, C51: 1.8pF, symbol Device:C
- added C52: 0.8pF, symbol Device:C
- added L2: ATB2012-50011, M17_misc_passive:ATB2012, symbol M17_RF:ATB2012-50011
- added L3: 2450FB15A050, M17_misc_passive:2450FB15A050, symbol M17_RF:2450FB15A050
- added L4: 5.6nH, symbol Device:L
Connections:
- net GND: now also C49.2
- net RFN09: now also L2.3
- net RFN24: now also C51.1
- net RFP09: now also L2.4
- net RFP24: now also C50.1
- net at FL1.1 (IN): now also C52.2
- net at FL2.1 (IN): now also L3.1 (IN)
- new net: C51.2, L3.4 (OUT2), L4.2
- new net: C52.1, L2.1
- new net: C49.1, L2.2
- new net: C50.2, L3.3 (OUT1), L4.1
Other:
- moved on the sheet: C38, C39, C40, C41, C42, FL1, FL2, J6, SW?

Commit message: Optimised IO routing, renumbered components
Parts:
- removed C42: 100pF, symbol Device:C
- added C510: 100pF, symbol Device:C
- C509: renamed from C41; Dielectric (none) -> C0G
- gave numbers to parts that had none: 2
- renumbered C32 to C501, C50 to C502, C51 to C503, C33 to C504, C49 to C505, C34 to C506, C52 to C507, C35 to C508, C39 to C511, C38 to C512, C40 to C513, C36 to C514, C37 to C515, FB5 to FB501, FL1 to FL501, FL2 to FL502, J6 to J501, J7 to J502, J8 to J503, L4 to L501, L3 to L502, L2 to L503, R13 to R501, X1 to X501
Connections:
- net GND: now also L502.2 (DC_Feed/RF_GND), L502.5 (GND)
- net at FL502.3 (OUT): now also C510.1
- net at SW501.4 (RF1): now also C510.2
Other:
- moved on the sheet: C509, C515, J502, J503, R3
