File: OpenHT-RF/rf.kicad_sch (KiCad schematic)
At the start: 31 parts, among them J501 Conn_Coaxial, J502 Conn_01x02, J503 Conn_01x02, SW501 RFSW8008, U501 AT86RF215, X501 ECS-TXO-20CSMV

Commit message: Fixed 3.3V power symbol
Use 3V3 everywhere instead of 3.3
Connections:
- net +3.3V is gone; now on net +3V3: FB501.1
Changed lines of the file:
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@@
-    )
-  )
-  (symbol (lib_id "power:+3.3V") (at 24.13 24.13 0) (unit 1)
-    (in_bom yes) (on_board yes) (dnp no) (fields_autoplaced)
-    (property "Reference" "#PWR0501" (at 24.13 27.94 0)
-      (effects (font (size 1.27 1.27)) hide)
-    )
-    (property "Value" "+3.3V" (at 24.13 20.32 0)
-      (effects (font (size 1.27 1.27)))
-    )
-    (property "Footprint" "" (at 24.13 24.13 0)
-      (effects (font (size 1.27 1.27)) hide)
-    )
-    (property "Datasheet" "" (at 24.13 24.13 0)
-      (effects (font (size 1.27 1.27)) hide)
-    )
-    (pin "1")
-    (instances
-      (project "OpenHT-RF"
-        (path "/3c300b59-23ec-47f8-bb91-29ca34130bcf/e3bba2b3-d2df-4b56-8e13-359b6c4f2426"
-          (reference "#PWR0501") (unit 1)
-        )
-      )
     )
   )
@@
         )
       )
+    )
+  )
+  (symbol (lib_id "power:+3V3") (at 24.13 24.13 0) (unit 1)
+    (in_bom yes) (on_board yes) (dnp no)
+    (property "Reference" "#PWR07" (at 24.13 27.94 0)
+      (effects (font (size 1.27 1.27)) hide)
+    )
+    (property "Value" "+3V3" (at 24.13 20.32 0)
+      (effects (font (size 1.27 1.27)))
+    )
+    (property "Footprint" "" (at 24.13 24.13 0)
+      (effects (font (size 1.27 1.27)) hide)
+    )
+    (property "Datasheet" "" (at 24.13 24.13 0)
+      (effects (font (size 1.27 1.27)) hide)
+    )
+    (pin "1")
+    (instances
+      (project "OpenHT-RF"
+        (path "/3c300b59-23ec-47f8-bb91-29ca34130bcf/1ac744a1-066f-4d1a-b0df-41e1d7c4818a"
+          (reference "#PWR07") (unit 1)
+        )
+        (path "/3c300b59-23ec-47f8-bb91-29ca34130bcf/e3bba2b3-d2df-4b56-8e13-359b6c4f2426"
+          (reference "#PWR0524") (unit 1)
+        )
+      )

Commit message: Updated QFN footprints
Parts:
- U501: footprint M17_QFN:VQFN-48-1EP_7x7mm_P0.5mm_EP5.6x5.6mm -> M17_QFN:VQFN-48-1EP_7x7mm_P0.5mm_EP5.6x5.6mm_ThermalVias
Changed lines of the file:
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@@
       (effects (font (size 1.27 1.27)))
     )
-    (property "Footprint" "M17_QFN:VQFN-48-1EP_7x7mm_P0.5mm_EP5.6x5.6mm" (at 130.81 41.91 0)
+    (property "Footprint" "M17_QFN:VQFN-48-1EP_7x7mm_P0.5mm_EP5.6x5.6mm_ThermalVias" (at 130.81 41.91 0)
       (effects (font (size 1.27 1.27)) hide)
     )

Commit message: Renamed RF differential signals
Connections:
- net RFN09 renamed RF09_N
- net RFN24 renamed RF24_N
- net RFP09 renamed RF09_P
- net RFP24 renamed RF24_P
Changed lines of the file:
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@@
     (effects (font (size 1.27 1.27)) (justify left bottom))
   )
-  (label "RFP09" (at 40.64 133.35 0) (fields_autoplaced)
+  (label "RF09_P" (at 40.64 133.35 0) (fields_autoplaced)
     (effects (font (size 1.27 1.27)) (justify left bottom))
   )
@@
     (effects (font (size 1.27 1.27)) (justify left bottom))
   )
-  (label "RFN24" (at 19.05 176.53 0) (fields_autoplaced)
+  (label "RF24_N" (at 19.05 176.53 0) (fields_autoplaced)
     (effects (font (size 1.27 1.27)) (justify left bottom))
   )
-  (label "RFN24" (at 207.01 66.04 180) (fields_autoplaced)
+  (label "RF24_N" (at 207.01 66.04 180) (fields_autoplaced)
     (effects (font (size 1.27 1.27)) (justify right bottom))
   )
-  (label "RFP24" (at 19.05 161.29 0) (fields_autoplaced)
+  (label "RF24_P" (at 19.05 161.29 0) (fields_autoplaced)
     (effects (font (size 1.27 1.27)) (justify left bottom))
   )
@@
     (effects (font (size 1.27 1.27)) (justify left bottom))
   )
-  (label "RFP24" (at 207.01 63.5 180) (fields_autoplaced)
+  (label "RF24_P" (at 207.01 63.5 180) (fields_autoplaced)
     (effects (font (size 1.27 1.27)) (justify right bottom))
   )
-  (label "RFN09" (at 207.01 72.39 180) (fields_autoplaced)
+  (label "RF09_N" (at 207.01 72.39 180) (fields_autoplaced)
     (effects (font (size 1.27 1.27)) (justify right bottom))
   )
-  (label "RFN09" (at 40.64 135.89 0) (fields_autoplaced)
+  (label "RF09_N" (at 40.64 135.89 0) (fields_autoplaced)
     (effects (font (size 1.27 1.27)) (justify left bottom))
   )
-  (label "RFP09" (at 207.01 69.85 180) (fields_autoplaced)
+  (label "RF09_P" (at 207.01 69.85 180) (fields_autoplaced)
     (effects (font (size 1.27 1.27)) (justify right bottom))
   )

Commit message: Added missing decoupling capacitors
Parts:
- added C517, C518, C519, C520, C521: 0.1uF, Capacitor_SMD:C_0402_1005Metric, symbol Device:C
Connections:
- net DEVDD: now also C517.1, C518.1, C519.1, C520.1, C521.1
- net GND: now also C517.2, C518.2, C519.2, C520.2, C521.2

Commit message: [WIP] Layout
Flipped the content upside down for the SMA connector. Reorganized GPIOs. RF routing started.
Parts:
- added R402: 100R, Resistor_SMD:R_0402_1005Metric, symbol Device:R
Connections:
- net RF24_N: now also C502.1; no longer C503.1
- net RF24_P: now also C503.1; no longer C502.1
- net S_SPI_MISO: now also R402.2; no longer U501.44 (MISO)
- new net: R402.1, U501.44 (MISO)
Other:
- moved on the sheet: C501, C504, C506, C508, C514, C515, C516, J502, J503, R3, R501, R503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

Commit message: Updated SMA connector
Parts:
- J501: value Conn_Coaxial -> EMPCB.CSMAFSTJ.A; footprint Connector_Coaxial:SMA_Amphenol_132289_EdgeMount -> M17_connectors:SMA_Taoglas_EMPCB.CSMAFSTJ.A
Changed lines of the file:
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@@
   )
   (symbol (lib_id "Connector:Conn_Coaxial") (at 213.36 149.86 0) (unit 1)
-    (in_bom yes) (on_board yes) (dnp no) (fields_autoplaced)
-    (property "Reference" "J501" (at 215.9001 149.5095 0)
+    (in_bom yes) (on_board yes) (dnp no)
+    (property "Reference" "J501" (at 217.17 150.7882 0)
       (effects (font (size 1.27 1.27)) (justify left))
     )
-    (property "Value" "Conn_Coaxial" (at 215.9001 151.4305 0)
+    (property "Value" "EMPCB.CSMAFSTJ.A" (at 217.17 153.67 0)
       (effects (font (size 1.27 1.27)) (justify left))
     )
-    (property "Footprint" "Connector_Coaxial:SMA_Amphenol_132289_EdgeMount" (at 213.36 149.86 0)
+    (property "Footprint" "M17_connectors:SMA_Taoglas_EMPCB.CSMAFSTJ.A" (at 213.36 149.86 0)
       (effects (font (size 1.27 1.27)) hide)
     )

Commit message: Various schematic updates
Edited IO names, updated load switch symbol, swapped RF switch inputs
Connections:
- net at C509.2: now also SW501.4 (RF1); no longer SW501.6 (RF2)
- net at C510.2: now also SW501.6 (RF2); no longer SW501.4 (RF1)
Other:
- moved on the sheet: C502, C503, C505, C507, C509, C510, C511, C512, C513, C520, C521, FL501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

Commit message: Added power supply decoupling capacitor
Parts:
- added C522: 10uF, Capacitor_SMD:C_0805_2012Metric, symbol Device:C
Connections:
- net DEVDD: now also C522.1
- net GND: now also C522.2
Changed lines of the file:
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@@
   (junction (at 173.99 104.14) (diameter 0) (color 0 0 0 0)
   )
+  (junction (at 171.45 104.14) (diameter 0) (color 0 0 0 0)
+  )
+  (junction (at 167.64 104.14) (diameter 0) (color 0 0 0 0)
+  )
+  (junction (at 85.09 140.97) (diameter 0) (color 0 0 0 0)
+  )
+  (junction (at 36.83 86.36) (diameter 0) (color 0 0 0 0)
+  )
+  (junction (at 101.6 67.31) (diameter 0) (color 0 0 0 0)
+  )
+  (junction (at 52.07 74.93) (diameter 0) (color 0 0 0 0)
+  )
+  (junction (at 166.37 104.14) (diameter 0) (color 0 0 0 0)
+  )
   (junction (at 50.8 26.67) (diameter 0) (color 0 0 0 0)
   )
-  (junction (at 171.45 104.14) (diameter 0) (color 0 0 0 0)
-  )
-  (junction (at 167.64 104.14) (diameter 0) (color 0 0 0 0)
-  )
-  (junction (at 85.09 140.97) (diameter 0) (color 0 0 0 0)
-  )
-  (junction (at 36.83 86.36) (diameter 0) (color 0 0 0 0)
-  )
-  (junction (at 101.6 67.31) (diameter 0) (color 0 0 0 0)
-  )
-  (junction (at 52.07 74.93) (diameter 0) (color 0 0 0 0)
-  )
-  (junction (at 166.37 104.14) (diameter 0) (color 0 0 0 0)
-  )
   (junction (at 179.07 129.54) (diameter 0) (color 0 0 0 0)
   )
@@
   (junction (at 48.26 86.36) (diameter 0) (color 0 0 0 0)
   )
+  (junction (at 60.96 26.67) (diameter 0) (color 0 0 0 0)
+  )
   (junction (at 168.91 104.14) (diameter 0) (color 0 0 0 0)
   )
@@
     (stroke (width 0) (type default))
   )
-  (wire (pts (xy 50.8 22.86) (xy 50.8 26.67))
+  (wire (pts (xy 60.96 22.86) (xy 60.96 26.67))
     (stroke (width 0) (type default))
   )
@@
     (stroke (width 0) (type default))
   )
+  (wire (pts (xy 50.8 26.67) (xy 60.96 26.67))
+    (stroke (width 0) (type default))
+  )
   (wire (pts (xy 43.18 104.14) (xy 43.18 105.41))
     (stroke (width 0) (type default))
@@
     (stroke (width 0) (type default))
   )
+  (wire (pts (xy 50.8 35.56) (xy 50.8 36.83))
+    (stroke (width 0) (type default))
+  )
   (wire (pts (xy 173.99 102.87) (xy 173.99 104.14))
     (stroke (width 0) (type default))
@@
     (stroke (width 0) (type default))
   )
-  (wire (pts (xy 50.8 26.67) (xy 58.42 26.67))
+  (wire (pts (xy 60.96 26.67) (xy 68.58 26.67))
     (stroke (width 0) (type default))
   )
@@
     (stroke (width 0) (type default))
   )
+  (wire (pts (xy 50.8 26.67) (xy 50.8 27.94))
+    (stroke (width 0) (type default))
+  )
   (wire (pts (xy 163.83 104.14) (xy 166.37 104.14))
     (stroke (width 0) (type default))
@@
     (stroke (width 0) (type default))
   )
-  (wire (pts (xy 50.8 22.86) (xy 58.42 22.86))
+  (wire (pts (xy 60.96 22.86) (xy 68.58 22.86))
     (stroke (width 0) (type default))
   )
@@
     (stroke (width 0) (type default))
   )
+  (wire (pts (xy 43.18 26.67) (xy 50.8 26.67))
+    (stroke (width 0) (type default))
+  )
   (wire (pts (xy 38.1 171.45) (xy 60.96 171.45))
     (stroke (width 0) (type default))
@@
   )
   (wire (pts (xy 181.61 29.21) (xy 181.61 39.37))
-    (stroke (width 0) (type default))
-  )
-  (wire (pts (xy 43.18 26.67) (xy 50.8 26.67))
     (stroke (width 0) (type default))
   )
@@
     (effects (font (size 1.27 1.27)) (justify left top))
   )
-  (label "EVDD" (at 58.42 22.86 180) (fields_autoplaced)
+  (label "EVDD" (at 68.58 22.86 180) (fields_autoplaced)
     (effects (font (size 1.27 1.27)) (justify right bottom))
   )
@@
     (effects (font (size 1.27 1.27)) (justify left bottom))
   )
-  (label "DEVDD" (at 58.42 26.67 180) (fields_autoplaced)
+  (label "DEVDD" (at 68.58 26.67 180) (fields_autoplaced)
     (effects (font (size 1.27 1.27)) (justify right bottom))
   )
@@
     )
   )
+  (symbol (lib_id "power:GND") (at 50.8 36.83 0) (unit 1)
+    (in_bom yes) (on_board yes) (dnp no) (fields_autoplaced)
+    (property "Reference" "#PWR0529" (at 50.8 43.18 0)
+      (effects (font (size 1.27 1.27)) hide)
+    )
+    (property "Value" "GND" (at 50.8 41.91 0)
+      (effects (font (size 1.27 1.27)))
+    )
+    (property "Footprint" "" (at 50.8 36.83 0)
+      (effects (font (size 1.27 1.27)) hide)
+    )
+    (property "Datasheet" "" (at 50.8 36.83 0)
+      (effects (font (size 1.27 1.27)) hide)
+    )
+    (pin "1")
+    (instances
+      (project "OpenHT-RF"
+        (path "/3c300b59-23ec-47f8-bb91-29ca34130bcf/e3bba2b3-d2df-4b56-8e13-359b6c4f2426"
+          (reference "#PWR0529") (unit 1)
+        )
+      )
+    )
+  )
   (symbol (lib_id "power:GND") (at 195.58 93.98 0) (unit 1)
     (in_bom yes) (on_board yes) (dnp no) (fields_autoplaced)
@@
         )
       )
+    )
+  )
+  (symbol (lib_id "Device:C") (at 50.8 31.75 0) (unit 1)
+    (in_bom yes) (on_board yes) (dnp no) (fields_autoplaced)
+    (property "Reference" "C522" (at 54.61 31.115 0)
+      (effects (font (size 1.27 1.27)) (justify left))
+    )
+    (property "Value" "10uF" (at 54.61 33.655 0)
+      (effects (font (size 1.27 1.27)) (justify left))
+    )
+    (property "Footprint" "Capacitor_SMD:C_0805_2012Metric" (at 51.7652 35.56 0)
+      (effects (font (size 1.27 1.27)) hide)
+    )
+    (property "Datasheet" "~" (at 50.8 31.75 0)
+      (effects (font (size 1.27 1.27)) hide)
+    )
+    (pin "1")
+    (pin "2")
+    (instances
+      (project "OpenHT-RF"
+        (path "/3c300b59-23ec-47f8-bb91-29ca34130bcf/e3bba2b3-d2df-4b56-8e13-359b6c4f2426"
+          (reference "C522") (unit 1)
+        )
+      )
