File: OpenHT-RF/rf.kicad_sch (KiCad schematic)
At the start: 41 parts, among them J202 MS300-10F, J501 EMPCB.CSMAFSTJ.A, J502 Conn_01x02, J503 Conn_01x02, SW501 RFSW8008, U501 AT86RF215, X501 ECS-TXO-20CSMV

Commit message: Fixed ERC errors
Changed lines of the file:
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@@
   (junction (at 163.83 104.14) (diameter 0) (color 0 0 0 0)
   )
+  (junction (at 54.61 26.67) (diameter 0) (color 0 0 0 0)
+  )
   (junction (at 184.15 123.19) (diameter 0) (color 0 0 0 0)
   )
@@
     (stroke (width 0) (type default))
   )
+  (wire (pts (xy 54.61 25.4) (xy 54.61 26.67))
+    (stroke (width 0) (type default))
+  )
   (wire (pts (xy 194.31 81.28) (xy 204.47 81.28))
     (stroke (width 0) (type default))
@@
     (stroke (width 0) (type default))
   )
-  (wire (pts (xy 50.8 26.67) (xy 60.96 26.67))
+  (wire (pts (xy 50.8 26.67) (xy 54.61 26.67))
     (stroke (width 0) (type default))
   )
@@
     (stroke (width 0) (type default))
   )
-  (wire (pts (xy 6.0174 -6.2506) (xy 8.5574 -6.2506))
-    (stroke (width 0) (type default))
-  )
   (wire (pts (xy 196.85 146.05) (xy 208.28 146.05))
     (stroke (width 0) (type default))
@@
   )
   (wire (pts (xy 24.13 24.13) (xy 24.13 26.67))
+    (stroke (width 0) (type default))
+  )
+  (wire (pts (xy 54.61 26.67) (xy 60.96 26.67))
     (stroke (width 0) (type default))
   )
@@
         )
       )
+    )
+  )
+  (symbol (lib_id "power:PWR_FLAG") (at 54.61 25.4 0) (unit 1)
+    (in_bom yes) (on_board yes) (dnp no) (fields_autoplaced)
+    (property "Reference" "#FLG0203" (at 54.61 23.495 0)
+      (effects (font (size 1.27 1.27)) hide)
+    )
+    (property "Value" "PWR_FLAG" (at 54.61 21.59 0)
+      (effects (font (size 1.27 1.27)))
+    )
+    (property "Footprint" "" (at 54.61 25.4 0)
+      (effects (font (size 1.27 1.27)) hide)
+    )
+    (property "Datasheet" "~" (at 54.61 25.4 0)
+      (effects (font (size 1.27 1.27)) hide)
+    )
+    (pin "1")
+    (instances
+      (project "OpenHT-RF"
+        (path "/3c300b59-23ec-47f8-bb91-29ca34130bcf/17571ff2-f5b8-49d7-92c6-d2c188350dd2"
+          (reference "#FLG0203") (unit 1)
+        )
+        (path "/3c300b59-23ec-47f8-bb91-29ca34130bcf/e3bba2b3-d2df-4b56-8e13-359b6c4f2426"
+          (reference "#FLG0501") (unit 1)
+        )
+      )

Commit message: Modified shields to use two symbols
Allows to have the MPN of the lid in the schematic alongside the frame
Parts:
- removed J202: MS300-10F, M17_misc_passive:MS300-10F, symbol Device:RFShield_TwoPieces
- added J504: MS300-10F, M17_misc_passive:MS300-10F, symbol M17_device:RFShield_Frame
- added J505: MS300-10C, symbol M17_device:RFShield_Lid
Connections:
- net GND: now also J504.1 (Shield)
Changed lines of the file:
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@@
+    )
+  )
+  (symbol (lib_id "M17_device:RFShield_Lid") (at 35.56 171.45 0) (unit 1)
+    (in_bom yes) (on_board no) (dnp no)
+    (property "Reference" "J505" (at 35.56 163.83 0)
+      (effects (font (size 1.27 1.27)))
+    )
+    (property "Value" "MS300-10C" (at 35.56 166.37 0)
+      (effects (font (size 1.27 1.27)))
+    )
+    (property "Footprint" "" (at 35.56 179.07 0)
+      (effects (font (size 1.27 1.27)) hide)
+    )
+    (property "Datasheet" "" (at 35.56 179.07 0)
+      (effects (font (size 1.27 1.27)) hide)
+    )
+    (property "MPN" "MS300-10C" (at 35.56 171.45 0)
+      (effects (font (size 1.27 1.27)) hide)
+    )
+    (instances
+      (project "OpenHT-RF"
+        (path "/3c300b59-23ec-47f8-bb91-29ca34130bcf/e3bba2b3-d2df-4b56-8e13-359b6c4f2426"
+          (reference "J505") (unit 1)
+        )
+      )
     )
   )
@@
     )
   )
+  (symbol (lib_id "M17_device:RFShield_Frame") (at 35.56 179.07 0) (unit 1)
+    (in_bom yes) (on_board yes) (dnp no)
+    (property "Reference" "J504" (at 52.07 177.8 0)
+      (effects (font (size 1.27 1.27)) (justify left))
+    )
+    (property "Value" "MS300-10F" (at 52.07 180.34 0)
+      (effects (font (size 1.27 1.27)) (justify left))
+    )
+    (property "Footprint" "M17_misc_passive:MS300-10F" (at 35.56 179.07 0)
+      (effects (font (size 1.27 1.27)) hide)
+    )
+    (property "Datasheet" "" (at 35.56 179.07 0)
+      (effects (font (size 1.27 1.27)) hide)
+    )
+    (property "MPN" "MS300-10F" (at 35.56 179.07 0)
+      (effects (font (size 1.27 1.27)) hide)
+    )
+    (pin "1")
+    (instances
+      (project "OpenHT-RF"
+        (path "/3c300b59-23ec-47f8-bb91-29ca34130bcf/e3bba2b3-d2df-4b56-8e13-359b6c4f2426"
+          (reference "J504") (unit 1)
+        )
+      )
+    )
+  )
   (symbol (lib_id "power:GND") (at 124.46 91.44 0) (unit 1)
     (in_bom yes) (on_board yes) (dnp no) (fields_autoplaced)
@@
         )
       )
-    )
-  )
-  (symbol (lib_id "Device:RFShield_TwoPieces") (at 35.56 179.07 0) (unit 1)
-    (in_bom yes) (on_board yes) (dnp no) (fields_autoplaced)
-    (property "Reference" "J202" (at 54.61 176.53 0)
-      (effects (font (size 1.27 1.27)) (justify left))
-    )
-    (property "Value" "MS300-10F" (at 54.61 179.07 0)
-      (effects (font (size 1.27 1.27)) (justify left))
-    )
-    (property "Footprint" "M17_misc_passive:MS300-10F" (at 35.56 181.61 0)
-      (effects (font (size 1.27 1.27)) hide)
-    )
-    (property "Datasheet" "~" (at 35.56 181.61 0)
-      (effects (font (size 1.27 1.27)) hide)
-    )
-    (property "MPN" "MS300-10F" (at 35.56 179.07 0)
-      (effects (font (size 1.27 1.27)) hide)
-    )
-    (pin "1")
-    (instances
-      (project "OpenHT-RF"
-        (path "/3c300b59-23ec-47f8-bb91-29ca34130bcf/17571ff2-f5b8-49d7-92c6-d2c188350dd2"
-          (reference "J202") (unit 1)
-        )
-        (path "/3c300b59-23ec-47f8-bb91-29ca34130bcf/e3bba2b3-d2df-4b56-8e13-359b6c4f2426"
-          (reference "J504") (unit 1)
-        )
-      )

Commit message: Completed components values
Completed dielectric, rated voltage, tolerance, MPN
Parts:
- C506, C511, C512, C513, C516: Dielectric (none) -> C0G
- J502, J503: now not fitted
- J505: Manual_Placement (none) -> 1
- R3, R402, R501, R503: Tolerance (none) -> 1%
- SW501: MPN (none) -> RFSW8008TR7
Other:
- moved on the sheet: C513
Changed lines of the file:
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@@
     (stroke (width 0) (type default))
   )
-  (wire (pts (xy 215.9 146.05) (xy 224.79 146.05))
+  (wire (pts (xy 217.17 146.05) (xy 224.79 146.05))
     (stroke (width 0) (type default))
   )
@@
     (stroke (width 0) (type default))
   )
-  (wire (pts (xy 196.85 146.05) (xy 208.28 146.05))
+  (wire (pts (xy 196.85 146.05) (xy 209.55 146.05))
     (stroke (width 0) (type default))
   )
@@
     )
   )
-  (netclass_flag "" (length 2.54) (shape round) (at 217.17 146.05 0) (fields_autoplaced)
+  (netclass_flag "" (length 2.54) (shape round) (at 218.44 146.05 0) (fields_autoplaced)
     (effects (font (size 1.27 1.27)) (justify left bottom))
-    (property "Netclass" "50Ohm" (at 217.8685 143.51 0)
+    (property "Netclass" "50Ohm" (at 219.1385 143.51 0)
       (effects (font (size 1.27 1.27) italic) (justify left))
     )
@@
     )
     (property "MPN" "MS300-10C" (at 35.56 171.45 0)
+      (effects (font (size 1.27 1.27)) hide)
+    )
+    (property "Manual_Placement" "1" (at 35.56 171.45 0)
       (effects (font (size 1.27 1.27)) hide)
     )
@@
       (effects (font (size 1.27 1.27)) hide)
     )
+    (property "Tolerance" "1%" (at 90.17 76.2 0)
+      (effects (font (size 1.27 1.27)) hide)
+    )
     (pin "1")
     (pin "2")
@@
   )
   (symbol (lib_id "Device:C") (at 187.96 128.27 0) (unit 1)
-    (in_bom yes) (on_board yes) (dnp no) (fields_autoplaced)
+    (in_bom yes) (on_board yes) (dnp no)
     (property "Reference" "C511" (at 191.77 127.635 0)
       (effects (font (size 1.27 1.27)) (justify left))
@@
       (effects (font (size 1.27 1.27)) hide)
     )
+    (property "Dielectric" "C0G" (at 191.77 132.715 0)
+      (effects (font (size 1.27 1.27)) (justify left))
+    )
     (pin "1")
     (pin "2")
@@
   )
   (symbol (lib_id "Device:C") (at 201.93 128.27 0) (unit 1)
-    (in_bom yes) (on_board yes) (dnp no) (fields_autoplaced)
+    (in_bom yes) (on_board yes) (dnp no)
     (property "Reference" "C512" (at 205.74 127.635 0)
       (effects (font (size 1.27 1.27)) (justify left))
@@
     (property "Datasheet" "~" (at 201.93 128.27 0)
       (effects (font (size 1.27 1.27)) hide)
+    )
+    (property "Dielectric" "C0G" (at 205.74 132.715 0)
+      (effects (font (size 1.27 1.27)) (justify left))
     )
     (pin "1")
@@
   (symbol (lib_id "Device:C") (at 101.6 76.2 0) (mirror y) (unit 1)
     (in_bom yes) (on_board yes) (dnp no)
-    (property "Reference" "C506" (at 97.79 75.565 0)
-      (effects (font (size 1.27 1.27)) (justify left))
-    )
-    (property "Value" "10pF" (at 97.79 78.105 0)
+    (property "Reference" "C506" (at 99.06 75.565 0)
+      (effects (font (size 1.27 1.27)) (justify left))
+    )
+    (property "Value" "10pF" (at 99.06 78.105 0)
       (effects (font (size 1.27 1.27)) (justify left))
     )
@@
     (property "Datasheet" "~" (at 101.6 76.2 0)
       (effects (font (size 1.27 1.27)) hide)
+    )
+    (property "Dielectric" "C0G" (at 96.52 80.645 0)
+      (effects (font (size 1.27 1.27)))
     )
     (pin "1")
@@
   )
   (symbol (lib_id "Connector_Generic:Conn_01x02") (at 209.55 59.69 0) (unit 1)
-    (in_bom yes) (on_board yes) (dnp no) (fields_autoplaced)
+    (in_bom yes) (on_board yes) (dnp yes) (fields_autoplaced)
     (property "Reference" "J502" (at 212.09 60.325 0)
       (effects (font (size 1.27 1.27)) (justify left))
@@
       (effects (font (size 1.27 1.27)) hide)
     )
+    (property "Tolerance" "1%" (at 120.65 63.5 0)
+      (effects (font (size 1.27 1.27)) hide)
+    )
     (pin "1")
     (pin "2")
@@
       (effects (font (size 1.27 1.27)) hide)
     )
+    (property "Dielectric" "C0G" (at 95.25 60.325 0)
+      (effects (font (size 1.27 1.27)) (justify right))
+    )
     (pin "1")
     (pin "2")
@@
     )
     (property "Datasheet" "~" (at 147.32 34.29 0)
+      (effects (font (size 1.27 1.27)) hide)
+    )
+    (property "Tolerance" "1%" (at 147.32 34.29 90)
       (effects (font (size 1.27 1.27)) hide)
     )
@@
     )
     (property "Datasheet" "https://www.qorvo.com/products/d/da006546" (at 191.77 138.43 0)
+      (effects (font (size 1.27 1.27)) hide)
+    )
+    (property "MPN" "RFSW8008TR7 " (at 191.77 138.43 0)
       (effects (font (size 1.27 1.27)) hide)
     )
@@
       (effects (font (size 1.27 1.27)) hide)
     )
+    (property "Tolerance" "1%" (at 99.06 50.8 90)
+      (effects (font (size 1.27 1.27)) hide)
+    )
     (pin "1")
     (pin "2")
@@
     )
   )
-  (symbol (lib_id "Device:C") (at 212.09 146.05 90) (unit 1)
-    (in_bom yes) (on_board yes) (dnp no) (fields_autoplaced)
-    (property "Reference" "C513" (at 212.09 139.7 90)
-      (effects (font (size 1.27 1.27)))
-    )
-    (property "Value" "100pF" (at 212.09 142.24 90)
-      (effects (font (size 1.27 1.27)))
-    )
-    (property "Footprint" "Capacitor_SMD:C_0402_1005Metric" (at 215.9 145.0848 0)
-      (effects (font (size 1.27 1.27)) hide)
-    )
-    (property "Datasheet" "~" (at 212.09 146.05 0)
-      (effects (font (size 1.27 1.27)) hide)
+  (symbol (lib_id "Device:C") (at 213.36 146.05 90) (unit 1)
+    (in_bom yes) (on_board yes) (dnp no)
+    (property "Reference" "C513" (at 213.36 139.7 90)
+      (effects (font (size 1.27 1.27)))
+    )
+    (property "Value" "100pF" (at 213.36 142.24 90)
+      (effects (font (size 1.27 1.27)))
+    )
+    (property "Footprint" "Capacitor_SMD:C_0402_1005Metric" (at 217.17 145.0848 0)
+      (effects (font (size 1.27 1.27)) hide)
+    )
+    (property "Datasheet" "~" (at 213.36 146.05 0)
+      (effects (font (size 1.27 1.27)) hide)
+    )
+    (property "Dielectric" "C0G" (at 213.36 149.86 90)
+      (effects (font (size 1.27 1.27)))
     )
     (pin "1")
@@
   )
   (symbol (lib_id "Connector_Generic:Conn_01x02") (at 209.55 78.74 0) (unit 1)
-    (in_bom yes) (on_board yes) (dnp no) (fields_autoplaced)
+    (in_bom yes) (on_board yes) (dnp yes) (fields_autoplaced)
     (property "Reference" "J503" (at 212.09 79.375 0)
       (effects (font (size 1.27 1.27)) (justify left))

Commit message: Fixed incorrect value for R502
Parts:
- R3: value 100k -> 100kR
Changed lines of the file:
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@@
       (effects (font (size 1.27 1.27)))
     )
-    (property "Value" "100k" (at 120.65 63.5 90)
+    (property "Value" "100kR" (at 120.65 63.5 90)
       (effects (font (size 1.27 1.27)))
     )

Commit message: Added MPN for L501
Parts:
- L501: MPN (none) -> LRC0402CS5N6GV001T
Changed lines of the file:
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@@
+      (effects (font (size 1.27 1.27)) hide)
+    )
+    (property "MPN" "LRC0402CS5N6GV001T" (at 64.77 132.08 0)
       (effects (font (size 1.27 1.27)) hide)
     )

Commit message: Added MPN for generic components
Parts:
- C501, C517, C518, C519, C520, C521: MPN (none) -> Generic C/0.1uF/0402/X7R/16V
- C502, C503: MPN (none) -> Generic C/1.8pF/0402/C0G/10V
- C504, C523: MPN (none) -> Generic C/1nF/0402/X7R/10V
- C505: MPN (none) -> Generic C/1nF/0402/C0G/10V
- C506: MPN (none) -> Generic C/10pF/0402/C0G/10V
- C507: MPN (none) -> Generic C/0.8pF/0402/C0G/10V
- C508, C514, C515: MPN (none) -> Generic C/1uF/0402/X5R/10V
- C509, C510, C513: MPN (none) -> Generic C/100pF/0402/C0G/10V
- C511: MPN (none) -> Generic C/220pF/0402/C0G/10V
- C512: MPN (none) -> Generic C/82pF/0402/C0G/10V
- C516: MPN (none) -> Generic C/2.2pF/0402/C0G/10V
- C522: MPN (none) -> Generic C/10uF/0805/X5R/10V
- R3: MPN (none) -> Generic R/100kR/0402/1%
- R402: MPN (none) -> Generic R/100R/0402/1%
- R501: MPN (none) -> Generic R/10kR/0402/1%
- R503: MPN (none) -> Generic R/220R/0402/1%
Changed lines of the file:
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@@
+      (effects (font (size 1.27 1.27)) hide)
+    )
+    (property "MPN" "Generic C/1nF/0402/X7R/10V" (at 199.39 153.67 0)
       (effects (font (size 1.27 1.27)) hide)
     )
@@
       (effects (font (size 1.27 1.27)) hide)
     )
+    (property "MPN" "Generic C/0.1uF/0402/X7R/16V" (at 46.99 72.39 0)
+      (effects (font (size 1.27 1.27)) hide)
+    )
     (pin "1")
     (pin "2")
@@
       (effects (font (size 1.27 1.27)) hide)
     )
+    (property "MPN" "Generic R/10kR/0402/1%" (at 90.17 76.2 0)
+      (effects (font (size 1.27 1.27)) hide)
+    )
     (pin "1")
     (pin "2")
@@
     (property "Dielectric" "C0G" (at 58.42 143.51 90)
       (effects (font (size 1.27 1.27)))
+    )
+    (property "MPN" "Generic C/1.8pF/0402/C0G/10V" (at 58.42 139.7 0)
+      (effects (font (size 1.27 1.27)) hide)
     )
     (pin "1")
@@
       (effects (font (size 1.27 1.27)) (justify left))
     )
+    (property "MPN" "Generic C/220pF/0402/C0G/10V" (at 187.96 128.27 0)
+      (effects (font (size 1.27 1.27)) hide)
+    )
     (pin "1")
     (pin "2")
@@
       (effects (font (size 1.27 1.27)) (justify left))
     )
+    (property "MPN" "Generic C/82pF/0402/C0G/10V" (at 201.93 128.27 0)
+      (effects (font (size 1.27 1.27)) hide)
+    )
     (pin "1")
     (pin "2")
@@
     (property "Dielectric" "C0G" (at 58.42 128.27 90)
       (effects (font (size 1.27 1.27)))
+    )
+    (property "MPN" "Generic C/1.8pF/0402/C0G/10V" (at 58.42 124.46 0)
+      (effects (font (size 1.27 1.27)) hide)
     )
     (pin "1")
@@
       (effects (font (size 1.27 1.27)) hide)
     )
+    (property "MPN" "Generic C/1uF/0402/X5R/10V" (at 114.3 76.2 0)
+      (effects (font (size 1.27 1.27)) hide)
+    )
     (pin "1")
     (pin "2")
@@
     (property "Dielectric" "C0G" (at 96.52 80.645 0)
       (effects (font (size 1.27 1.27)))
+    )
+    (property "MPN" "Generic C/10pF/0402/C0G/10V" (at 101.6 76.2 0)
+      (effects (font (size 1.27 1.27)) hide)
     )
     (pin "1")
@@
       (effects (font (size 1.27 1.27)) hide)
     )
+    (property "MPN" "Generic C/1uF/0402/X5R/10V" (at 195.58 90.17 0)
+      (effects (font (size 1.27 1.27)) hide)
+    )
     (pin "1")
     (pin "2")
@@
     (property "Dielectric" "C0G" (at 97.79 175.26 0)
       (effects (font (size 1.27 1.27)) (justify left))
+    )
+    (property "MPN" "Generic C/1nF/0402/C0G/10V" (at 93.98 170.18 0)
+      (effects (font (size 1.27 1.27)) hide)
     )
     (pin "1")
@@
       (effects (font (size 1.27 1.27)) hide)
     )
+    (property "MPN" "Generic C/0.1uF/0402/X7R/16V" (at 81.28 99.06 0)
+      (effects (font (size 1.27 1.27)) hide)
+    )
     (pin "1")
     (pin "2")
@@
       (effects (font (size 1.27 1.27)) hide)
     )
+    (property "MPN" "Generic C/0.1uF/0402/X7R/16V" (at 87.63 99.06 0)
+      (effects (font (size 1.27 1.27)) hide)
+    )
     (pin "1")
     (pin "2")
@@
       (effects (font (size 1.27 1.27)))
     )
+    (property "MPN" "Generic C/100pF/0402/C0G/10V" (at 153.67 162.56 0)
+      (effects (font (size 1.27 1.27)) hide)
+    )
     (pin "1")
     (pin "2")
@@
     )
     (property "Datasheet" "~" (at 83.82 67.31 0)
+      (effects (font (size 1.27 1.27)) hide)
+    )
+    (property "MPN" "Generic C/1nF/0402/X7R/10V" (at 83.82 67.31 0)
       (effects (font (size 1.27 1.27)) hide)
     )
@@
       (effects (font (size 1.27 1.27)) hide)
     )
+    (property "MPN" "Generic C/10uF/0805/X5R/10V" (at 50.8 31.75 0)
+      (effects (font (size 1.27 1.27)) hide)
+    )
     (pin "1")
     (pin "2")
@@
     )
     (property "Tolerance" "1%" (at 120.65 63.5 0)
+      (effects (font (size 1.27 1.27)) hide)
+    )
+    (property "MPN" "Generic R/100kR/0402/1%" (at 120.65 63.5 0)
       (effects (font (size 1.27 1.27)) hide)
     )
@@
       (effects (font (size 1.27 1.27)))
     )
+    (property "MPN" "Generic C/100pF/0402/C0G/10V" (at 153.67 129.54 0)
+      (effects (font (size 1.27 1.27)) hide)
+    )
     (pin "1")
     (pin "2")
@@
       (effects (font (size 1.27 1.27)) (justify right))
     )
+    (property "MPN" "Generic C/2.2pF/0402/C0G/10V" (at 91.44 55.88 0)
+      (effects (font (size 1.27 1.27)) hide)
+    )
     (pin "1")
     (pin "2")
@@
     )
     (property "Tolerance" "1%" (at 147.32 34.29 90)
+      (effects (font (size 1.27 1.27)) hide)
+    )
+    (property "MPN" "Generic R/100R/0402/1%" (at 147.32 34.29 0)
       (effects (font (size 1.27 1.27)) hide)
     )
@@
     )
     (property "Datasheet" "~" (at 199.39 55.88 0)
+      (effects (font (size 1.27 1.27)) hide)
+    )
+    (property "MPN" "Generic C/1uF/0402/X5R/10V" (at 199.39 55.88 0)
       (effects (font (size 1.27 1.27)) hide)
     )
@@
       (effects (font (size 1.27 1.27)) hide)
     )
+    (property "MPN" "Generic C/0.1uF/0402/X7R/16V" (at 48.26 99.06 0)
+      (effects (font (size 1.27 1.27)) hide)
+    )
     (pin "1")
     (pin "2")
@@
     )
     (property "Datasheet" "~" (at 59.69 99.06 0)
+      (effects (font (size 1.27 1.27)) hide)
+    )
+    (property "MPN" "Generic C/0.1uF/0402/X7R/16V" (at 59.69 99.06 0)
       (effects (font (size 1.27 1.27)) hide)
     )
@@
       (effects (font (size 1.27 1.27)))
     )
+    (property "MPN" "Generic C/0.8pF/0402/C0G/10V" (at 107.95 162.56 0)
+      (effects (font (size 1.27 1.27)) hide)
+    )
     (pin "1")
     (pin "2")
@@
       (effects (font (size 1.27 1.27)) hide)
     )
+    (property "MPN" "Generic R/220R/0402/1%" (at 99.06 50.8 0)
+      (effects (font (size 1.27 1.27)) hide)
+    )
     (pin "1")
     (pin "2")
@@
       (effects (font (size 1.27 1.27)) hide)
     )
+    (property "MPN" "Generic C/0.1uF/0402/X7R/16V" (at 36.83 99.06 0)
+      (effects (font (size 1.27 1.27)) hide)
+    )
     (pin "1")
     (pin "2")
@@
       (effects (font (size 1.27 1.27)))
     )
-    (pin "1")
+    (property "MPN" "Generic C/100pF/0402/C0G/10V" (at 213.36 146.05 0)
+      (effects (font (size 1.27 1.27)) hide)
+    )
+    (pin "1")

Commit message: Removed C507
Addresses #4
Parts:
- removed C507: 0.8pF, Capacitor_SMD:C_0402_1005Metric, symbol Device:C
Connections:
- net at L503.1: now also FL501.1 (IN)
Changed lines of the file:
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@@
     (stroke (width 0) (type default))
   )
-  (wire (pts (xy 92.71 162.56) (xy 104.14 162.56))
+  (wire (pts (xy 92.71 162.56) (xy 121.92 162.56))
     (stroke (width 0) (type default))
   )
@@
   )
   (wire (pts (xy 187.96 123.19) (xy 187.96 124.46))
-    (stroke (width 0) (type default))
-  )
-  (wire (pts (xy 111.76 162.56) (xy 121.92 162.56))
     (stroke (width 0) (type default))
   )
@@
     (effects (font (size 1.27 1.27)) (justify left bottom))
     (property "Netclass" "50Ohm" (at 144.2085 127 0)
-      (effects (font (size 1.27 1.27) italic) (justify left))
-    )
-  )
-  (netclass_flag "" (length 2.54) (shape round) (at 114.3 162.56 0) (fields_autoplaced)
-    (effects (font (size 1.27 1.27)) (justify left bottom))
-    (property "Netclass" "50Ohm" (at 114.9985 160.02 0)
       (effects (font (size 1.27 1.27) italic) (justify left))
     )
@@
         )
       )
-    )
-  )
-  (symbol (lib_id "Device:C") (at 107.95 162.56 90) (unit 1)
-    (in_bom yes) (on_board yes) (dnp no)
-    (property "Reference" "C507" (at 107.95 156.21 90)
-      (effects (font (size 1.27 1.27)))
-    )
-    (property "Value" "0.8pF" (at 107.95 158.75 90)
-      (effects (font (size 1.27 1.27)))
-    )
-    (property "Footprint" "Capacitor_SMD:C_0402_1005Metric" (at 111.76 161.5948 0)
-      (effects (font (size 1.27 1.27)) hide)
-    )
-    (property "Datasheet" "~" (at 107.95 162.56 0)
-      (effects (font (size 1.27 1.27)) hide)
-    )
-    (property "Dielectric" "C0G" (at 107.95 166.37 90)
-      (effects (font (size 1.27 1.27)))
-    )
-    (property "MPN" "Generic C/0.8pF/0402/C0G/10V" (at 107.95 162.56 0)
-      (effects (font (size 1.27 1.27)) hide)
-    )
-    (pin "1")
-    (pin "2")
-    (instances
-      (project "OpenHT-RF"
-        (path "/3c300b59-23ec-47f8-bb91-29ca34130bcf/e3bba2b3-d2df-4b56-8e13-359b6c4f2426"
-          (reference "C507") (unit 1)
-        )
-      )
