File: OpenHT-RF/pwr.kicad_sch (KiCad schematic)
At the start: 47 parts, among them J9 Conn_01x02, SW1 SW_Push, U2 LTC2954-1, U3 TPS65261RHBx, U4 AP7330-W5-7

Commit message: Optimised IO routing, renumbered components
Parts:
- added TP201, TP202, TP203, TP204, TP205, TP206: TestPoint, symbol Connector:TestPoint
- renumbered C44 to C201, C30 to C202, C53 to C203, C54 to C204, C22 to C205, C46 to C206, C27 to C207, C47 to C208, C67 to C209, C48 to C210, C68 to C211, C23 to C212, C61 to C213, C26 to C214, C62 to C215, C60 to C216, C63 to C217, C29 to C218, C64 to C219, C31 to C220, C43 to C221, C65 to C222, C45 to C223, C66 to C224, C28 to C225, F1 to F201, J9 to J201, L1 to L201, L5 to L202, R22 to R201, R19 to R202, R23 to R203, R25 to R204, R14 to R205, R24 to R206, R17 to R207, R18 to R208, R20 to R209, R21 to R210, R26 to R211, R27 to R212, R15 to R213, R16 to R214, SW1 to SW201, U2 to U201, U3 to U202, U4 to U203
Connections:
- net +1V0: now also TP204.1
- net +1V8: now also TP203.1
- net +3V3: now also TP202.1
- net +BATT: now also TP201.1
- net GND: now also TP206.1
- net PWR_EN: now also TP205.1

Commit message: Updated power routing, added test points
Parts:
- added JP201: Jumper_2_Bridged, symbol Jumper:Jumper_2_Bridged
Connections:
- net GND: now also JP201.1 (A); no longer R203.1
- new net: JP201.2 (B), R203.1
Other:
- note added: "Open this jumper to disable UVLO"
Changed lines of the file:
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@@
     (stroke (width 0) (type default))
   )
-  (wire (pts (xy 39.37 119.38) (xy 39.37 121.92))
+  (wire (pts (xy 39.37 119.38) (xy 39.37 124.46))
     (stroke (width 0) (type default))
   )
@@
   )
   (wire (pts (xy 184.15 69.85) (xy 187.96 69.85))
+    (stroke (width 0) (type default))
+  )
+  (wire (pts (xy 39.37 134.62) (xy 39.37 138.43))
     (stroke (width 0) (type default))
   )
@@
     (effects (font (size 1.27 1.27)) (justify left top))
   )
+  (text "Open this jumper to disable UVLO" (at 36.83 153.67 90)
+    (effects (font (size 1.27 1.27)) (justify left bottom))
+  )
   (label "PWR_EN" (at 138.43 43.18 0) (fields_autoplaced)
     (effects (font (size 1.27 1.27)) (justify left bottom))
@@
         (path "/3c300b59-23ec-47f8-bb91-29ca34130bcf/17571ff2-f5b8-49d7-92c6-d2c188350dd2"
           (reference "C209") (unit 1)
+        )
+      )
+    )
+  )
+  (symbol (lib_id "Jumper:Jumper_2_Bridged") (at 39.37 129.54 90) (unit 1)
+    (in_bom yes) (on_board yes) (dnp no)
+    (property "Reference" "JP201" (at 41.91 133.35 90)
+      (effects (font (size 1.27 1.27)) (justify right))
+    )
+    (property "Value" "Jumper_2_Bridged" (at 40.64 131.445 90)
+      (effects (font (size 1.27 1.27)) (justify right) hide)
+    )
+    (property "Footprint" "" (at 39.37 129.54 0)
+      (effects (font (size 1.27 1.27)) hide)
+    )
+    (property "Datasheet" "~" (at 39.37 129.54 0)
+      (effects (font (size 1.27 1.27)) hide)
+    )
+    (pin "1")
+    (pin "2")
+    (instances
+      (project "OpenHT-RF"
+        (path "/3c300b59-23ec-47f8-bb91-29ca34130bcf/17571ff2-f5b8-49d7-92c6-d2c188350dd2"
+          (reference "JP201") (unit 1)
         )
       )
@@
     )
   )
-  (symbol (lib_id "power:GND") (at 39.37 121.92 0) (unit 1)
-    (in_bom yes) (on_board yes) (dnp no) (fields_autoplaced)
-    (property "Reference" "#PWR0209" (at 39.37 128.27 0)
-      (effects (font (size 1.27 1.27)) hide)
-    )
-    (property "Value" "GND" (at 39.37 127 0)
-      (effects (font (size 1.27 1.27)))
-    )
-    (property "Footprint" "" (at 39.37 121.92 0)
-      (effects (font (size 1.27 1.27)) hide)
-    )
-    (property "Datasheet" "" (at 39.37 121.92 0)
-      (effects (font (size 1.27 1.27)) hide)
-    )
+  (symbol (lib_id "power:GND") (at 39.37 138.43 0) (unit 1)
+    (in_bom yes) (on_board yes) (dnp no) (fields_autoplaced)
+    (property "Reference" "#PWR0209" (at 39.37 144.78 0)
+      (effects (font (size 1.27 1.27)) hide)
+    )
+    (property "Value" "GND" (at 39.37 143.51 0)
+      (effects (font (size 1.27 1.27)))
+    )
+    (property "Footprint" "" (at 39.37 138.43 0)
+      (effects (font (size 1.27 1.27)) hide)
+    )
+    (property "Datasheet" "" (at 39.37 138.43 0)
+      (effects (font (size 1.27 1.27)) hide)
+    )

Commit message: [WIP] symbol-footprint association
Parts:
- C201, C202, C203, C204, C205, C212, C213, C214, C215, C216, C217, C220, C225: footprint (none) -> Capacitor_SMD:C_0402_1005Metric
- C206, C207, C208, C209, C210, C211, C218, C219, C221, C222, C223, C224: footprint (none) -> Capacitor_SMD:C_0805_2012Metric
- F201: footprint (none) -> Fuse:Fuse_1812_4532Metric
- J201, JP201: footprint (none) -> Connector_PinHeader_2.54mm:PinHeader_1x02_P2.54mm_Vertical
- L201, L202: footprint (none) -> Inductor_SMD:L_Taiyo-Yuden_NR-50xx
- R201, R202, R203, R204, R205, R206, R207, R208, R209, R210, R211, R212, R213, R214: footprint (none) -> Resistor_SMD:R_0402_1005Metric
- SW201: value SW_Push -> 1571300-2; Manufacturer (none) -> TE Connectivity
- TP201, TP202, TP203, TP204, TP205, TP206: footprint (none) -> TestPoint:TestPoint_Loop_D2.50mm_Drill1.0mm

Commit message: Fixed BST capacitor placement
Parts:
- SW201: value 1571300-2 -> ~
Connections:
- net +1V8: no longer C215.2
- net +3.3V: no longer C214.2
- net at L202.1, U202.10 (LX2): now also C215.2
- net at L201.1, U202.26 (LX1): now also C214.2
Other:
- moved on the sheet: C214, C215, L201, L202
Changed lines of the file:
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@@
   (junction (at 123.19 106.68) (diameter 0) (color 0 0 0 0)
   )
+  (junction (at 185.42 39.37) (diameter 0) (color 0 0 0 0)
+  )
   (junction (at 111.76 91.44) (diameter 0) (color 0 0 0 0)
   )
-  (junction (at 187.96 39.37) (diameter 0) (color 0 0 0 0)
-  )
-  (junction (at 187.96 91.44) (diameter 0) (color 0 0 0 0)
+  (junction (at 185.42 91.44) (diameter 0) (color 0 0 0 0)
   )
   (junction (at 39.37 107.95) (diameter 0) (color 0 0 0 0)
@@
     (stroke (width 0) (type default))
   )
+  (wire (pts (xy 185.42 39.37) (xy 191.77 39.37))
+    (stroke (width 0) (type default))
+  )
   (wire (pts (xy 134.62 54.61) (xy 146.05 54.61))
     (stroke (width 0) (type default))
@@
     (stroke (width 0) (type default))
   )
-  (wire (pts (xy 186.69 95.25) (xy 187.96 95.25))
+  (wire (pts (xy 184.15 95.25) (xy 185.42 95.25))
     (stroke (width 0) (type default))
   )
@@
     (stroke (width 0) (type default))
   )
-  (wire (pts (xy 184.15 39.37) (xy 187.96 39.37))
+  (wire (pts (xy 173.99 39.37) (xy 185.42 39.37))
     (stroke (width 0) (type default))
   )
@@
     (stroke (width 0) (type default))
   )
-  (wire (pts (xy 186.69 43.18) (xy 187.96 43.18))
+  (wire (pts (xy 184.15 43.18) (xy 185.42 43.18))
     (stroke (width 0) (type default))
   )
@@
     (stroke (width 0) (type default))
   )
-  (wire (pts (xy 187.96 91.44) (xy 203.2 91.44))
-    (stroke (width 0) (type default))
-  )
   (wire (pts (xy 134.62 39.37) (xy 134.62 43.18))
     (stroke (width 0) (type default))
@@
     (stroke (width 0) (type default))
   )
-  (wire (pts (xy 173.99 95.25) (xy 179.07 95.25))
+  (wire (pts (xy 173.99 95.25) (xy 176.53 95.25))
     (stroke (width 0) (type default))
   )
@@
     (stroke (width 0) (type default))
   )
+  (wire (pts (xy 199.39 91.44) (xy 203.2 91.44))
+    (stroke (width 0) (type default))
+  )
   (wire (pts (xy 254 137.16) (xy 254 135.89))
     (stroke (width 0) (type default))
@@
     (stroke (width 0) (type default))
   )
-  (wire (pts (xy 173.99 39.37) (xy 176.53 39.37))
-    (stroke (width 0) (type default))
-  )
   (wire (pts (xy 123.19 106.68) (xy 134.62 106.68))
     (stroke (width 0) (type default))
@@
     (stroke (width 0) (type default))
   )
-  (wire (pts (xy 184.15 91.44) (xy 187.96 91.44))
-    (stroke (width 0) (type default))
-  )
   (wire (pts (xy 77.47 104.14) (xy 87.63 104.14))
     (stroke (width 0) (type default))
   )
-  (wire (pts (xy 173.99 91.44) (xy 176.53 91.44))
+  (wire (pts (xy 173.99 91.44) (xy 185.42 91.44))
     (stroke (width 0) (type default))
   )
@@
     (stroke (width 0) (type default))
   )
-  (wire (pts (xy 187.96 91.44) (xy 187.96 95.25))
+  (wire (pts (xy 185.42 91.44) (xy 185.42 95.25))
     (stroke (width 0) (type default))
   )
@@
     (stroke (width 0) (type default))
   )
-  (wire (pts (xy 173.99 43.18) (xy 179.07 43.18))
+  (wire (pts (xy 173.99 43.18) (xy 176.53 43.18))
     (stroke (width 0) (type default))
   )
@@
     (stroke (width 0) (type default))
   )
+  (wire (pts (xy 185.42 91.44) (xy 191.77 91.44))
+    (stroke (width 0) (type default))
+  )
   (wire (pts (xy 34.29 80.01) (xy 35.56 80.01))
     (stroke (width 0) (type default))
   )
+  (wire (pts (xy 199.39 39.37) (xy 203.2 39.37))
+    (stroke (width 0) (type default))
+  )
   (wire (pts (xy 203.2 48.26) (xy 203.2 49.53))
     (stroke (width 0) (type default))
@@
     (stroke (width 0) (type default))
   )
-  (wire (pts (xy 187.96 39.37) (xy 187.96 43.18))
+  (wire (pts (xy 185.42 39.37) (xy 185.42 43.18))
     (stroke (width 0) (type default))
   )
@@
   )
   (wire (pts (xy 254 135.89) (xy 267.97 135.89))
-    (stroke (width 0) (type default))
-  )
-  (wire (pts (xy 187.96 39.37) (xy 203.2 39.37))
     (stroke (width 0) (type default))
   )
@@
     )
   )
-  (symbol (lib_id "Device:L") (at 180.34 91.44 90) (unit 1)
-    (in_bom yes) (on_board yes) (dnp no)
-    (property "Reference" "L202" (at 180.34 87.63 90)
-      (effects (font (size 1.27 1.27)))
-    )
-    (property "Value" "47uH" (at 180.34 90.17 90)
-      (effects (font (size 1.27 1.27)))
-    )
-    (property "Footprint" "Inductor_SMD:L_Taiyo-Yuden_NR-50xx" (at 180.34 91.44 0)
-      (effects (font (size 1.27 1.27)) hide)
-    )
-    (property "Datasheet" "~" (at 180.34 91.44 0)
-      (effects (font (size 1.27 1.27)) hide)
-    )
-    (property "MPN" "NRS5030T470MMGJ" (at 180.34 85.09 90)
+  (symbol (lib_id "Device:L") (at 195.58 91.44 90) (unit 1)
+    (in_bom yes) (on_board yes) (dnp no)
+    (property "Reference" "L202" (at 195.58 87.63 90)
+      (effects (font (size 1.27 1.27)))
+    )
+    (property "Value" "47uH" (at 195.58 90.17 90)
+      (effects (font (size 1.27 1.27)))
+    )
+    (property "Footprint" "Inductor_SMD:L_Taiyo-Yuden_NR-50xx" (at 195.58 91.44 0)
+      (effects (font (size 1.27 1.27)) hide)
+    )
+    (property "Datasheet" "~" (at 195.58 91.44 0)
+      (effects (font (size 1.27 1.27)) hide)
+    )
+    (property "MPN" "NRS5030T470MMGJ" (at 195.58 85.09 90)
       (effects (font (size 1.27 1.27)))
     )
@@
     )
   )
-  (symbol (lib_id "Device:C") (at 182.88 95.25 90) (unit 1)
-    (in_bom yes) (on_board yes) (dnp no)
-    (property "Reference" "C215" (at 179.07 93.98 90)
-      (effects (font (size 1.27 1.27)))
-    )
-    (property "Value" "47nF" (at 179.07 96.52 90)
-      (effects (font (size 1.27 1.27)))
-    )
-    (property "Footprint" "Capacitor_SMD:C_0402_1005Metric" (at 186.69 94.2848 0)
-      (effects (font (size 1.27 1.27)) hide)
-    )
-    (property "Datasheet" "~" (at 182.88 95.25 0)
-      (effects (font (size 1.27 1.27)) hide)
-    )
-    (property "Dielectric" "X5R or better" (at 193.04 93.98 90)
-      (effects (font (size 1.27 1.27)))
-    )
-    (property "Voltage" "10V or higher" (at 193.04 96.52 90)
+  (symbol (lib_id "Device:C") (at 180.34 95.25 90) (unit 1)
+    (in_bom yes) (on_board yes) (dnp no)
+    (property "Reference" "C215" (at 176.53 93.98 90)
+      (effects (font (size 1.27 1.27)))
+    )
+    (property "Value" "47nF" (at 176.53 96.52 90)
+      (effects (font (size 1.27 1.27)))
+    )
+    (property "Footprint" "Capacitor_SMD:C_0402_1005Metric" (at 184.15 94.2848 0)
+      (effects (font (size 1.27 1.27)) hide)
+    )
+    (property "Datasheet" "~" (at 180.34 95.25 0)
+      (effects (font (size 1.27 1.27)) hide)
+    )
+    (property "Dielectric" "X5R or better" (at 180.34 87.63 90)
+      (effects (font (size 1.27 1.27)))
+    )
+    (property "Voltage" "10V or higher" (at 180.34 90.17 90)
       (effects (font (size 1.27 1.27)))
     )
@@
     )
   )
-  (symbol (lib_id "Device:L") (at 180.34 39.37 90) (unit 1)
-    (in_bom yes) (on_board yes) (dnp no)
-    (property "Reference" "L201" (at 180.34 35.56 90)
-      (effects (font (size 1.27 1.27)))
-    )
-    (property "Value" "33uH" (at 180.34 38.1 90)
-      (effects (font (size 1.27 1.27)))
-    )
-    (property "Footprint" "Inductor_SMD:L_Taiyo-Yuden_NR-50xx" (at 180.34 39.37 0)
-      (effects (font (size 1.27 1.27)) hide)
-    )
-    (property "Datasheet" "~" (at 180.34 39.37 0)
-      (effects (font (size 1.27 1.27)) hide)
-    )
-    (property "MPN" "NRS5030T330MMGJ" (at 180.34 33.02 90)
+  (symbol (lib_id "Device:L") (at 195.58 39.37 90) (unit 1)
+    (in_bom yes) (on_board yes) (dnp no)
+    (property "Reference" "L201" (at 195.58 35.56 90)
+      (effects (font (size 1.27 1.27)))
+    )
+    (property "Value" "33uH" (at 195.58 38.1 90)
+      (effects (font (size 1.27 1.27)))
+    )
+    (property "Footprint" "Inductor_SMD:L_Taiyo-Yuden_NR-50xx" (at 195.58 39.37 0)
+      (effects (font (size 1.27 1.27)) hide)
+    )
+    (property "Datasheet" "~" (at 195.58 39.37 0)
+      (effects (font (size 1.27 1.27)) hide)
+    )
+    (property "MPN" "NRS5030T330MMGJ" (at 195.58 33.02 90)
       (effects (font (size 1.27 1.27)))
     )
@@
     )
   )
-  (symbol (lib_id "Device:C") (at 182.88 43.18 90) (unit 1)
-    (in_bom yes) (on_board yes) (dnp no)
-    (property "Reference" "C214" (at 179.07 41.91 90)
-      (effects (font (size 1.27 1.27)))
-    )
-    (property "Value" "47nF" (at 179.07 44.45 90)
-      (effects (font (size 1.27 1.27)))
-    )
-    (property "Footprint" "Capacitor_SMD:C_0402_1005Metric" (at 186.69 42.2148 0)
-      (effects (font (size 1.27 1.27)) hide)
-    )
-    (property "Datasheet" "~" (at 182.88 43.18 0)
-      (effects (font (size 1.27 1.27)) hide)
-    )
-    (property "Dielectric" "X5R or better" (at 193.04 41.91 90)
-      (effects (font (size 1.27 1.27)))
-    )
-    (property "Voltage" "10V or higher" (at 193.04 44.45 90)
+  (symbol (lib_id "Device:C") (at 180.34 43.18 90) (unit 1)
+    (in_bom yes) (on_board yes) (dnp no)
+    (property "Reference" "C214" (at 176.53 41.91 90)
+      (effects (font (size 1.27 1.27)))
+    )
+    (property "Value" "47nF" (at 176.53 44.45 90)
+      (effects (font (size 1.27 1.27)))
+    )
+    (property "Footprint" "Capacitor_SMD:C_0402_1005Metric" (at 184.15 42.2148 0)
+      (effects (font (size 1.27 1.27)) hide)
+    )
+    (property "Datasheet" "~" (at 180.34 43.18 0)
+      (effects (font (size 1.27 1.27)) hide)
+    )
+    (property "Dielectric" "X5R or better" (at 180.34 35.56 90)
+      (effects (font (size 1.27 1.27)))
+    )
+    (property "Voltage" "10V or higher" (at 180.34 38.1 90)
       (effects (font (size 1.27 1.27)))
     )
@@
       (effects (font (size 1.27 1.27)) (justify left))
     )
-    (property "Value" "1571300-2" (at 36.83 46.355 90)
-      (effects (font (size 1.27 1.27)) (justify left))
-    )
+    (property "Value" "~" (at 36.83 46.355 90)
+      (effects (font (size 1.27 1.27)) (justify left))
+    )

Commit message: Updated M17_kicad_library
Connections:
- net GND: now also U202.27 (PGND1); no longer U202. (PGND1)
Changed lines of the file:
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@@
     (pin "4")
     (pin "5")
-    (pin "")
     (pin "22")
     (pin "23")
@@
     (pin "25")
     (pin "26")
+    (pin "27")
     (pin "28")
     (pin "31")
@@
     (pin "4")
     (pin "5")
-    (pin "")
     (pin "22")
     (pin "23")
@@
     (pin "25")
     (pin "26")
+    (pin "27")
     (pin "28")
     (pin "31")
@@
     (pin "4")
     (pin "5")
-    (pin "")
     (pin "22")
     (pin "23")
@@
     (pin "25")
     (pin "26")
+    (pin "27")
     (pin "28")
     (pin "31")
@@
     (pin "4")
     (pin "5")
-    (pin "")
     (pin "22")
     (pin "23")
@@
     (pin "25")
     (pin "26")
+    (pin "27")
     (pin "28")
     (pin "31")

Commit message: Updated switches
Parts:
- SW201: value ~ -> 436351045816; footprint (none) -> M17_misc_passive:SW_SPST_436351045816
Changed lines of the file:
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@@
       (effects (font (size 1.27 1.27)) (justify left))
     )
-    (property "Value" "~" (at 36.83 46.355 90)
+    (property "Value" "436351045816" (at 36.83 46.355 90)
       (effects (font (size 1.27 1.27)) (justify left))
     )
-    (property "Footprint" "" (at 35.56 44.45 0)
+    (property "Footprint" "M17_misc_passive:SW_SPST_436351045816" (at 35.56 44.45 0)
       (effects (font (size 1.27 1.27)) hide)
     )

Commit message: Fixed 3.3V power symbol
Use 3V3 everywhere instead of 3.3
Connections:
- net +3.3V is gone; now on net +3V3: C218.1, C221.1, C223.1, L201.2, R209.1
Changed lines of the file:
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@@
-    )
-  )
-  (symbol (lib_id "power:+3.3V") (at 246.38 39.37 0) (unit 1)
-    (in_bom yes) (on_board yes) (dnp no) (fields_autoplaced)
-    (property "Reference" "#PWR0239" (at 246.38 43.18 0)
-      (effects (font (size 1.27 1.27)) hide)
-    )
-    (property "Value" "+3.3V" (at 246.38 35.56 0)
-      (effects (font (size 1.27 1.27)))
-    )
-    (property "Footprint" "" (at 246.38 39.37 0)
-      (effects (font (size 1.27 1.27)) hide)
-    )
-    (property "Datasheet" "" (at 246.38 39.37 0)
-      (effects (font (size 1.27 1.27)) hide)
-    )
-    (pin "1")
-    (instances
-      (project "OpenHT-RF"
-        (path "/3c300b59-23ec-47f8-bb91-29ca34130bcf/17571ff2-f5b8-49d7-92c6-d2c188350dd2"
-          (reference "#PWR0239") (unit 1)
-        )
-      )
     )
   )
@@
         )
       )
+    )
+  )
+  (symbol (lib_id "power:+3V3") (at 246.38 39.37 0) (unit 1)
+    (in_bom yes) (on_board yes) (dnp no) (fields_autoplaced)
+    (property "Reference" "#PWR0244" (at 246.38 43.18 0)
+      (effects (font (size 1.27 1.27)) hide)
+    )
+    (property "Value" "+3V3" (at 246.38 35.56 0)
+      (effects (font (size 1.27 1.27)))
+    )
+    (property "Footprint" "" (at 246.38 39.37 0)
+      (effects (font (size 1.27 1.27)) hide)
+    )
+    (property "Datasheet" "" (at 246.38 39.37 0)
+      (effects (font (size 1.27 1.27)) hide)
+    )
+    (pin "1")
+    (instances
+      (project "OpenHT-RF"
+        (path "/3c300b59-23ec-47f8-bb91-29ca34130bcf/17571ff2-f5b8-49d7-92c6-d2c188350dd2"
+          (reference "#PWR0244") (unit 1)
+        )
+      )
