File: OpenHT-RF/pwr.kicad_sch (KiCad schematic)
At the start: 64 parts, among them J201 Conn_01x02, J202 MS338-10F, Q201 DMP3099L-7, SW201 436351045816, U201 LTC2954-1, U202 TPS65261RHBx, U203 AP7330-W5-7, U204 TPS22810DBVR

Commit message: Added DC-DC shield
Parts:
- J202: footprint (none) -> M17_misc_passive:MS338-10F
- L201: footprint Inductor_SMD:L_Taiyo-Yuden_NR-50xx -> M17_misc_passive:L_Taiyo-Yuden_NR-5030
Changed lines of the file:
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@@
       (effects (font (size 1.27 1.27)))
     )
-    (property "Footprint" "Inductor_SMD:L_Taiyo-Yuden_NR-50xx" (at 196.85 38.1 0)
+    (property "Footprint" "M17_misc_passive:L_Taiyo-Yuden_NR-5030" (at 196.85 38.1 0)
       (effects (font (size 1.27 1.27)) hide)
     )
@@
       (effects (font (size 1.27 1.27)) (justify left))
     )
-    (property "Footprint" "" (at 132.08 182.88 0)
-      (effects (font (size 1.27 1.27)) hide)
-    )
+    (property "Footprint" "M17_misc_passive:MS338-10F" (at 132.08 182.88 0)
+      (effects (font (size 1.27 1.27)) hide)
+    )
