File: OpenHT-RF/pwr.kicad_sch (KiCad schematic)
At the start: 69 parts, among them J201 Conn_01x02, J202 MS338-10F, Q201 DMP3099L-7, SW201 436351045816, U201 LTC2954-1, U202 TPS65261RHBx, U203 AP7330-W5-7, U204 TPS22810DBVR

Commit message: Fixed ERC errors
Parts:
- F201: MPN (none) -> SMD1812B200TF/16
Other:
- moved on the sheet: C203, C204, F201, J201, Q201, R202, SW201, TP201, TP202, TP203, TP204, TP205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

Commit message: Modified shields to use two symbols
Allows to have the MPN of the lid in the schematic alongside the frame
Parts:
- removed J202: MS338-10F, M17_misc_passive:MS338-10F, symbol Device:RFShield_TwoPieces
- added J202: MS338-10F, M17_misc_passive:MS338-10F, symbol M17_device:RFShield_Frame
- added J203: MS338-10C, symbol M17_device:RFShield_Lid
Connections:
- net GND: now also J202.1 (Shield)
Changed lines of the file:
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@@
+    )
+  )
+  (symbol (lib_id "M17_device:RFShield_Frame") (at 132.08 180.34 0) (unit 1)
+    (in_bom yes) (on_board yes) (dnp no)
+    (property "Reference" "J202" (at 151.13 177.8 0)
+      (effects (font (size 1.27 1.27)) (justify left))
+    )
+    (property "Value" "MS338-10F" (at 151.13 180.34 0)
+      (effects (font (size 1.27 1.27)) (justify left))
+    )
+    (property "Footprint" "M17_misc_passive:MS338-10F" (at 132.08 180.34 0)
+      (effects (font (size 1.27 1.27)) hide)
+    )
+    (property "Datasheet" "" (at 132.08 180.34 0)
+      (effects (font (size 1.27 1.27)) hide)
+    )
+    (property "MPN" "MS338-10F" (at 132.08 180.34 0)
+      (effects (font (size 1.27 1.27)) hide)
+    )
+    (pin "1")
+    (instances
+      (project "OpenHT-RF"
+        (path "/3c300b59-23ec-47f8-bb91-29ca34130bcf/17571ff2-f5b8-49d7-92c6-d2c188350dd2"
+          (reference "J202") (unit 1)
+        )
+      )
     )
   )
@@
     )
   )
+  (symbol (lib_id "M17_device:RFShield_Lid") (at 132.08 172.72 0) (unit 1)
+    (in_bom yes) (on_board no) (dnp no)
+    (property "Reference" "J203" (at 132.08 165.1 0)
+      (effects (font (size 1.27 1.27)))
+    )
+    (property "Value" "MS338-10C" (at 132.08 167.64 0)
+      (effects (font (size 1.27 1.27)))
+    )
+    (property "Footprint" "" (at 132.08 180.34 0)
+      (effects (font (size 1.27 1.27)) hide)
+    )
+    (property "Datasheet" "" (at 132.08 180.34 0)
+      (effects (font (size 1.27 1.27)) hide)
+    )
+    (property "MPN" "MS338-10C" (at 132.08 172.72 0)
+      (effects (font (size 1.27 1.27)) hide)
+    )
+    (instances
+      (project "OpenHT-RF"
+        (path "/3c300b59-23ec-47f8-bb91-29ca34130bcf/17571ff2-f5b8-49d7-92c6-d2c188350dd2"
+          (reference "J203") (unit 1)
+        )
+      )
+    )
+  )
   (symbol (lib_id "power:PWR_FLAG") (at 62.23 21.59 0) (unit 1)
     (in_bom yes) (on_board yes) (dnp no) (fields_autoplaced)
@@
         )
       )
-    )
-  )
-  (symbol (lib_id "Device:RFShield_TwoPieces") (at 132.08 180.34 0) (unit 1)
-    (in_bom yes) (on_board yes) (dnp no) (fields_autoplaced)
-    (property "Reference" "J202" (at 151.13 177.8 0)
-      (effects (font (size 1.27 1.27)) (justify left))
-    )
-    (property "Value" "MS338-10F" (at 151.13 180.34 0)
-      (effects (font (size 1.27 1.27)) (justify left))
-    )
-    (property "Footprint" "M17_misc_passive:MS338-10F" (at 132.08 182.88 0)
-      (effects (font (size 1.27 1.27)) hide)
-    )
-    (property "Datasheet" "~" (at 132.08 182.88 0)
-      (effects (font (size 1.27 1.27)) hide)
-    )
-    (property "MPN" "MS338-10F" (at 132.08 180.34 0)
-      (effects (font (size 1.27 1.27)) hide)
-    )
-    (pin "1")
-    (instances
-      (project "OpenHT-RF"
-        (path "/3c300b59-23ec-47f8-bb91-29ca34130bcf/17571ff2-f5b8-49d7-92c6-d2c188350dd2"
-          (reference "J202") (unit 1)
-        )
-      )

Commit message: Completed components values
Completed dielectric, rated voltage, tolerance, MPN
Parts:
- C227: value 100nF -> 0.1uF
- J203: Manual_Placement (none) -> 1
- R201, R202, R203, R204, R205, R206, R207, R208, R213, R214, R301: Tolerance (none) -> 1%
Changed lines of the file:
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@@
       (effects (font (size 1.27 1.27)) hide)
     )
+    (property "Tolerance" "1%" (at 82.55 96.52 0)
+      (effects (font (size 1.27 1.27)) hide)
+    )
     (pin "1")
     (pin "2")
@@
       (effects (font (size 1.27 1.27)) hide)
     )
+    (property "Tolerance" "1%" (at 189.23 57.15 0)
+      (effects (font (size 1.27 1.27)) hide)
+    )
     (pin "1")
     (pin "2")
@@
       (effects (font (size 1.27 1.27)) hide)
     )
+    (property "Tolerance" "1%" (at 57.15 29.21 0)
+      (effects (font (size 1.27 1.27)) hide)
+    )
     (pin "1")
     (pin "2")
@@
       (effects (font (size 1.27 1.27)) hide)
     )
+    (property "Tolerance" "1%" (at 96.52 171.45 0)
+      (effects (font (size 1.27 1.27)) hide)
+    )
     (pin "1")
     (pin "2")
@@
       (effects (font (size 1.27 1.27)) hide)
     )
+    (property "Tolerance" "1%" (at 231.14 144.78 0)
+      (effects (font (size 1.27 1.27)) hide)
+    )
     (pin "1")
     (pin "2")
@@
       (effects (font (size 1.27 1.27)) hide)
     )
+    (property "Tolerance" "1%" (at 77.47 96.52 0)
+      (effects (font (size 1.27 1.27)) hide)
+    )
     (pin "1")
     (pin "2")
@@
       (effects (font (size 1.27 1.27)) hide)
     )
+    (property "Tolerance" "1%" (at 189.23 109.22 0)
+      (effects (font (size 1.27 1.27)) hide)
+    )
     (pin "1")
     (pin "2")
@@
       (effects (font (size 1.27 1.27)) hide)
     )
+    (property "Manual_Placement" "1" (at 132.08 172.72 0)
+      (effects (font (size 1.27 1.27)) hide)
+    )
     (instances
       (project "OpenHT-RF"
@@
       (effects (font (size 1.27 1.27)) hide)
     )
+    (property "Tolerance" "1%" (at 34.29 107.95 0)
+      (effects (font (size 1.27 1.27)) hide)
+    )
     (pin "1")
     (pin "2")
@@
       (effects (font (size 1.27 1.27)) (justify left))
     )
-    (property "Value" "100nF" (at 52.07 177.165 0)
+    (property "Value" "0.1uF" (at 52.07 177.165 0)
       (effects (font (size 1.27 1.27)) (justify left))
     )
@@
       (effects (font (size 1.27 1.27)) hide)
     )
+    (property "Tolerance" "1%" (at 39.37 115.57 0)
+      (effects (font (size 1.27 1.27)) hide)
+    )
     (pin "1")
     (pin "2")
@@
       (effects (font (size 1.27 1.27)) hide)
     )
+    (property "Tolerance" "1%" (at 231.14 154.94 0)
+      (effects (font (size 1.27 1.27)) hide)
+    )
     (pin "1")
     (pin "2")
@@
       (effects (font (size 1.27 1.27)) hide)
     )
+    (property "Tolerance" "1%" (at 74.93 124.46 0)
+      (effects (font (size 1.27 1.27)) hide)
+    )

Commit message: Added MPN for SMD jumpers
Parts:
- JP201, JP202, JP203, JP204: MPN (none) -> 10129380-902001BLF or equivalent
Changed lines of the file:
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@@
       (effects (font (size 1.27 1.27)) hide)
     )
+    (property "MPN" "10129380-902001BLF or equivalent" (at 39.37 129.54 0)
+      (effects (font (size 1.27 1.27)) hide)
+    )
     (pin "1")
     (pin "2")
@@
       (effects (font (size 1.27 1.27)) hide)
     )
+    (property "MPN" "10129380-902001BLF or equivalent" (at 270.51 90.17 0)
+      (effects (font (size 1.27 1.27)) hide)
+    )
     (pin "1")
     (pin "2")
@@
       (effects (font (size 1.27 1.27)) hide)
     )
+    (property "MPN" "10129380-902001BLF or equivalent" (at 270.51 38.1 0)
+      (effects (font (size 1.27 1.27)) hide)
+    )
     (pin "1")
     (pin "2")
@@
       (effects (font (size 1.27 1.27)) hide)
     )
+    (property "MPN" "10129380-902001BLF or equivalent" (at 255.27 139.7 0)
+      (effects (font (size 1.27 1.27)) hide)
+    )

Commit message: Fixed tolerance for R214
Parts:
- R214: Tolerance 1% -> 0.1%
Changed lines of the file:
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@@
       (effects (font (size 1.27 1.27)) hide)
     )
-    (property "Tolerance" "1%" (at 231.14 154.94 0)
+    (property "Tolerance" "0.1%" (at 231.14 154.94 0)
       (effects (font (size 1.27 1.27)) hide)
     )

Commit message: Added MPN for generic components
Parts:
- C201, C205, C220, C225: MPN (none) -> Generic C/1uF/0402/X5R/10V
- C202: MPN (none) -> Generic C/18nF/0402/X7R/10V
- C203, C204: MPN (none) -> Generic C/0.15uF/0402/X5R/10V
- C206, C207, C208, C209, C210, C211, C218, C219, C221, C222, C223, C224: MPN (none) -> Generic C/0.15uF/0805/X5R/25V
- C212: MPN (none) -> Generic C/3.9pF/0402/C0G/10V
- C213: MPN (none) -> Generic C/4.5pF/0402/C0G/10V
- C214, C215: MPN (none) -> Generic C/47nF/0402/X5R/10V
- C216: MPN (none) -> Generic C/1.2nF/0402/X7R/10V
- C217: MPN (none) -> Generic C/1nF/0402/X7R/10V
- C226: MPN (none) -> Generic C/6.8nF/0402/X5R/10V
- C227: MPN (none) -> Generic C/0.1uF/0402/X7R/16V
- C228, C229: MPN (none) -> Generic C/470pF/0402/X7R/16V
- R201: MPN (none) -> Generic R/200kR/0402/1%
- R202: MPN (none) -> Generic R/1kR/0402/1%
- R203: MPN (none) -> Generic R/47.5kR/0402/1%
- R204: MPN (none) -> Generic R/110kR/0402/1%
- R205, R206: MPN (none) -> Generic R/100kR/0402/1%
- R207: MPN (none) -> Generic R/1.6kR/0402/1%
- R208: MPN (none) -> Generic R/3.16kR/0402/1%
- R209: MPN (none) -> Generic R/43kR/0402/0.1%
- R210: MPN (none) -> Generic R/9.53kR/0402/0.1%
- R211: MPN (none) -> Generic R/20kR/0402/0.1%
- R212: MPN (none) -> Generic R/10kR/0402/0.1%
- R213: MPN (none) -> Generic R/2.55kR/0402/1%
- R214: MPN (none) -> Generic R/10.2kR/0402/0.1%
- R301: MPN (none) -> Generic R/100R/0402/1%
Changed lines of the file:
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@@
       (effects (font (size 1.27 1.27)))
     )
+    (property "MPN" "Generic C/0.15uF/0805/X5R/25V" (at 124.46 97.79 0)
+      (effects (font (size 1.27 1.27)) hide)
+    )
     (pin "1")
     (pin "2")
@@
       (effects (font (size 1.27 1.27)) hide)
     )
+    (property "MPN" "Generic R/100kR/0402/1%" (at 82.55 96.52 0)
+      (effects (font (size 1.27 1.27)) hide)
+    )
     (pin "1")
     (pin "2")
@@
       (effects (font (size 1.27 1.27)))
     )
+    (property "MPN" "Generic C/0.15uF/0805/X5R/25V" (at 260.35 96.52 0)
+      (effects (font (size 1.27 1.27)) hide)
+    )
     (pin "1")
     (pin "2")
@@
       (effects (font (size 1.27 1.27)) hide)
     )
+    (property "MPN" "Generic C/1uF/0402/X5R/10V" (at 194.31 144.78 0)
+      (effects (font (size 1.27 1.27)) hide)
+    )
     (pin "1")
     (pin "2")
@@
       (effects (font (size 1.27 1.27)))
     )
+    (property "MPN" "Generic C/0.15uF/0805/X5R/25V" (at 260.35 44.45 0)
+      (effects (font (size 1.27 1.27)) hide)
+    )
     (pin "1")
     (pin "2")
@@
       (effects (font (size 1.27 1.27)) hide)
     )
+    (property "MPN" "Generic C/470pF/0402/X7R/16V" (at 215.9 95.25 0)
+      (effects (font (size 1.27 1.27)) hide)
+    )
     (pin "1")
     (pin "2")
@@
       (effects (font (size 1.27 1.27)) hide)
     )
+    (property "MPN" "Generic C/0.15uF/0402/X5R/10V" (at 87.63 50.8 0)
+      (effects (font (size 1.27 1.27)) hide)
+    )
     (pin "1")
     (pin "2")
@@
       (effects (font (size 1.27 1.27)) hide)
     )
+    (property "MPN" "Generic R/1.6kR/0402/1%" (at 189.23 57.15 0)
+      (effects (font (size 1.27 1.27)) hide)
+    )
     (pin "1")
     (pin "2")
@@
       (effects (font (size 1.27 1.27)))
     )
+    (property "MPN" "Generic C/0.15uF/0805/X5R/25V" (at 124.46 45.72 0)
+      (effects (font (size 1.27 1.27)) hide)
+    )
     (pin "1")
     (pin "2")
@@
       (effects (font (size 1.27 1.27)))
     )
+    (property "MPN" "Generic C/0.15uF/0805/X5R/25V" (at 248.92 96.52 0)
+      (effects (font (size 1.27 1.27)) hide)
+    )
     (pin "1")
     (pin "2")
@@
       (effects (font (size 1.27 1.27)))
     )
+    (property "MPN" "Generic C/0.15uF/0805/X5R/25V" (at 237.49 96.52 0)
+      (effects (font (size 1.27 1.27)) hide)
+    )
     (pin "1")
     (pin "2")
@@
       (effects (font (size 1.27 1.27)) hide)
     )
+    (property "MPN" "Generic C/4.5pF/0402/C0G/10V" (at 181.61 113.03 0)
+      (effects (font (size 1.27 1.27)) hide)
+    )
     (pin "1")
     (pin "2")
@@
       (effects (font (size 1.27 1.27)) hide)
     )
+    (property "MPN" "Generic R/1kR/0402/1%" (at 57.15 29.21 0)
+      (effects (font (size 1.27 1.27)) hide)
+    )
     (pin "1")
     (pin "2")
@@
       (effects (font (size 1.27 1.27)))
     )
+    (property "MPN" "Generic C/0.15uF/0805/X5R/25V" (at 113.03 97.79 0)
+      (effects (font (size 1.27 1.27)) hide)
+    )
     (pin "1")
     (pin "2")
@@
       (effects (font (size 1.27 1.27)) hide)
     )
+    (property "MPN" "Generic R/43kR/0402/0.1%" (at 204.47 43.18 0)
+      (effects (font (size 1.27 1.27)) hide)
+    )
     (pin "1")
     (pin "2")
@@
       (effects (font (size 1.27 1.27)) hide)
     )
+    (property "MPN" "Generic C/470pF/0402/X7R/16V" (at 215.9 43.18 0)
+      (effects (font (size 1.27 1.27)) hide)
+    )
     (pin "1")
     (pin "2")
@@
       (effects (font (size 1.27 1.27)) hide)
     )
+    (property "MPN" "Generic R/100R/0402/1%" (at 96.52 171.45 0)
+      (effects (font (size 1.27 1.27)) hide)
+    )
     (pin "1")
     (pin "2")
@@
       (effects (font (size 1.27 1.27)) hide)
     )
+    (property "MPN" "Generic C/18nF/0402/X7R/10V" (at 59.69 147.32 0)
+      (effects (font (size 1.27 1.27)) hide)
+    )
     (pin "1")
     (pin "2")
@@
       (effects (font (size 1.27 1.27)) hide)
     )
+    (property "MPN" "Generic C/1nF/0402/X7R/10V" (at 189.23 116.84 0)
+      (effects (font (size 1.27 1.27)) hide)
+    )
     (pin "1")
     (pin "2")
@@
       (effects (font (size 1.27 1.27)) hide)
     )
+    (property "MPN" "Generic C/0.15uF/0402/X5R/10V" (at 93.98 50.8 0)
+      (effects (font (size 1.27 1.27)) hide)
+    )
     (pin "1")
     (pin "2")
@@
       (effects (font (size 1.27 1.27)))
     )
+    (property "MPN" "Generic C/47nF/0402/X5R/10V" (at 181.61 93.98 0)
+      (effects (font (size 1.27 1.27)) hide)
+    )
     (pin "1")
     (pin "2")
@@
       (effects (font (size 1.27 1.27)))
     )
+    (property "MPN" "Generic C/0.15uF/0805/X5R/25V" (at 237.49 44.45 0)
+      (effects (font (size 1.27 1.27)) hide)
+    )
     (pin "1")
     (pin "2")
@@
       (effects (font (size 1.27 1.27)) hide)
     )
+    (property "MPN" "Generic C/3.9pF/0402/C0G/10V" (at 181.61 60.96 0)
+      (effects (font (size 1.27 1.27)) hide)
+    )
     (pin "1")
     (pin "2")
@@
       (effects (font (size 1.27 1.27)) hide)
     )
+    (property "MPN" "Generic R/2.55kR/0402/1%" (at 231.14 144.78 0)
+      (effects (font (size 1.27 1.27)) hide)
+    )
     (pin "1")
     (pin "2")
@@
       (effects (font (size 1.27 1.27)) hide)
     )
+    (property "MPN" "Generic R/100kR/0402/1%" (at 77.47 96.52 0)
+      (effects (font (size 1.27 1.27)) hide)
+    )
     (pin "1")
     (pin "2")
@@
       (effects (font (size 1.27 1.27)) hide)
     )
+    (property "MPN" "Generic C/1uF/0402/X5R/10V" (at 25.4 109.22 0)
+      (effects (font (size 1.27 1.27)) hide)
+    )
     (pin "1")
     (pin "2")
@@
       (effects (font (size 1.27 1.27)) hide)
     )
+    (property "MPN" "Generic C/6.8nF/0402/X5R/10V" (at 91.44 180.34 0)
+      (effects (font (size 1.27 1.27)) hide)
+    )
     (pin "1")
     (pin "2")
@@
       (effects (font (size 1.27 1.27)) hide)
     )
+    (property "MPN" "Generic R/3.16kR/0402/1%" (at 189.23 109.22 0)
+      (effects (font (size 1.27 1.27)) hide)
+    )
     (pin "1")
     (pin "2")
@@
       (effects (font (size 1.27 1.27)))
     )
+    (property "MPN" "Generic C/47nF/0402/X5R/10V" (at 181.61 41.91 0)
+      (effects (font (size 1.27 1.27)) hide)
+    )
     (pin "1")
     (pin "2")
@@
       (effects (font (size 1.27 1.27)) hide)
     )
+    (property "MPN" "Generic C/1.2nF/0402/X7R/10V" (at 189.23 64.77 0)
+      (effects (font (size 1.27 1.27)) hide)
+    )
     (pin "1")
     (pin "2")
@@
       (effects (font (size 1.27 1.27)))
     )
+    (property "MPN" "Generic C/0.15uF/0805/X5R/25V" (at 113.03 45.72 0)
+      (effects (font (size 1.27 1.27)) hide)
+    )
     (pin "1")
     (pin "2")
@@
       (effects (font (size 1.27 1.27)) hide)
     )
+    (property "MPN" "Generic R/200kR/0402/1%" (at 34.29 107.95 0)
+      (effects (font (size 1.27 1.27)) hide)
+    )
     (pin "1")
     (pin "2")
@@
       (effects (font (size 1.27 1.27)) hide)
     )
+    (property "MPN" "Generic C/0.1uF/0402/X7R/16V" (at 55.88 175.26 0)
+      (effects (font (size 1.27 1.27)) hide)
+    )
     (pin "1")
     (pin "2")
@@
       (effects (font (size 1.27 1.27)) hide)
     )
+    (property "MPN" "Generic C/1uF/0402/X5R/10V" (at 81.28 124.46 0)
+      (effects (font (size 1.27 1.27)) hide)
+    )
     (pin "1")
     (pin "2")
@@
       (effects (font (size 1.27 1.27)) hide)
     )
+    (property "MPN" "Generic R/47.5kR/0402/1%" (at 39.37 115.57 0)
+      (effects (font (size 1.27 1.27)) hide)
+    )
     (pin "1")
     (pin "2")
@@
       (effects (font (size 1.27 1.27)) hide)
     )
+    (property "MPN" "Generic R/10.2kR/0402/0.1%" (at 231.14 154.94 0)
+      (effects (font (size 1.27 1.27)) hide)
+    )
     (pin "1")
     (pin "2")
@@
       (effects (font (size 1.27 1.27)) hide)
     )
+    (property "MPN" "Generic R/20kR/0402/0.1%" (at 204.47 95.25 0)
+      (effects (font (size 1.27 1.27)) hide)
+    )
     (pin "1")
     (pin "2")
@@
       (effects (font (size 1.27 1.27)))
     )
+    (property "MPN" "Generic C/0.15uF/0805/X5R/25V" (at 248.92 44.45 0)
+      (effects (font (size 1.27 1.27)) hide)
+    )
     (pin "1")
     (pin "2")
@@
       (effects (font (size 1.27 1.27)))
     )
+    (property "MPN" "Generic C/0.15uF/0805/X5R/25V" (at 135.89 45.72 0)
+      (effects (font (size 1.27 1.27)) hide)
+    )
     (pin "1")
     (pin "2")
@@
       (effects (font (size 1.27 1.27)) hide)
     )
+    (property "MPN" "Generic C/1uF/0402/X5R/10V" (at 245.11 144.78 0)
+      (effects (font (size 1.27 1.27)) hide)
+    )
     (pin "1")
     (pin "2")
@@
       (effects (font (size 1.27 1.27)))
     )
+    (property "MPN" "Generic C/0.15uF/0805/X5R/25V" (at 135.89 97.79 0)
+      (effects (font (size 1.27 1.27)) hide)
+    )
     (pin "1")
     (pin "2")
@@
       (effects (font (size 1.27 1.27)) hide)
     )
+    (property "MPN" "Generic R/10kR/0402/0.1%" (at 204.47 105.41 0)
+      (effects (font (size 1.27 1.27)) hide)
+    )
     (pin "1")
     (pin "2")
@@
       (effects (font (size 1.27 1.27)) hide)
     )
+    (property "MPN" "Generic R/9.53kR/0402/0.1%" (at 204.47 53.34 0)
+      (effects (font (size 1.27 1.27)) hide)
+    )
     (pin "1")
     (pin "2")
@@
       (effects (font (size 1.27 1.27)) hide)
     )
+    (property "MPN" "Generic R/110kR/0402/1%" (at 74.93 124.46 0)
+      (effects (font (size 1.27 1.27)) hide)
+    )

Commit message: Fixed incorrect MPN for 4.7uF capacitors
Parts:
- C206, C207, C208, C209, C210, C211, C218, C219, C221, C222, C223, C224: MPN Generic C/0.15uF/0805/X5R/25V -> Generic C/4.7uF/0805/X5R/25V
Changed lines of the file:
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@@
       (effects (font (size 1.27 1.27)))
     )
-    (property "MPN" "Generic C/0.15uF/0805/X5R/25V" (at 124.46 97.79 0)
+    (property "MPN" "Generic C/4.7uF/0805/X5R/25V" (at 124.46 97.79 0)
       (effects (font (size 1.27 1.27)) hide)
     )
@@
       (effects (font (size 1.27 1.27)))
     )
-    (property "MPN" "Generic C/0.15uF/0805/X5R/25V" (at 260.35 96.52 0)
+    (property "MPN" "Generic C/4.7uF/0805/X5R/25V" (at 260.35 96.52 0)
       (effects (font (size 1.27 1.27)) hide)
     )
@@
       (effects (font (size 1.27 1.27)))
     )
-    (property "MPN" "Generic C/0.15uF/0805/X5R/25V" (at 260.35 44.45 0)
+    (property "MPN" "Generic C/4.7uF/0805/X5R/25V" (at 260.35 44.45 0)
       (effects (font (size 1.27 1.27)) hide)
     )
@@
       (effects (font (size 1.27 1.27)))
     )
-    (property "MPN" "Generic C/0.15uF/0805/X5R/25V" (at 124.46 45.72 0)
+    (property "MPN" "Generic C/4.7uF/0805/X5R/25V" (at 124.46 45.72 0)
       (effects (font (size 1.27 1.27)) hide)
     )
@@
       (effects (font (size 1.27 1.27)))
     )
-    (property "MPN" "Generic C/0.15uF/0805/X5R/25V" (at 248.92 96.52 0)
+    (property "MPN" "Generic C/4.7uF/0805/X5R/25V" (at 248.92 96.52 0)
       (effects (font (size 1.27 1.27)) hide)
     )
@@
       (effects (font (size 1.27 1.27)))
     )
-    (property "MPN" "Generic C/0.15uF/0805/X5R/25V" (at 237.49 96.52 0)
+    (property "MPN" "Generic C/4.7uF/0805/X5R/25V" (at 237.49 96.52 0)
       (effects (font (size 1.27 1.27)) hide)
     )
@@
       (effects (font (size 1.27 1.27)))
     )
-    (property "MPN" "Generic C/0.15uF/0805/X5R/25V" (at 113.03 97.79 0)
+    (property "MPN" "Generic C/4.7uF/0805/X5R/25V" (at 113.03 97.79 0)
       (effects (font (size 1.27 1.27)) hide)
     )
@@
       (effects (font (size 1.27 1.27)))
     )
-    (property "MPN" "Generic C/0.15uF/0805/X5R/25V" (at 237.49 44.45 0)
+    (property "MPN" "Generic C/4.7uF/0805/X5R/25V" (at 237.49 44.45 0)
       (effects (font (size 1.27 1.27)) hide)
     )
@@
       (effects (font (size 1.27 1.27)))
     )
-    (property "MPN" "Generic C/0.15uF/0805/X5R/25V" (at 113.03 45.72 0)
+    (property "MPN" "Generic C/4.7uF/0805/X5R/25V" (at 113.03 45.72 0)
       (effects (font (size 1.27 1.27)) hide)
     )
@@
       (effects (font (size 1.27 1.27)))
     )
-    (property "MPN" "Generic C/0.15uF/0805/X5R/25V" (at 248.92 44.45 0)
+    (property "MPN" "Generic C/4.7uF/0805/X5R/25V" (at 248.92 44.45 0)
       (effects (font (size 1.27 1.27)) hide)
     )
@@
       (effects (font (size 1.27 1.27)))
     )
-    (property "MPN" "Generic C/0.15uF/0805/X5R/25V" (at 135.89 45.72 0)
+    (property "MPN" "Generic C/4.7uF/0805/X5R/25V" (at 135.89 45.72 0)
       (effects (font (size 1.27 1.27)) hide)
     )
@@
       (effects (font (size 1.27 1.27)))
     )
-    (property "MPN" "Generic C/0.15uF/0805/X5R/25V" (at 135.89 97.79 0)
+    (property "MPN" "Generic C/4.7uF/0805/X5R/25V" (at 135.89 97.79 0)
       (effects (font (size 1.27 1.27)) hide)
     )

Commit message: Fixed TPS22810DBV pinout
Addresses #1
Parts:
- U204: symbol M17_power:TPS22810DRV -> M17_power:TPS22810DBV
Connections:
- net +BATT: now also U204.1 (VIN); no longer U204.6 (VIN)
- net GND: now also U204.2 (GND); no longer U204.4 (GND)
- net PWR_EN: now also U204.3 (EN/UVLO); no longer U204.5 (EN/UVLO)
- net VDD: now also U204.6 (VOUT); no longer U204.1 (VOUT)
- net at R301.1: now also U204.5 (QOD); no longer U204.2 (QOD)
- net at C226.1: now also U204.4 (CT); no longer U204.3 (CT)
Changed lines of the file:
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@@
     )
   )
-  (symbol (lib_id "M17_power:TPS22810DRV") (at 78.74 171.45 0) (unit 1)
+  (symbol (lib_id "M17_power:TPS22810DBV") (at 78.74 171.45 0) (unit 1)
     (in_bom yes) (on_board yes) (dnp no) (fields_autoplaced)
-    (property "Reference" "U204" (at 78.74 162.56 0)
+    (property "Reference" "U204" (at 78.74 161.29 0)
       (effects (font (size 1.27 1.27)))
     )
-    (property "Value" "TPS22810DBVR" (at 78.74 165.1 0)
+    (property "Value" "TPS22810DBVR" (at 78.74 163.83 0)
       (effects (font (size 1.27 1.27)))
     )
