File: OpenHT-RF/OpenHT-RF.kicad_pcb (KiCad board)
At the start: 2 copper layers, 60 x 127 mm, 160 parts, among them J201 Conn_01x02, J301 Conn_01x06, J302 Conn_01x08, J303 Conn_02x08_Odd_Even, J304 Conn_01x10, J305 Conn_01x08, J401 Conn_01x06, J501 Conn_Coaxial, J502 Conn_01x02, J503 Conn_01x02, SW501 RFSW8008, U201 LTC2954-1, U202 TPS65261RHBx, U203 AP7330-W5-7, U401 LIFCL-40-7SG72I, U501 AT86RF215, X501 ECS-TXO-20CSMV

Commit message: Updated switches
Parts:
- added SW101: 436351045816, M17_misc_passive:SW_SPST_436351045816, F.Cu at (96.5, 151.3)
- added SW201: 436351045816, M17_misc_passive:SW_SPST_436351045816, F.Cu at (96.5, 159.3)
Changed lines of the file:
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@@
     )
+  )
+  (footprint "M17_misc_passive:SW_SPST_436351045816" (layer "F.Cu")
+    (at 96.52 159.266)
+    (descr "Würth Elektronik Right-Angle Tactile SMD Switch 12VDC, 0.05A (https://www.we-online.com/components/products/datasheet/436351045816.pdf)")
+    (tags "SMD Tactile Switch Right-Angle")
+    (property "Manufacturer" "TE Connectivity")
+    (property "Sheetfile" "pwr.kicad_sch")
+    (property "Sheetname" "Power supply")
+    (property "ki_description" "Push button switch, generic, two pins")
+    (property "ki_keywords" "switch normally-open pushbutton push-button")
+    (attr smd)
+    (fp_text reference "SW201" (at 0 -2.54 unlocked) (layer "F.SilkS")
+        (effects (font (size 1 1) (thickness 0.1)))
+    )
+    (fp_text value "436351045816" (at 0 0 unlocked) (layer "F.Fab")
+        (effects (font (size 1 1) (thickness 0.15)))
+    )
+    (fp_text user "${REFERENCE}" (at 0 1.5 unlocked) (layer "F.Fab")
+        (effects (font (size 1 1) (thickness 0.15)))
+    )
+    (fp_line (start -2.35 -1.75) (end -0.55 -1.75)
+      (stroke (width 0.2) (type default)) (layer "F.SilkS"))
+    (fp_line (start -2.35 1.75) (end -0.55 1.75)
+      (stroke (width 0.2) (type default)) (layer "F.SilkS"))
+    (fp_line (start -1.3 2.75) (end -1.3 1.75)
+      (stroke (width 0.2) (type default)) (layer "F.SilkS"))
+    (fp_line (start -1.3 2.75) (end 1.3 2.75)
+      (stroke (width 0.2) (type default)) (layer "F.SilkS"))
+    (fp_line (start 0.55 -1.75) (end 2.35 -1.75)
+      (stroke (width 0.2) (type default)) (layer "F.SilkS"))
+    (fp_line (start 0.55 1.75) (end 2.35 1.75)
+      (stroke (width 0.2) (type default)) (layer "F.SilkS"))
+    (fp_line (start 1.3 1.75) (end 1.3 2.75)
+      (stroke (width 0.2) (type default)) (layer "F.SilkS"))
+    (fp_rect (start -3.6 -1.95) (end 3.6 2.95)
+      (stroke (width 0.1) (type default)) (fill none) (layer "F.CrtYd"))
+    (fp_rect (start -2.35 1.75) (end 2.35 -1.75)
+      (stroke (width 0.1) (type default)) (fill none) (layer "F.Fab"))
+    (pad "" np_thru_hole circle (at 0 -1.375) (size 0.75 0.75) (drill 0.75) (layers "F&B.Cu" "*.Mask"))
+    (pad "" np_thru_hole circle (at 0 1.375) (size 0.75 0.75) (drill 0.75) (layers "F&B.Cu" "*.Mask"))
+    (pad "1" smd roundrect (at -2.8 -0.85) (size 1.2 1) (layers "F.Cu" "F.Paste" "F.Mask") (roundrect_rratio 0.25)
+      (net 125 "Net-(U201-~{PB})") (pinfunction "1") (pintype "passive") (thermal_bridge_angle 45))
+    (pad "1" smd roundrect (at 2.8 -0.85) (size 1.2 1) (layers "F.Cu" "F.Paste" "F.Mask") (roundrect_rratio 0.25)
+      (net 125 "Net-(U201-~{PB})") (pinfunction "1") (pintype "passive") (thermal_bridge_angle 45))
+    (pad "2" smd roundrect (at -2.8 0.85) (size 1.2 1) (layers "F.Cu" "F.Paste" "F.Mask") (roundrect_rratio 0.25)
+      (net 2 "GND") (pinfunction "2") (pintype "passive") (thermal_bridge_angle 45))
+    (pad "2" smd roundrect (at 2.8 0.85) (size 1.2 1) (layers "F.Cu" "F.Paste" "F.Mask") (roundrect_rratio 0.25)
+      (net 2 "GND") (pinfunction "2") (pintype "passive") (thermal_bridge_angle 45))
   )
   (footprint "Resistor_SMD:R_0402_1005Metric" (layer "F.Cu")
@@
     )
   )
+  (footprint "M17_misc_passive:SW_SPST_436351045816" (layer "F.Cu")
+    (at 96.52 151.266)
+    (descr "Würth Elektronik Right-Angle Tactile SMD Switch 12VDC, 0.05A (https://www.we-online.com/components/products/datasheet/436351045816.pdf)")
+    (tags "SMD Tactile Switch Right-Angle")
+    (property "Sheetfile" "OpenHT-RF.kicad_sch")
+    (property "Sheetname" "")
+    (property "ki_description" "Push button switch, generic, two pins")
+    (property "ki_keywords" "switch normally-open pushbutton push-button")
+    (attr smd)
+    (fp_text reference "SW101" (at 0 -2.54 unlocked) (layer "F.SilkS")
+        (effects (font (size 1 1) (thickness 0.1)))
+    )
+    (fp_text value "436351045816" (at 0 0 unlocked) (layer "F.Fab")
+        (effects (font (size 1 1) (thickness 0.15)))
+    )
+    (fp_text user "${REFERENCE}" (at 0 1.5 unlocked) (layer "F.Fab")
+        (effects (font (size 1 1) (thickness 0.15)))
+    )
+    (fp_line (start -2.35 -1.75) (end -0.55 -1.75)
+      (stroke (width 0.2) (type default)) (layer "F.SilkS"))
+    (fp_line (start -2.35 1.75) (end -0.55 1.75)
+      (stroke (width 0.2) (type default)) (layer "F.SilkS"))
+    (fp_line (start -1.3 2.75) (end -1.3 1.75)
+      (stroke (width 0.2) (type default)) (layer "F.SilkS"))
+    (fp_line (start -1.3 2.75) (end 1.3 2.75)
+      (stroke (width 0.2) (type default)) (layer "F.SilkS"))
+    (fp_line (start 0.55 -1.75) (end 2.35 -1.75)
+      (stroke (width 0.2) (type default)) (layer "F.SilkS"))
+    (fp_line (start 0.55 1.75) (end 2.35 1.75)
+      (stroke (width 0.2) (type default)) (layer "F.SilkS"))
+    (fp_line (start 1.3 1.75) (end 1.3 2.75)
+      (stroke (width 0.2) (type default)) (layer "F.SilkS"))
+    (fp_rect (start -3.6 -1.95) (end 3.6 2.95)
+      (stroke (width 0.1) (type default)) (fill none) (layer "F.CrtYd"))
+    (fp_rect (start -2.35 1.75) (end 2.35 -1.75)
+      (stroke (width 0.1) (type default)) (fill none) (layer "F.Fab"))
+    (pad "" np_thru_hole circle (at 0 -1.375) (size 0.75 0.75) (drill 0.75) (layers "F&B.Cu" "*.Mask"))
+    (pad "" np_thru_hole circle (at 0 1.375) (size 0.75 0.75) (drill 0.75) (layers "F&B.Cu" "*.Mask"))
+    (pad "1" smd roundrect (at -2.8 -0.85) (size 1.2 1) (layers "F.Cu" "F.Paste" "F.Mask") (roundrect_rratio 0.25)
+      (net 2 "GND") (pinfunction "1") (pintype "passive") (thermal_bridge_angle 45))
+    (pad "1" smd roundrect (at 2.8 -0.85) (size 1.2 1) (layers "F.Cu" "F.Paste" "F.Mask") (roundrect_rratio 0.25)
+      (net 2 "GND") (pinfunction "1") (pintype "passive") (thermal_bridge_angle 45))
+    (pad "2" smd roundrect (at -2.8 0.85) (size 1.2 1) (layers "F.Cu" "F.Paste" "F.Mask") (roundrect_rratio 0.25)
+      (net 102 "Net-(R101-Pad1)") (pinfunction "2") (pintype "passive") (thermal_bridge_angle 45))
+    (pad "2" smd roundrect (at 2.8 0.85) (size 1.2 1) (layers "F.Cu" "F.Paste" "F.Mask") (roundrect_rratio 0.25)
+      (net 102 "Net-(R101-Pad1)") (pinfunction "2") (pintype "passive") (thermal_bridge_angle 45))
+  )
   (footprint "Capacitor_SMD:C_0402_1005Metric" (layer "F.Cu")

Commit message: Layout [WIP]
Parts:
- U202: footprint M17_QFN:VQFN-32-1EP_5x5mm_P0.5mm_EP3.45x3.45mm -> M17_QFN:VQFN-32-1EP_5x5mm_P0.5mm_EP3.45x3.45mm_ThermalVias
- U401: footprint M17_QFN:QFN-72-1EP_10x10mm_P0.5mm_EP6.2x6.2mm -> M17_QFN:QFN-72-1EP_10x10mm_P0.5mm_EP6.2x6.2mm_ThermalVias
- U501: footprint M17_QFN:VQFN-48-1EP_7x7mm_P0.5mm_EP5.6x5.6mm -> M17_QFN:VQFN-48-1EP_7x7mm_P0.5mm_EP5.6x5.6mm_ThermalVias
- moved C202 121.3 mm to (157.2, 36.7), turned to 180 degrees
- moved C216 104.2 mm to (156.7, 34.2), turned to -90 degrees
- moved C217 101.7 mm to (164.1, 48.1)
- moved R208 101.7 mm to (162.6, 47.6)
- moved R205 100.6 mm to (157.0, 46.1)
- moved R212 100.5 mm to (159.5, 47.6)
- moved R211 100.5 mm to (161.1, 48.2)
- moved C205 99.7 mm to (159.5, 46.4)
- moved C207 99.6 mm to (170.5, 42.3)
- moved C209 99.6 mm to (168.2, 42.3)
- moved C211 99.6 mm to (165.9, 42.3)
- moved L202 99.6 mm to (168.2, 47.4)
- moved C222 99.4 mm to (174.0, 48.2)
- moved C224 99.4 mm to (174.0, 50.4)
- moved C219 99.2 mm to (174.0, 45.9)
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Connections:
- C218 pad 1: +3.3V -> +3V3
- C221 pad 1: +3.3V -> +3V3
- C223 pad 1: +3.3V -> +3V3
- FB501 pad 1: +3.3V -> +3V3
- J303 pad 1: +3V3 -> unconnected-(J303-Pin_1-Pad1)
- J401 pad 5: +3.3V -> +3V3
- L201 pad 2: +3.3V -> +3V3
- R209 pad 1: +3.3V -> +3V3
- SW501 pad 8: (no net) -> unconnected-(SW501-NC-Pad8)
- U202 pad 33: unconnected-(U202A-PAD-Pad33) -> GND
Routing:
- net GND: track 0.00 -> 23.3 mm
- net +BATT: track 0.00 -> 15.9 mm
- net +1V8: track 0.00 -> 9.35 mm
- net /Power supply/PWR_EN: track 0.00 -> 6.63 mm
- net Net-(U202B-FB1): track 0.00 -> 6.63 mm
- net Net-(U202A-VDIV): track 0.00 -> 6.59 mm
- net Net-(U202B-COMP1): track 0.00 -> 5.69 mm
- net Net-(U202C-COMP2): track 0.00 -> 4.52 mm
- net Net-(U202C-FB2): track 0.00 -> 4.30 mm
- net Net-(U202B-LX1): track 0.00 -> 3.97 mm
- net /Power supply/SS_CAP: track 0.00 -> 3.42 mm
- net Net-(U202C-LX2): track 0.00 -> 2.54 mm
- net Net-(U202C-BST2): track 0.00 -> 2.25 mm
- net Net-(U202A-V7V): track 0.00 -> 2.23 mm
- net Net-(U202B-BST1): track 0.00 -> 2.22 mm
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- added copper zone on F.Cu, net +1V8
- added copper zone on F.Cu, net +3V3
- added copper zone on F.Cu, net +BATT
- added copper zone on F.Cu, net GND
- added copper zone on In1.Cu, net GND
- added copper zone on F.Cu, net Net-(U202B-LX1)
- added copper zone on F.Cu, net Net-(U202C-LX2)
Other:
- copper layers 2 -> 4

Commit message: Layout [WIP]
Parts:
- added C517: 0.1uF, Capacitor_SMD:C_0402_1005Metric, F.Cu at (85.4, 50.3)
- added C518: 0.1uF, Capacitor_SMD:C_0402_1005Metric, F.Cu at (85.4, 52.3)
- added C519: 0.1uF, Capacitor_SMD:C_0402_1005Metric, F.Cu at (85.4, 54.3)
- added C520: 0.1uF, Capacitor_SMD:C_0402_1005Metric, F.Cu at (85.4, 56.2)
- added C521: 0.1uF, Capacitor_SMD:C_0402_1005Metric, F.Cu at (85.4, 58.2)
- moved C508 139.5 mm to (93.3, 50.6)
- moved C515 135.6 mm to (93.3, 56.9), turned to -90 degrees
- moved U501 131.4 mm to (98.4, 54.1), turned to 90 degrees
- moved SW101 121.9 mm to (19.3, 56.9)
- moved SW201 121.9 mm to (19.3, 64.9)
- moved C506 115.9 mm to (104.4, 54.2), turned to 90 degrees
- moved R501 112.4 mm to (105.5, 54.2), turned to 90 degrees
- moved X501 105.7 mm to (109.6, 54.1), turned to 180 degrees
- moved C504 104.8 mm to (107.0, 54.8), turned to 180 degrees
- moved TP401 19.0 mm to (115.9, 28.0)
- moved C203 11.5 mm to (160.0, 95.8), turned to 180 degrees
- moved C220 11.3 mm to (159.9, 98.9), turned to 180 degrees
- moved C225 7.05 mm to (167.0, 99.0)
- moved C513 6.79 mm to (236.1, 26.0), turned to 180 degrees
- moved JP201 4.82 mm to (154.2, 97.8)
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Connections:
- net /RF/RFN09 renamed /RF/RF09_N
- net /RF/RFN24 renamed /RF/RF24_N
- net /RF/RFP09 renamed /RF/RF09_P
- net /RF/RFP24 renamed /RF/RF24_P
- U401 pad 22: /FPGA/LVDS_RXCLK_P -> /FPGA/LVDS_RX24_P
- U401 pad 23: /FPGA/LVDS_RXCLK_N -> /FPGA/LVDS_RX24_N
- U401 pad 24: /FPGA/LVDS_RX09_P -> /FPGA/LVDS_RXCLK_P
- U401 pad 25: /FPGA/LVDS_RX09_N -> /FPGA/LVDS_RXCLK_N
- U401 pad 27: /FPGA/LVDS_RX24_P -> /FPGA/LVDS_RX09_P
- U401 pad 28: /FPGA/LVDS_RX24_N -> /FPGA/LVDS_RX09_N
- U401 pad 30: /FPGA/LVDS_TXCLK_P -> /FPGA/LVDS_TX_P
- U401 pad 31: /FPGA/LVDS_TXCLK_N -> /FPGA/LVDS_TX_N
- U401 pad 33: /FPGA/LVDS_TX_P -> /FPGA/LVDS_TXCLK_P
- U401 pad 34: /FPGA/LVDS_TX_N -> /FPGA/LVDS_TXCLK_N
Routing:
- net /FPGA/LVDS_TX_P: track 0.00 -> 7.89 mm
- net /FPGA/LVDS_TX_N: track 0.00 -> 7.43 mm
- net /FPGA/LVDS_TXCLK_P: track 0.00 -> 5.94 mm
- net /FPGA/LVDS_RX09_P: track 0.00 -> 5.86 mm
- net /FPGA/LVDS_TXCLK_N: track 0.00 -> 5.64 mm
- net /FPGA/LVDS_RX09_N: track 0.00 -> 5.56 mm
- net /FPGA/LVDS_RX24_P: track 0.00 -> 4.54 mm
- net /FPGA/LVDS_RX24_N: track 0.00 -> 4.54 mm
- net /FPGA/LVDS_RXCLK_N: track 0.00 -> 3.96 mm
- net /FPGA/LVDS_RXCLK_P: track 0.00 -> 3.96 mm

Commit message: [WIP] Layout
Connectors are now correctly placed for the Nucleo Board
Parts:
- J301, J302, J303: moved to B.Cu
- J304: footprint Connector_PinSocket_2.54mm:PinSocket_1x10_P2.54mm_Vertical -> Connector_PinHeader_2.54mm:PinHeader_1x10_P2.54mm_Vertical; moved to B.Cu
- J305: footprint Connector_PinSocket_2.54mm:PinSocket_1x08_P2.54mm_Vertical -> Connector_PinHeader_2.54mm:PinHeader_1x08_P2.54mm_Vertical; moved to B.Cu
- moved R305 237.2 mm to (255.7, 68.8), turned to 180 degrees
- moved R313 222.1 mm to (246.6, 123.2), turned to 180 degrees
- moved C101 187.9 mm to (208.7, 90.4)
- moved JP301 187.9 mm to (205.3, 122.2)
- moved R101 187.9 mm to (208.8, 88.5)
- moved R307 187.9 mm to (207.4, 117.4)
- moved R308 187.9 mm to (207.4, 119.4)
- moved R312 187.9 mm to (210.4, 119.4)
- moved R314 187.9 mm to (213.3, 115.4)
- moved R315 187.9 mm to (213.3, 117.4)
- moved R316 187.9 mm to (213.3, 119.4)
- moved SW101 187.9 mm to (206.5, 73.0)
- moved SW201 187.9 mm to (206.5, 81.0)
- moved TP301 187.9 mm to (200.8, 105.5)
- moved TP302 187.9 mm to (200.8, 110.1)
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Routing:
- net GND: track 23.3 -> 57.3 mm, vias 0 -> 1
- net /FPGA/VCC: track 0.00 -> 19.5 mm
- net /FPGA/VCCAUX: track 0.00 -> 17.8 mm
- net /RF/DEVDD: track 0.00 -> 9.24 mm
- net Net-(U501-TCXO): track 0.00 -> 7.84 mm
- net Net-(U401F-VCCADC18): track 0.00 -> 4.19 mm
- net /FPGA/VCCIO_3V3: track 0.00 -> 3.84 mm
- net /RF/RF24_N: track 0.00 -> 3.67 mm
- net /RF/RF24_P: track 0.00 -> 3.67 mm
- net /FPGA/LVDS_TX_N: track 7.43 -> 11.1 mm
- net Net-(U501-XTAL2): track 0.00 -> 3.53 mm
- net /FPGA/LVDS_RX24_N: track 4.54 -> 8.06 mm
- net /FPGA/LVDS_RX24_P: track 4.54 -> 8.06 mm
- net /FPGA/LVDS_TXCLK_N: track 5.64 -> 9.15 mm
- net /FPGA/LVDS_TX_P: track 7.89 -> 11.4 mm
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
Commit message: [WIP] Layout
Routed FPGA IOs and LVDS pairs
Parts:
- LS101: value Speaker -> SP-1605; footprint Connector_PinHeader_2.54mm:PinHeader_1x02_P2.54mm_Vertical -> M17_connectors:Pin_1x02_P2.54mm_horizontal_SMD; moved to B.Cu
- moved JP401 110.4 mm to (181.2, 113.0)
- moved C225 100.0 mm to (198.3, 37.9)
- moved R213 100.0 mm to (198.3, 39.1)
- moved C203 100.0 mm to (191.3, 34.7)
- moved C204 100.0 mm to (198.0, 34.2)
- moved C220 100.0 mm to (191.2, 37.8)
- moved R202 100.0 mm to (191.4, 33.2)
- moved R214 100.0 mm to (198.8, 40.9)
- moved R313 100.0 mm to (198.1, 35.7)
- moved U201 100.0 mm to (194.7, 34.4)
- moved U203 100.0 mm to (194.7, 38.9)
- moved TP401 93.0 mm to (133.9, 114.3)
- moved F201 86.1 mm to (156.2, 36.3)
- moved C202 78.4 mm to (166.0, 55.4)
- moved C205 78.4 mm to (175.7, 53.1)
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Connections:
- R309 pad 2: /Connectors/INITN -> /Connectors/SPI_NSS2
- R310 pad 2: /Connectors/SPI_NSS2 -> /Connectors/INITN
- U401 pad 42: /Connectors/IO0 -> /Connectors/IO5
- U401 pad 44: /Connectors/IO1 -> /Connectors/IO4
- U401 pad 51: /Connectors/IO2 -> /Connectors/IO3
- U401 pad 52: /Connectors/IO3 -> /Connectors/IO2
- U401 pad 53: /Connectors/IO4 -> /Connectors/IO1
- U401 pad 55: /Connectors/IO5 -> /Connectors/IO0
Routing:
- net /Connectors/IO4: track 0.00 -> 71.3 mm, vias 0 -> 2
- net /Connectors/IO5: track 0.00 -> 70.5 mm, vias 0 -> 2
- net /Connectors/IO3: track 0.00 -> 66.2 mm, vias 0 -> 2
- net /FPGA/CLK_IN: track 1.76 -> 60.7 mm
- net Net-(J305-Pin_2): track 0.00 -> 56.8 mm, vias 0 -> 2
- net /FPGA/TDI/SSI: track 0.00 -> 56.5 mm, vias 0 -> 2
- net /FPGA/TMS/SCSN: track 0.00 -> 56.2 mm, vias 0 -> 2
- net Net-(J304-Pin_10): track 0.00 -> 55.1 mm
- net /Connectors/PROGRAMN: track 0.00 -> 52.7 mm
- net /FPGA/TCK/SCLK: track 0.00 -> 51.5 mm, vias 0 -> 2
- net Net-(J303-Pin_5): track 0.00 -> 49.2 mm, vias 0 -> 2
- net /Connectors/IO2: track 0.00 -> 48.5 mm, vias 0 -> 1
- net /Connectors/IO1: track 0.00 -> 43.9 mm, vias 0 -> 1
- net /Connectors/IO6: track 0.00 -> 39.9 mm, vias 0 -> 1
- net /Connectors/IO0: track 0.00 -> 38.6 mm, vias 0 -> 1
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
Commit message: [WIP] Layout
Flipped the content upside down for the SMA connector. Reorganized GPIOs. RF routing started.
Parts:
- removed R312: 100R, Resistor_SMD:R_0402_1005Metric
- added R402: 100R, Resistor_SMD:R_0402_1005Metric, F.Cu at (165.0, 81.1)
- added R504: 100R, Resistor_SMD:R_0402_1005Metric, F.Cu at (151.3, 118.4)
- moved C510 135.6 mm to (168.6, 135.4)
- moved FL502 135.4 mm to (164.4, 135.4)
- moved FL501 134.8 mm to (164.4, 129.9)
- moved C509 134.6 mm to (168.6, 130.0)
- moved SW501 126.2 mm to (171.6, 132.4), turned to 180 degrees
- moved C513 126.0 mm to (173.2, 135.1), turned to -90 degrees
- moved C511 125.3 mm to (173.4, 130.0)
- moved C512 124.8 mm to (172.1, 129.9)
- moved J501 113.2 mm to (166.9, 151.7), turned to -90 degrees
- moved C501 98.7 mm to (173.9, 120.5), turned to 0 degrees
- moved L502 69.2 mm to (157.3, 127.9), turned to -90 degrees
- moved C507 65.2 mm to (160.2, 126.2), turned to -90 degrees
- moved R314 65.2 mm to (198.0, 33.0)
- moved L501 63.5 mm to (157.3, 125.3)
- moved X501 62.5 mm to (173.9, 118.3)
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Connections:
- C502 pad 1: /RF/RF24_P -> /RF/RF24_N
- C503 pad 1: /RF/RF24_N -> /RF/RF24_P
- J301 pad 1: /Connectors/IO6 -> Net-(J301-Pin_1)
- J301 pad 2: /Connectors/IO7 -> Net-(J301-Pin_2)
- J301 pad 3: /Connectors/PTT -> Net-(J301-Pin_3)
- J301 pad 4: unconnected-(J301-Pin_4-Pad4) -> Net-(J301-Pin_4)
- J301 pad 5: unconnected-(J301-Pin_5-Pad5) -> /Connectors/PTT
- J303 pad 5: Net-(J303-Pin_5) -> /Connectors/SPI_MISO
- J304 pad 10: Net-(J304-Pin_10) -> /Connectors/IO3
- J304 pad 8: Net-(J304-Pin_8) -> /Connectors/IO4
- J305 pad 1: Net-(J305-Pin_1) -> /Connectors/IO2
- J305 pad 2: Net-(J305-Pin_2) -> unconnected-(J305-Pin_2-Pad2)
- J305 pad 6: /Connectors/IO2 -> unconnected-(J305-Pin_6-Pad6)
- R301 pad 1: /FPGA/TDO/SSO -> Net-(J301-Pin_1)
- R301 pad 2: Net-(J303-Pin_5) -> /Connectors/PGOOD
- R304 pad 1: /FPGA/TMS/SCSN -> /Connectors/SPI_NSS2
- R305 pad 1: Net-(J304-Pin_5) -> Net-(J301-Pin_2)
- R305 pad 2: /Connectors/PGOOD -> /Connectors/DONE
- R306 pad 2: /Connectors/IO5 -> /Connectors/IO6
- R307 pad 2: /Connectors/IO4 -> /Connectors/IO5
- R308 pad 1: Net-(J304-Pin_8) -> Net-(J304-Pin_5)
- R308 pad 2: /Connectors/IO3 -> /Connectors/IO7
- R309 pad 2: /Connectors/SPI_NSS2 -> /FPGA/TMS/SCSN
- R310 pad 1: Net-(J304-Pin_10) -> Net-(J301-Pin_3)
- R310 pad 2: /Connectors/INITN -> /Connectors/PROGRAMN
- R311 pad 1: Net-(J305-Pin_1) -> Net-(J301-Pin_4)
- R311 pad 2: /Connectors/PROGRAMN -> /Connectors/INITN
- U401 pad 42: /Connectors/IO5 -> /Connectors/IO1
- U401 pad 44: /Connectors/IO4 -> /Connectors/IO0
- U401 pad 51: /Connectors/IO3 -> /Connectors/IO2
- U401 pad 52: /Connectors/IO2 -> /Connectors/IO3
- U401 pad 53: /Connectors/IO1 -> /Connectors/IO4
- U401 pad 55: /Connectors/IO0 -> /Connectors/IO5
- U501 pad 44: /FPGA/TDO/SSO -> Net-(U501-MISO)
Routing:
- net /Connectors/SPI_MISO: track 0.00 -> 77.9 mm, vias 0 -> 2
- net Net-(J305-Pin_2): track 56.8 -> 0.00 mm, vias 2 -> 0
- net Net-(J304-Pin_10): track 55.1 -> 0.00 mm
- net /Connectors/IO5: track 70.5 -> 20.5 mm
- net Net-(J303-Pin_5): track 49.2 -> 0.00 mm, vias 2 -> 0
- net Net-(J301-Pin_2): track 0.00 -> 47.9 mm, vias 0 -> 1
- net /Connectors/PROGRAMN: track 52.7 -> 4.89 mm
- net /Connectors/IO4: track 71.3 -> 23.7 mm, vias 2 -> 1
- net Net-(J305-Pin_5): track 0.00 -> 46.2 mm, vias 0 -> 1
- net Net-(J301-Pin_4): track 0.00 -> 42.9 mm
- net Net-(J301-Pin_3): track 0.00 -> 41.7 mm
- net /Connectors/IO3: track 66.2 -> 26.9 mm, vias 2 -> 1
- net Net-(JP401-C): track 38.6 -> 1.04 mm, vias 3 -> 1
- net /FPGA/TMS/SCSN: track 56.2 -> 20.3 mm
- net /FPGA/TDI/SSI: track 56.5 -> 83.4 mm
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
Commit message: Updated PCB layout + step file
PTT and power button now in their final location
Parts:
- added C226: 6.8nF, Capacitor_SMD:C_0402_1005Metric, F.Cu at (136.3, 46.2)
- added C227: 100nF, Capacitor_SMD:C_0402_1005Metric, F.Cu at (142.8, 44.3)
- added C301: 100nF, Capacitor_SMD:C_0402_1005Metric, F.Cu at (132.1, 42.3)
- added R215: 100R, Resistor_SMD:R_0402_1005Metric, F.Cu at (136.3, 44.2)
- added R312: 200kR, Resistor_SMD:R_0402_1005Metric, F.Cu at (129.2, 42.3)
- added R317: 100kR, Resistor_SMD:R_0402_1005Metric, F.Cu at (129.2, 44.3)
- added U204: TPS22810DBVR, Package_TO_SOT_SMD:SOT-23-6, F.Cu at (139.5, 44.7)
- J501: value Conn_Coaxial -> EMPCB.CSMAFSTJ.A; footprint Connector_Coaxial:SMA_Amphenol_132289_EdgeMount -> M17_connectors:SMA_Taoglas_EMPCB.CSMAFSTJ.A
- SW101, SW201: moved to B.Cu
- moved SW101 107.0 mm to (129.1, 129.9), turned to 90 degrees
- moved U201 94.1 mm to (176.5, 126.7)
- moved R202 94.1 mm to (173.2, 125.6)
- moved C203 94.1 mm to (173.3, 127.0)
- moved R313 94.1 mm to (179.8, 128.0)
- moved C204 94.0 mm to (179.8, 126.4)
- moved R314 94.0 mm to (179.8, 125.2)
- moved JP201 93.3 mm to (142.1, 108.3)
- moved R101 87.6 mm to (129.2, 125.0)
- moved D301 86.2 mm to (137.5, 72.0), turned to -90 degrees
- moved TP206 85.5 mm to (179.1, 49.3)
- moved TP204 84.9 mm to (175.4, 49.3)
- moved JP301 84.9 mm to (140.1, 67.7)
- moved C101 84.9 mm to (130.9, 124.5), turned to 90 degrees
- moved TP205 84.9 mm to (179.2, 45.2)
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Connections:
- C509 pad 2: Net-(SW501-RF2) -> Net-(SW501-RF1)
- C510 pad 2: Net-(SW501-RF1) -> Net-(SW501-RF2)
- J301 pad 6: unconnected-(J301-Pin_6-Pad6) -> Net-(J301-Pin_6)
- J302 pad 8: +BATT -> VDD
- J304 pad 8: /Connectors/IO4 -> /Connectors/FPGA_RST
- R306 pad 2: /Connectors/IO6 -> /Connectors/IO5
- R307 pad 2: /Connectors/IO5 -> /Connectors/IO4
- R308 pad 2: /Connectors/IO7 -> /Connectors/IO6
- U401 pad 53: /Connectors/IO4 -> /Connectors/FPGA_RST
- U401 pad 55: /Connectors/IO5 -> /Connectors/IO4
- U401 pad 56: /Connectors/IO6 -> /Connectors/IO5
- U401 pad 57: /Connectors/IO7 -> /Connectors/IO6
Routing:
- net /Connectors/PTT: track 0.00 -> 26.6 mm
- net /Connectors/FPGA_RST: track 0.00 -> 23.7 mm, vias 0 -> 1
- net /Connectors/IO7: track 23.2 -> 0.00 mm, vias 2 -> 0
- net Net-(J501-In): track 0.00 -> 20.1 mm
- net Net-(R101-Pad1): track 0.00 -> 4.63 mm, vias 0 -> 1
- net /Connectors/IO0: track 48.6 -> 44.6 mm
- net Net-(SW501-RF1): track 0.00 -> 3.55 mm
- net Net-(SW501-RF2): track 0.00 -> 3.47 mm
- net /FPGA/LVDS_RX09_P: track 31.7 -> 34.9 mm
- net /FPGA/LVDS_RX09_N: track 31.7 -> 34.9 mm
- net /Connectors/IO4: track 23.7 -> 20.5 mm, vias 1 -> 2
- net /FPGA/LVDS_RX24_P: track 32.0 -> 34.9 mm
- net /FPGA/LVDS_RX24_N: track 32.0 -> 34.9 mm
- net /FPGA/LVDS_RXCLK_P: track 32.0 -> 34.9 mm
- net /FPGA/LVDS_RXCLK_N: track 32.0 -> 34.9 mm
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