File: OpenHT-RF/OpenHT-RF.kicad_pcb (KiCad board)
At the start: 4 copper layers, 60 x 127 mm, 175 parts, among them J201 Conn_01x02, J301 Conn_01x06, J302 Conn_01x08, J303 Conn_02x08_Odd_Even, J304 Conn_01x10, J305 Conn_01x08, J401 Conn_01x06, J501 EMPCB.CSMAFSTJ.A, J502 Conn_01x02, J503 Conn_01x02, SW101 436351045816, SW201 436351045816, SW501 RFSW8008, U201 LTC2954-1, U202 TPS65261RHBx, U203 AP7330-W5-7, U204 TPS22810DBVR, U401 LIFCL-40-7SG72I, U501 AT86RF215, X501 ECS-TXO-20CSMV

Commit message: Power rails routing
Parts:
- moved J502 109.0 mm to (154.0, 138.6), turned to 90 degrees
- moved J503 95.4 mm to (169.7, 126.0), turned to 90 degrees
- moved JP401 79.5 mm to (132.0, 50.7)
- moved TP301 68.0 mm to (115.1, 49.4)
- moved TP302 68.0 mm to (103.8, 45.3)
- moved TP303 68.0 mm to (115.1, 53.2)
- moved TP306 68.0 mm to (111.4, 45.3)
- moved TP201 68.0 mm to (103.7, 49.1)
- moved TP202 68.0 mm to (103.7, 52.9)
- moved TP203 68.0 mm to (107.5, 49.2)
- moved TP204 68.0 mm to (107.5, 53.2)
- moved TP205 68.0 mm to (111.3, 49.1)
- moved TP206 68.0 mm to (111.2, 53.2)
- moved TP304 68.0 mm to (107.7, 45.1)
- moved TP308 68.0 mm to (115.3, 45.2)
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Routing:
- net /Power supply/PWR_EN: track 6.63 -> 129.6 mm
- net /FPGA/VCC: track 18.3 -> 99.6 mm, vias 2 -> 11
- net Net-(J305-Pin_3): track 0.00 -> 36.8 mm, vias 0 -> 1
- net Net-(J305-Pin_4): track 0.00 -> 34.9 mm
- net VDD: track 0.00 -> 30.9 mm
- net Net-(D301-A): track 0.00 -> 30.0 mm
- net +BATT: track 15.9 -> 35.9 mm, vias 0 -> 15
- net /Power supply/SS_CAP: track 3.42 -> 16.1 mm, vias 0 -> 2
- net Net-(U201-~{PB}): track 0.00 -> 7.72 mm, vias 0 -> 1
- net +1V0: track 0.00 -> 6.02 mm
- net +1V8: track 22.3 -> 16.3 mm, vias 0 -> 14
- net /FPGA/VCCAUX: track 17.8 -> 22.7 mm, vias 0 -> 8
- net /Connectors/MCU_NRST: track 0.00 -> 3.80 mm
- net /Connectors/PGOOD: track 0.00 -> 2.42 mm
- net /FPGA/TCK/SCLK: track 76.3 -> 78.4 mm
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- added copper zone on In2.Cu, net +1V8
- added copper zone on In2.Cu, net +BATT

Commit message: Routed FPGA power supply tracks
Parts:
- moved FB501 73.1 mm to (149.4, 113.0), turned to -90 degrees
- moved FB403 49.4 mm to (166.0, 87.2), turned to 180 degrees
- moved FB404 46.9 mm to (166.0, 86.1), turned to 180 degrees
- moved FB402 41.0 mm to (165.7, 74.7), turned to -90 degrees
- moved TP401 39.8 mm to (168.4, 96.1)
- moved R401 11.1 mm to (129.5, 56.1)
- moved C220 7.47 mm to (169.3, 68.3), turned to -90 degrees
- moved JP301 7.24 mm to (139.7, 68.3)
- moved FB401 6.16 mm to (162.1, 67.8)
- moved C225 5.74 mm to (163.7, 68.2), turned to -90 degrees
- moved R213 3.74 mm to (163.2, 65.8), turned to 0 degrees
- moved U203 3.42 mm to (166.5, 66.8), turned to 180 degrees
- moved R214 2.68 mm to (163.7, 64.1), turned to 90 degrees
- moved C409 0.33 mm to (148.1, 83.2)
- moved C411 0.31 mm to (162.7, 79.7)
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Routing:
- net +3V3: track 1.52 -> 25.6 mm, vias 0 -> 8
- net /FPGA/VCCAUX: track 22.7 -> 42.6 mm, vias 8 -> 13
- net +BATT: track 35.9 -> 17.6 mm
- net Net-(U401B-PR13B): track 7.17 -> 24.5 mm
- net /FPGA/VCCIO_3V3: track 5.17 -> 14.8 mm, vias 1 -> 0
- net /FPGA/TCK/SCLK: track 78.4 -> 85.4 mm
- net /Connectors/SPI_MISO: track 77.9 -> 83.0 mm
- net /FPGA/TDI/SSI: track 83.4 -> 88.5 mm
- net +1V8: track 16.3 -> 20.5 mm, vias 14 -> 18
- net /FPGA/VCC: track 99.6 -> 95.8 mm, vias 11 -> 10
- net +1V0: track 6.02 -> 3.69 mm
- net Net-(U401F-VCCADC18): track 5.06 -> 7.37 mm
- net /Connectors/IO0: track 44.3 -> 43.1 mm
- net /FPGA/CLK_IN: track 59.8 -> 60.9 mm
- net /Connectors/IO6: track 22.5 -> 21.9 mm
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- added copper zone on In2.Cu, net +3V3
- added copper zone on In2.Cu, net /FPGA/VCCAUX

Commit message: Power supply routing
Finished routing power to the transceiver
Parts:
- added C522: 10uF, Capacitor_SMD:C_0805_2012Metric, F.Cu at (148.3, 114.7)
- moved R202 1.15 mm to (177.2, 126.9), turned to -90 degrees
- moved C502 1.07 mm to (158.3, 124.3)
- moved C503 1.07 mm to (157.2, 124.3)
- moved L501 1.07 mm to (157.8, 126.2)
- moved L502 1.07 mm to (157.8, 128.9)
- moved C516 1.05 mm to (166.5, 112.9)
- moved C220 0.99 mm to (169.3, 67.3), turned to 90 degrees
- moved R503 0.93 mm to (164.6, 113.4)
- moved FB501 0.92 mm to (149.1, 112.1)
- moved C519 0.50 mm to (165.3, 115.3)
- moved R502 0.40 mm to (166.8, 116.7)
- moved C508 0.26 mm to (154.6, 112.5)
- moved C517 0.18 mm to (153.7, 115.0)
- moved C521 0.17 mm to (153.7, 118.9)
- moved FB401 0.13 mm to (162.1, 67.7)
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Routing:
- net +BATT: track 17.6 -> 98.2 mm, vias 15 -> 16
- net /RF/DEVDD: track 11.5 -> 67.9 mm, vias 0 -> 9
- net +3V3: track 25.6 -> 63.8 mm, vias 8 -> 12
- net GND: track 57.1 -> 62.3 mm, vias 124 -> 180
- net +1V0: track 3.69 -> 4.97 mm
- net Net-(FL502-IN): track 9.22 -> 8.08 mm
- net /FPGA/CLK_IN: track 60.9 -> 61.6 mm
- net /RF/RF24_N: track 3.33 -> 4.02 mm
- net /RF/RF24_P: track 3.33 -> 4.02 mm
- net Net-(J305-Pin_5): track 46.2 -> 46.8 mm
- net +1V8: track 20.5 -> 21.1 mm, vias 18 -> 19
- net Net-(U501-CLKO): track 2.99 -> 2.42 mm
- added copper zone on F.Cu, net /RF/DEVDD
- added copper zone on In2.Cu, net /RF/DEVDD

Commit message: [WIP] PCB Routing
Routed most of the board.
Parts:
- added C523: 1nF, Capacitor_SMD:C_0402_1005Metric, F.Cu at (173.0, 131.3)
- TP201, TP202, TP203, TP204, TP205, TP206, TP301, TP302, TP303, TP304, TP305, TP306, TP307, TP308, TP401: footprint TestPoint:TestPoint_Loop_D2.50mm_Drill1.0mm -> Connector_Pin:Pin_D0.7mm_L6.5mm_W1.8mm_FlatFork
- moved TP302 90.9 mm to (176.8, 99.4), turned to 90 degrees
- moved TP301 82.2 mm to (176.8, 103.6), turned to 90 degrees
- moved TP304 78.9 mm to (176.8, 83.2), turned to 90 degrees
- moved C203 76.6 mm to (173.0, 53.2), turned to 180 degrees
- moved R202 76.4 mm to (174.6, 50.5), turned to 0 degrees
- moved U201 73.4 mm to (176.3, 53.0), turned to 0 degrees
- moved J401 71.6 mm to (176.7, 123.4)
- moved R314 71.5 mm to (179.6, 51.4), turned to 180 degrees
- moved TP303 70.6 mm to (176.9, 87.2), turned to 90 degrees
- moved C204 70.3 mm to (179.6, 52.6), turned to 0 degrees
- moved TP308 70.2 mm to (177.4, 77.9)
- moved R313 68.7 mm to (179.6, 54.2), turned to 180 degrees
- moved TP306 67.6 mm to (173.9, 71.2)
- moved TP203 64.6 mm to (171.1, 38.0)
- moved TP307 59.2 mm to (173.9, 68.5)
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Connections:
- J303 pad 5: /Connectors/SPI_MISO -> /FPGA/TDO/SSO
- R401 pad 1: /FPGA/VCCIO_3V3 -> +3V3
- R402 pad 1: /FPGA/TDO/SSO -> Net-(U401B-PR10B/TDO/SSO)
- R402 pad 2: /Connectors/SPI_MISO -> /FPGA/TDO/SSO
- R504 pad 2: /Connectors/SPI_MISO -> /FPGA/TDO/SSO
- TP308 pad 1: /Connectors/IO7 -> /Connectors/FPGA_RST
- U401 pad 45: /FPGA/TDO/SSO -> Net-(U401B-PR10B/TDO/SSO)
Routing:
- net /FPGA/TDO/SSO: track 4.77 -> 124.7 mm, vias 0 -> 4
- net Net-(U201-~{PB}): track 7.72 -> 93.3 mm
- net /Connectors/SPI_MISO: track 83.5 -> 0.00 mm, vias 2 -> 0
- net /Power supply/PWR_EN: track 129.6 -> 58.6 mm, vias 0 -> 2
- net /Connectors/PGOOD: track 2.42 -> 63.3 mm, vias 0 -> 2
- net +3V3: track 63.8 -> 116.5 mm, vias 12 -> 13
- net /FPGA/TDI/SSI: track 88.5 -> 133.1 mm, vias 2 -> 4
- net Net-(JP401-C): track 1.04 -> 45.1 mm
- net /Connectors/MCU_NRST: track 3.80 -> 45.4 mm, vias 0 -> 2
- net /FPGA/TMS/SCSN: track 20.1 -> 61.6 mm
- net /Connectors/SW_CTL2: track 2.43 -> 43.3 mm, vias 0 -> 1
- net /FPGA/TCK/SCLK: track 85.8 -> 125.1 mm, vias 3 -> 6
- net +BATT: track 98.2 -> 58.9 mm, vias 16 -> 18
- net /Connectors/SW_CTL1: track 2.33 -> 36.6 mm, vias 0 -> 1
- net /Connectors/RF_RST: track 2.13 -> 31.7 mm, vias 1 -> 2
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- added copper zone on B.Cu, net GND
- added copper zone on In2.Cu, net GND

Commit message: [WIP] PCB Routing
Parts:
- removed TP204: TestPoint, Connector_Pin:Pin_D0.7mm_L6.5mm_W1.8mm_FlatFork
- added TP402: TestPoint, Connector_Pin:Pin_D0.7mm_L6.5mm_W1.8mm_FlatFork, F.Cu at (162.0, 66.5)
- SW101, SW201: moved to F.Cu
- moved TP205 21.6 mm to (145.5, 66.2)
- moved C203 13.9 mm to (181.0, 41.9), turned to 90 degrees
- moved R202 11.4 mm to (183.6, 43.5), turned to -90 degrees
- moved U201 9.25 mm to (181.2, 45.1), turned to -90 degrees
- moved TP202 8.17 mm to (140.8, 54.2)
- moved J201 7.22 mm to (137.4, 33.0)
- moved F201 7.22 mm to (139.3, 39.4)
- moved R214 6.38 mm to (167.5, 59.0), turned to 0 degrees
- moved R313 5.77 mm to (180.0, 48.5), turned to 90 degrees
- moved JP201 5.73 mm to (179.6, 55.2)
- moved U203 5.37 mm to (167.1, 61.5)
- moved C220 5.30 mm to (170.1, 62.1)
- moved C225 5.04 mm to (166.5, 64.0), turned to 0 degrees
- moved TP203 4.76 mm to (175.8, 37.2)
- moved C204 4.57 mm to (181.6, 48.5), turned to -90 degrees
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Routing:
- net +BATT: track 58.9 -> 81.7 mm, vias 18 -> 20
- net +3V3: track 116.5 -> 128.6 mm
- net /FPGA/VCC: track 95.0 -> 101.3 mm, vias 10 -> 12
- net Net-(J305-Pin_3): track 41.0 -> 47.2 mm
- net +1V8: track 21.1 -> 25.6 mm
- net Net-(R101-Pad1): track 4.63 -> 8.09 mm, vias 1 -> 0
- net Net-(JP201-B): track 13.9 -> 16.5 mm
- net /Connectors/PGOOD: track 63.3 -> 65.5 mm
- net /Power supply/SS_CAP: track 16.1 -> 18.1 mm
- net /Connectors/MCU_NRST: track 45.4 -> 47.0 mm
- net /Power supply/PWR_EN: track 58.6 -> 60.2 mm
- net Net-(U203-ADJ): track 2.83 -> 4.11 mm
- net GND: track 62.3 -> 61.2 mm, vias 198 -> 215
- net Net-(U201-~{PB}): track 93.3 -> 94.3 mm, vias 1 -> 2
- net /FPGA/TDI/SSI: track 133.1 -> 133.7 mm

Commit message: Updated Power supply
Parts:
- added C228: 470pF, Capacitor_SMD:C_0402_1005Metric, F.Cu at (150.4, 48.2)
- added C229: 470pF, Capacitor_SMD:C_0402_1005Metric, F.Cu at (166.1, 50.4)
- L202: footprint Inductor_SMD:L_Taiyo-Yuden_NR-50xx -> M17_misc_passive:L_Wurth_WE-LQSF-4828
- R207: value 8.66kR -> 1.6kR
- moved U203 0.71 mm to (167.6, 60.9)
- moved C220 0.71 mm to (170.6, 61.5)
- moved C225 0.71 mm to (166.9, 63.4)
- moved FB401 0.71 mm to (164.8, 63.4)
- moved R213 0.71 mm to (164.6, 61.3)
- moved L202 0.52 mm to (165.1, 42.1)
- moved R214 0.46 mm to (167.6, 58.6)
Routing:
- net Net-(U202B-FB1): track 6.58 -> 7.84 mm
- net Net-(U202C-FB2): track 4.75 -> 5.90 mm
- net +1V8: track 25.6 -> 26.7 mm
- net +BATT: track 81.7 -> 81.2 mm
- net Net-(JP201-B): track 16.5 -> 16.0 mm

Commit message: Layout improvements and current measurement jumpers
Parts:
- added JP202: Jumper_2_Bridged, Connector_PinHeader_2.54mm:PinHeader_1x02_P2.54mm_Vertical_SMD_Pin1Right, F.Cu at (140.2, 61.7)
- added JP203: Jumper_2_Bridged, Connector_PinHeader_2.54mm:PinHeader_1x02_P2.54mm_Vertical_SMD_Pin1Right, F.Cu at (179.0, 39.0)
- added JP204: Jumper_2_Bridged, Connector_PinHeader_2.54mm:PinHeader_1x02_P2.54mm_Vertical_SMD_Pin1Right, F.Cu at (169.5, 68.6)
- C101: footprint Capacitor_SMD:C_0402_1005Metric -> Connector_PinHeader_2.54mm:PinHeader_1x02_P2.54mm_Vertical_SMD_Pin1Right
- JP201: footprint Connector_PinHeader_2.54mm:PinHeader_1x02_P2.54mm_Vertical -> Connector_PinHeader_2.54mm:PinHeader_1x02_P2.54mm_Vertical_SMD_Pin1Right
- moved TP205 36.3 mm to (177.6, 49.2)
- moved C226 23.8 mm to (150.0, 44.1)
- moved R215 23.8 mm to (150.0, 42.1)
- moved U204 23.8 mm to (153.0, 42.6)
- moved C227 23.8 mm to (153.7, 40.2)
- moved D301 23.6 mm to (153.1, 38.5)
- moved TP202 15.4 mm to (141.9, 69.6)
- moved JP401 9.62 mm to (140.1, 50.0)
- moved TP206 9.07 mm to (131.4, 37.2)
- moved F201 8.54 mm to (130.9, 40.9), turned to 0 degrees
- moved TP203 8.50 mm to (176.8, 45.6)
- moved TP201 8.19 mm to (134.6, 38.5)
- moved FB401 4.88 mm to (164.6, 68.3)
- moved R401 4.88 mm to (137.3, 55.6), turned to 90 degrees
- moved TP307 2.21 mm to (176.1, 68.2)
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Connections:
- C218 pad 1: +3V3 -> Net-(JP202-A)
- C219 pad 1: +1V8 -> Net-(JP203-A)
- C221 pad 1: +3V3 -> Net-(JP202-A)
- C222 pad 1: +1V8 -> Net-(JP203-A)
- C223 pad 1: +3V3 -> Net-(JP202-A)
- C224 pad 1: +1V8 -> Net-(JP203-A)
- C225 pad 1: +1V0 -> Net-(JP204-A)
- C228 pad 1: +3V3 -> Net-(JP202-A)
- C229 pad 1: +1V8 -> Net-(JP203-A)
- L201 pad 2: +3V3 -> Net-(JP202-A)
- L202 pad 2: +1V8 -> Net-(JP203-A)
- R209 pad 1: +3V3 -> Net-(JP202-A)
- R211 pad 1: +1V8 -> Net-(JP203-A)
- R213 pad 1: +1V0 -> Net-(JP204-A)
- U203 pad 5: +1V0 -> Net-(JP204-A)
Routing:
- net VDD: track 49.8 -> 79.7 mm
- net Net-(D301-A): track 30.4 -> 59.8 mm
- net +BATT: track 81.2 -> 56.2 mm, vias 20 -> 18
- net Net-(JP203-A): track 0.00 -> 24.0 mm, vias 0 -> 11
- net Net-(JP202-A): track 0.00 -> 16.0 mm, vias 0 -> 9
- net Net-(JP204-A): track 0.00 -> 10.9 mm
- net +1V8: track 26.7 -> 16.1 mm, vias 18 -> 9
- net Net-(JP401-C): track 45.1 -> 39.5 mm
- net +3V3: track 128.5 -> 125.0 mm, vias 13 -> 10
- net /FPGA/VCC: track 101.3 -> 97.9 mm, vias 12 -> 10
- net /Connectors/PGOOD: track 65.2 -> 67.1 mm
- net Net-(JP201-B): track 16.0 -> 17.3 mm, vias 2 -> 0
- net /Power supply/PWR_EN: track 60.2 -> 58.9 mm
- net /Connectors/IO6: track 23.9 -> 25.0 mm
- net Net-(J305-Pin_3): track 47.2 -> 48.2 mm
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- added copper zone on F.Cu, net Net-(JP202-A)
- added copper zone on In2.Cu, net Net-(JP202-A)
- added copper zone on F.Cu, net Net-(JP203-A)
- added copper zone on In2.Cu, net Net-(JP203-A)
- removed copper zone on F.Cu, net +1V8
- removed copper zone on F.Cu, net +3V3
