File: OpenHT-RF/OpenHT-RF.kicad_pcb (KiCad board)
At the start: 4 copper layers, 60 x 127 mm, 199 parts, among them J201 Conn_01x02, J202 MS338-10F, J301 Conn_01x06, J302 Conn_01x08, J303 Conn_02x08_Odd_Even, J304 Conn_01x10, J305 Conn_01x08, J401 Conn_01x06, J402 MS300-10F, J501 EMPCB.CSMAFSTJ.A, J502 Conn_01x02, J503 Conn_01x02, J504 MS300-10F, Q201 DMP3099L-7, SW101 436351045816, SW201 436351045816, SW501 RFSW8008, U201 LTC2954-1, U202 TPS65261RHBx, U203 AP7330-W5-7, U204 TPS22810DBVR, U401 LIFCL-40-9SG72C, U501 AT86RF215, X501 ECS-TXO-20CSMV

Commit message: Fixed differential pairs and RF related DRC errors
Parts:
- moved C408 0.06 mm to (218.0, 89.5)
Routing:
- net GND: track 258.7 -> 268.6 mm, vias 905 -> 902

Commit message: Updated stackup
Other:
- board text added: "0.0175 mm"
- board text added: "0.02 mm"
- board text added: "0.215 mm"
- board text added: "1.6400 mm"
- board text added: "4.74"
- board text removed: "0.0152 mm"
- board text removed: "0.02032 mm"
- board text removed: "0.2104 mm"
- board text removed: "1.6268 mm"
- board text removed: "4.5"
